File: Fill_Station_ControlBoard/Fill_Station_ControlBoard.kicad_pcb (KiCad board)
At the start: 2 copper layers, 10 parts, among them J6 RJ45_Wuerth_7499010211A, SW1 CK_KMS2xxG, U1 STM32H747IITx, U2 USBLC6-2SC6, U3 MCP2561-E-P, U5 LAN8742A, Y1 Crystal, Y2 Crystal

Commit message: Assignation footprint pis valeurs resistances del
Parts:
- added C1: *, Capacitor_SMD:C_0603_1608Metric, F.Cu at (388.6, 97.6)
- added C10: 470pF, Capacitor_SMD:C_0603_1608Metric, F.Cu at (384.2, 81.0)
- added C11: 10n, Capacitor_SMD:C_0603_1608Metric, F.Cu at (384.2, 83.5)
- added C12: ~, Capacitor_SMD:C_0603_1608Metric, F.Cu at (384.2, 86.0)
- added C13: ~, Capacitor_SMD:C_0603_1608Metric, F.Cu at (384.2, 88.5)
- added C14: *, Capacitor_SMD:C_0603_1608Metric, F.Cu at (392.6, 97.6)
- added C15: *, Capacitor_SMD:C_0603_1608Metric, F.Cu at (392.6, 100.1)
- added C16: *, Capacitor_SMD:C_0603_1608Metric, F.Cu at (392.6, 102.6)
- added C17: *, Capacitor_SMD:C_0603_1608Metric, F.Cu at (392.6, 105.1)
- added C18: *, Capacitor_SMD:C_0603_1608Metric, F.Cu at (392.6, 107.6)
- added C19: *, Capacitor_SMD:C_0603_1608Metric, F.Cu at (392.6, 110.1)
- added C2: *, Capacitor_SMD:C_0603_1608Metric, F.Cu at (388.6, 100.1)
- added C20: *, Capacitor_SMD:C_0603_1608Metric, F.Cu at (396.6, 97.6)
- added C21: 0.1u, Capacitor_SMD:C_0603_1608Metric, F.Cu at (415.3, 97.6)
- added C22: 10u, Capacitor_SMD:C_0603_1608Metric, F.Cu at (415.3, 100.1)
- added C23: 2.2u, Capacitor_SMD:C_0603_1608Metric, F.Cu at (396.6, 100.1)
- added C24: 2.2u, Capacitor_SMD:C_0603_1608Metric, F.Cu at (396.6, 102.6)
- added C25: 2.2u, Capacitor_SMD:C_0603_1608Metric, F.Cu at (396.6, 105.1)
- added C26: 6pF, Capacitor_SMD:C_0603_1608Metric, F.Cu at (396.6, 107.6)
- added C27: 6pF, Capacitor_SMD:C_0603_1608Metric, F.Cu at (396.6, 110.1)
- added C28: ~, Capacitor_SMD:C_0603_1608Metric, F.Cu at (384.2, 91.0)
- added C29: ~, Capacitor_SMD:C_0603_1608Metric, F.Cu at (388.2, 73.4)
- added C3: *, Capacitor_SMD:C_0603_1608Metric, F.Cu at (388.6, 102.6)
- added C30: ~, Capacitor_SMD:C_0603_1608Metric, F.Cu at (388.2, 76.0)
- added C31: 2.2u, Capacitor_SMD:C_0603_1608Metric, F.Cu at (400.6, 97.6)
- added C32: 100n, Capacitor_SMD:C_0603_1608Metric, F.Cu at (400.6, 100.1)
- added C33: *, Capacitor_SMD:C_0603_1608Metric, F.Cu at (400.6, 102.6)
- added C34: *, Capacitor_SMD:C_0603_1608Metric, F.Cu at (400.6, 105.1)
- added C35: 10n, Capacitor_SMD:C_0603_1608Metric, F.Cu at (388.2, 78.5)
- added C36: 10uF, Capacitor_SMD:C_0603_1608Metric, F.Cu at (388.2, 81.0)
- added C37: 100nF, Capacitor_SMD:C_0603_1608Metric, F.Cu at (388.2, 83.5)
- added C38: 1uF, Capacitor_SMD:C_0603_1608Metric, F.Cu at (388.2, 86.0)
- added C39: 22u, Capacitor_SMD:C_0603_1608Metric, F.Cu at (388.2, 88.5)
- added C4: *, Capacitor_SMD:C_0603_1608Metric, F.Cu at (388.6, 105.1)
- added C40: ~, Capacitor_SMD:C_0603_1608Metric, F.Cu at (388.2, 91.0)
- added C41: ~, Capacitor_SMD:C_0603_1608Metric, F.Cu at (392.2, 73.4)
- added C42: 22u, Capacitor_SMD:C_0603_1608Metric, F.Cu at (392.2, 76.0)
- added C43: 22u, Capacitor_SMD:C_0603_1608Metric, F.Cu at (392.2, 78.5)
- added C44: ~, Capacitor_SMD:C_0603_1608Metric, F.Cu at (392.2, 81.0)
- added C5: *, Capacitor_SMD:C_0603_1608Metric, F.Cu at (388.6, 107.6)
- added C50: ~, Capacitor_SMD:C_0603_1608Metric, F.Cu at (392.2, 83.5)
- added C51: ~, Capacitor_SMD:C_0603_1608Metric, F.Cu at (392.2, 86.0)
- added C6: 0.1uF, Capacitor_SMD:C_0603_1608Metric, F.Cu at (384.2, 73.4)
- added C7: 10uF, Capacitor_SMD:C_0603_1608Metric, F.Cu at (384.2, 76.0)
- added C8: *, Capacitor_SMD:C_0603_1608Metric, F.Cu at (388.6, 110.1)
- added C87: 0.1u, Capacitor_SMD:C_0603_1608Metric, F.Cu at (392.2, 88.5)
- added C9: 1uF, Capacitor_SMD:C_0603_1608Metric, F.Cu at (384.2, 78.5)
- added C92: 10n, Capacitor_SMD:C_0603_1608Metric, F.Cu at (415.3, 102.6)
- added D1: ESDA5V3L, Package_TO_SOT_SMD:SOT-23-3, F.Cu at (403.8, 92.0)
- added D2: LED, LED_SMD:LED_0603_1608Metric, F.Cu at (388.6, 112.7)
- added D4: LED, LED_SMD:LED_0603_1608Metric, F.Cu at (388.6, 115.2)
- added D5: LED, LED_SMD:LED_0603_1608Metric, F.Cu at (388.6, 117.8)
- added R1: 33, Capacitor_SMD:C_0603_1608Metric, F.Cu at (415.6, 90.5)
- added R10: 22k, Resistor_SMD:R_0603_1608Metric_Pad0.98x0.95mm_HandSolder, F.Cu at (406.8, 100.1)
- added R11: 22k, Resistor_SMD:R_0603_1608Metric_Pad0.98x0.95mm_HandSolder, F.Cu at (406.8, 102.6)
- added R12: 22k, Resistor_SMD:R_0603_1608Metric_Pad0.98x0.95mm_HandSolder, F.Cu at (406.8, 105.1)
- added R13: 22k, Resistor_SMD:R_0603_1608Metric_Pad0.98x0.95mm_HandSolder, F.Cu at (406.8, 107.6)
- added R14: 10k, Resistor_SMD:R_0603_1608Metric_Pad0.98x0.95mm_HandSolder, F.Cu at (384.4, 97.6)
- added R15: 0, Resistor_SMD:R_0603_1608Metric_Pad0.98x0.95mm_HandSolder, F.Cu at (384.4, 100.1)
- added R16: 0, Resistor_SMD:R_0603_1608Metric_Pad0.98x0.95mm_HandSolder, F.Cu at (384.4, 102.6)
- added R17: 10k, Resistor_SMD:R_0603_1608Metric_Pad0.98x0.95mm_HandSolder, F.Cu at (400.8, 73.4)
- added R18: 270, Resistor_SMD:R_0603_1608Metric_Pad0.98x0.95mm_HandSolder, F.Cu at (400.8, 76.0)
- added R19: 270, Resistor_SMD:R_0603_1608Metric_Pad0.98x0.95mm_HandSolder, F.Cu at (400.8, 78.5)
- added R2: 33, Resistor_SMD:R_0603_1608Metric_Pad0.98x0.95mm_HandSolder, F.Cu at (396.4, 73.4)
- added R20: 33, Capacitor_SMD:C_0603_1608Metric, F.Cu at (415.6, 93.0)
- added R21: 33, Resistor_SMD:R_0603_1608Metric_Pad0.98x0.95mm_HandSolder, F.Cu at (400.8, 81.0)
- added R22: 33, Resistor_SMD:R_0603_1608Metric_Pad0.98x0.95mm_HandSolder, F.Cu at (400.8, 83.5)
- added R23: 33, Resistor_SMD:R_0603_1608Metric_Pad0.98x0.95mm_HandSolder, F.Cu at (400.8, 86.0)
- added R24: 33, Resistor_SMD:R_0603_1608Metric_Pad0.98x0.95mm_HandSolder, F.Cu at (400.8, 88.5)
- added R25: 33, Resistor_SMD:R_0603_1608Metric_Pad0.98x0.95mm_HandSolder, F.Cu at (405.1, 73.4)
- added R26: 2.5k, Resistor_SMD:R_0603_1608Metric_Pad0.98x0.95mm_HandSolder, F.Cu at (405.1, 76.0)
- added R27: 100k, Resistor_SMD:R_0603_1608Metric_Pad0.98x0.95mm_HandSolder, F.Cu at (384.4, 105.1)
- added R28: 33, Resistor_SMD:R_0603_1608Metric_Pad0.98x0.95mm_HandSolder, F.Cu at (405.1, 78.5)
- added R29: 33, Resistor_SMD:R_0603_1608Metric_Pad0.98x0.95mm_HandSolder, F.Cu at (406.8, 110.1)
- added R3: 5.1k, Resistor_SMD:R_0603_1608Metric_Pad0.98x0.95mm_HandSolder, F.Cu at (396.4, 76.0)
- added R30: 10k, Resistor_SMD:R_0603_1608Metric_Pad0.98x0.95mm_HandSolder, F.Cu at (405.1, 81.0)
- added R31: 10k, Resistor_SMD:R_0603_1608Metric_Pad0.98x0.95mm_HandSolder, F.Cu at (405.1, 83.5)
- added R32: 10k, Resistor_SMD:R_0603_1608Metric_Pad0.98x0.95mm_HandSolder, F.Cu at (405.1, 86.0)
- added R33: 10k, Resistor_SMD:R_0603_1608Metric_Pad0.98x0.95mm_HandSolder, F.Cu at (405.1, 88.5)
- added R34: 33, Resistor_SMD:R_0603_1608Metric_Pad0.98x0.95mm_HandSolder, F.Cu at (411.1, 97.6)
- added R35: 0, Resistor_SMD:R_0603_1608Metric_Pad0.98x0.95mm_HandSolder, F.Cu at (411.1, 100.1)
- added R36: 0, Resistor_SMD:R_0603_1608Metric_Pad0.98x0.95mm_HandSolder, F.Cu at (411.1, 102.6)
- added R37: 0, Resistor_SMD:R_0603_1608Metric_Pad0.98x0.95mm_HandSolder, F.Cu at (411.1, 105.1)
- added R38: 22k, Resistor_SMD:R_0603_1608Metric_Pad0.98x0.95mm_HandSolder, F.Cu at (411.1, 107.6)
- added R39: 10k, Resistor_SMD:R_0603_1608Metric_Pad0.98x0.95mm_HandSolder, F.Cu at (384.4, 107.6)
- added R4: 5.1k, Resistor_SMD:R_0603_1608Metric_Pad0.98x0.95mm_HandSolder, F.Cu at (396.4, 78.5)
- added R40: 0, Resistor_SMD:R_0603_1608Metric_Pad0.98x0.95mm_HandSolder, F.Cu at (384.4, 110.1)
- added R41: 100, Resistor_SMD:R_0603_1608Metric_Pad0.98x0.95mm_HandSolder, F.Cu at (409.5, 73.4)
- added R42: 33, Resistor_SMD:R_0603_1608Metric_Pad0.98x0.95mm_HandSolder, F.Cu at (409.5, 76.0)
- added R43: 33, Resistor_SMD:R_0603_1608Metric_Pad0.98x0.95mm_HandSolder, F.Cu at (409.5, 78.5)
- added R44: 120, Resistor_SMD:R_0603_1608Metric_Pad0.98x0.95mm_HandSolder, F.Cu at (409.5, 81.0)
- added R45: 33, Resistor_SMD:R_0603_1608Metric_Pad0.98x0.95mm_HandSolder, F.Cu at (415.8, 73.4)
- added R46: 10k, Resistor_SMD:R_0603_1608Metric_Pad0.98x0.95mm_HandSolder, F.Cu at (409.5, 83.5)
- added R47: 33, Resistor_SMD:R_0603_1608Metric_Pad0.98x0.95mm_HandSolder, F.Cu at (415.8, 76.0)
- added R48: 0, Resistor_SMD:R_0603_1608Metric_Pad0.98x0.95mm_HandSolder, F.Cu at (409.5, 86.0)
- added R49: 33, Resistor_SMD:R_0603_1608Metric_Pad0.98x0.95mm_HandSolder, F.Cu at (415.8, 78.5)
- added R5: *, Resistor_SMD:R_0603_1608Metric_Pad0.98x0.95mm_HandSolder, F.Cu at (396.4, 81.0)
- added R50: 33, Resistor_SMD:R_0603_1608Metric_Pad0.98x0.95mm_HandSolder, F.Cu at (415.8, 81.0)
- added R51: 33, Resistor_SMD:R_0603_1608Metric_Pad0.98x0.95mm_HandSolder, F.Cu at (415.8, 83.5)
- added R52: 33, Resistor_SMD:R_0603_1608Metric_Pad0.98x0.95mm_HandSolder, F.Cu at (415.8, 86.0)
- added R53: 4.42k, Resistor_SMD:R_0805_2012Metric, F.Cu at (392.8, 112.8)
- added R54: 620, Resistor_SMD:R_0603_1608Metric_Pad0.98x0.95mm_HandSolder, F.Cu at (384.4, 112.6)
- added R55: 280, Resistor_SMD:R_0603_1608Metric_Pad0.98x0.95mm_HandSolder, F.Cu at (384.4, 115.1)
- added R6: 60, Resistor_SMD:R_0603_1608Metric_Pad0.98x0.95mm_HandSolder, F.Cu at (396.4, 83.5)
- added R7: 60, Resistor_SMD:R_0603_1608Metric_Pad0.98x0.95mm_HandSolder, F.Cu at (396.4, 86.0)
- added R8: 12.1k, Resistor_SMD:R_0603_1608Metric_Pad0.98x0.95mm_HandSolder, F.Cu at (396.4, 88.5)
- added R9: 22k, Resistor_SMD:R_0603_1608Metric_Pad0.98x0.95mm_HandSolder, F.Cu at (406.8, 97.6)
- added U3: TCAN337G, Package_TO_SOT_SMD:TSOT-23-8_HandSoldering, F.Cu at (397.7, 92.1)
- Y1: value Crystal -> Crystal 25MHz
- Y2: value Crystal -> Crystal 32.768 kHz
- moved U5 64.3 mm to (106.4, 65.2)
- moved J6 56.6 mm to (186.0, 92.6), turned to 90 degrees
- moved U1 14.6 mm to (134.5, 63.5)
- moved U3 10.2 mm to (143.7, 91.2)
Connections:
- U1 pad 138: unconnected-(U1-PA14-Pad138) -> /JTCK
- U1 pad 139: unconnected-(U1-PA15-Pad139) -> /JTDI
- U1 pad 146: CAN.STBY -> /CAN.STBY
- U1 pad 162: unconnected-(U1-PB3-Pad162) -> /JTDO
- U1 pad 163: unconnected-(U1-PB4-Pad163) -> /NJTRST
- U1 pad 168: CAN.RXD -> /CAN.TXD
- U1 pad 169: CAN.TXD -> /CAN.RXD
- U1 pad 72: unconnected-(U1-PE10-Pad72) -> /GPIO1
- U1 pad 73: unconnected-(U1-PE11-Pad73) -> /GPIO2
- U1 pad 74: unconnected-(U1-PE12-Pad74) -> /GPIO3
- U1 pad 75: unconnected-(U1-PE13-Pad75) -> /GPIO4
- U1 pad 76: unconnected-(U1-PE14-Pad76) -> /GPIO5
- U1 pad 77: unconnected-(U1-PE15-Pad77) -> /GPIO6
- Y1 pad 2: /Eth.CLKIN -> Net-(C26-Pad2)

Commit message: Fait des trucs (commencer arrangement de pièces sur PCB
Parts:
- removed the U3 at (143.7, 91.2)
- added J3: USB_C_Receptacle_USB2.0_14P, Connector_USB:USB_C_Receptacle_Amphenol_12401548E4-2A_CircularHoles, F.Cu at (233.5, 31.5)
- added J5: Micro_SD_Card_Det1, Connector_Card:microSD_HC_Hirose_DM3AT-SF-PEJM5, F.Cu at (180.7, 33.9)
- added J8: DE9_Socket_MountingHoles, Connector_Dsub:DSUB-9_Socket_Vertical_P2.77x2.84mm_MountingHoles, F.Cu at (257.3, 105.2)
- moved R17 451.8 mm to (-48.3, 123.0)
- moved R25 451.8 mm to (-43.9, 123.0)
- moved R33 364.6 mm to (41.6, 116.9), turned to 180 degrees
- moved R41 362.1 mm to (53.5, 140.0), turned to 180 degrees
- moved R26 357.4 mm to (51.7, 128.9), turned to 180 degrees
- moved R28 354.1 mm to (54.0, 124.1), turned to -90 degrees
- moved R31 351.9 mm to (56.0, 127.5), turned to -90 degrees
- moved C11 350.4 mm to (40.2, 149.9), turned to 90 degrees
- moved C30 348.1 mm to (46.5, 142.5), turned to -90 degrees
- moved R32 347.4 mm to (60.5, 130.0), turned to 180 degrees
- moved C50 346.2 mm to (51.5, 145.0), turned to 90 degrees
- moved R53 345.9 mm to (51.5, 56.5), turned to 90 degrees
- moved D4 345.3 mm to (47.5, 61.7), turned to 90 degrees
- moved R8 343.7 mm to (56.5, 139.4), turned to -90 degrees
- moved R19 342.5 mm to (62.9, 135.0)
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Connections:
- net /Communication/CAN.FAULT renamed /CAN.FAULT
- R42 pad 1: /Communication/CAN.TXD -> /CAN.TXD
- R43 pad 1: /Communication/CAN.RXD -> /CAN.RXD
- R5 pad 1: /Communication/CAN.STBY -> /CAN.STBY

Commit message: Modifs de l'organisation des pages
Parts:
- removed C50: ~, Capacitor_SMD:C_0603_1608Metric
- removed C87: 0.1u, Capacitor_SMD:C_0603_1608Metric
- removed C92: 10n, Capacitor_SMD:C_0603_1608Metric
- removed D1: ESDA5V3L, Package_TO_SOT_SMD:SOT-23-3
- removed the D5 at (56.5, 61.5)
- removed the D5 at (149.0, 117.0)
- removed D6: ESD9B3.3ST5G, Diode_SMD:D_SOD-923
- removed R12, R13, R38: 22k, Resistor_SMD:R_0603_1608Metric_Pad0.98x0.95mm_HandSolder
- removed R15, R16, R35, R36, R37, R40, R48: 0, Resistor_SMD:R_0603_1608Metric_Pad0.98x0.95mm_HandSolder
- removed R29, R34, R45, R47, R49, R50, R51, R52: 33, Resistor_SMD:R_0603_1608Metric_Pad0.98x0.95mm_HandSolder
- removed R41: 100, Resistor_SMD:R_0603_1608Metric_Pad0.98x0.95mm_HandSolder
- added C48: 100n, Capacitor_SMD:C_0603_1608Metric, F.Cu at (-57.9, 49.8)
- added C54: 100n, Capacitor_SMD:C_0603_1608Metric, F.Cu at (-57.9, 52.3)
- added C55: 100n, Capacitor_SMD:C_0603_1608Metric, F.Cu at (-57.9, 54.8)
- added C56: 100n, Capacitor_SMD:C_0603_1608Metric, F.Cu at (-57.9, 57.3)
- added C57: 100n, Capacitor_SMD:C_0603_1608Metric, F.Cu at (-57.9, 59.8)
- added D10: BAV99, Package_TO_SOT_SMD:SOT-23, F.Cu at (-97.9, 95.2)
- added D11: BAV99, Package_TO_SOT_SMD:SOT-23, F.Cu at (-97.9, 99.6)
- added D12: BAV99, Package_TO_SOT_SMD:SOT-23, F.Cu at (-97.9, 104.1)
- added D5: LED, LED_SMD:LED_0603_1608Metric, F.Cu at (-33.7, 116.8)
- added J4: Conn_02x05_Counter_Clockwise, Connector_PinSocket_2.00mm:PinSocket_2x05_P2.00mm_Vertical, F.Cu at (-67.9, 63.1)
- added J7: 436500200, MOLEX:MOLEX_436500200, F.Cu at (-79.0, 77.9)
- added J9: 436500200, MOLEX:MOLEX_436500200, F.Cu at (-65.7, 77.9)
- C1, C14, C15, C16, C17, C18, C19, C2, C20, C3, C4, C5, C8: value * -> 100n
- C11: value 10n -> 1u
- C21: value 0.1u -> 100n
- C22: value 10u -> 100n
- C28: footprint Capacitor_SMD:C_0603_1608Metric -> Capacitor_SMD:C_0402_1005Metric
- C36: value 10uF -> 100n
- C39: value 22u -> 1nF
- C40: value ~ -> 1u
- C41, C44: value ~ -> 4.7u
- C42: value 22u -> 1u
- C43: value 22u -> 100n
- C51: value ~ -> 100n
- J5: value Micro_SD_Card_Det1 -> 436500200; footprint Connector_Card:microSD_HC_Hirose_DM3AT-SF-PEJM5 -> MOLEX:MOLEX_436500200
- R10, R11: value 22k -> 49.9
- R5: value * -> 10k
- R6, R7: value 60 -> 49.9
- R9: value 22k -> 33; footprint Resistor_SMD:R_0603_1608Metric_Pad0.98x0.95mm_HandSolder -> Capacitor_SMD:C_0603_1608Metric
- moved C44 307.3 mm to (-57.9, 47.3), turned to 0 degrees
- moved C41 303.6 mm to (-57.9, 39.8), turned to 0 degrees
- moved C40 302.2 mm to (-61.9, 59.8), turned to 0 degrees
- moved C43 298.2 mm to (-57.9, 44.8)
- moved J8 295.4 mm to (-31.9, 44.8), turned to 0 degrees
- moved C42 292.0 mm to (-57.9, 42.3), turned to 0 degrees
- moved R44 287.9 mm to (-51.7, 62.3), turned to 0 degrees
- moved R46 280.5 mm to (-51.7, 64.8), turned to 0 degrees
- moved U3 278.4 mm to (-46.0, 55.9)
- moved R43 278.0 mm to (-51.7, 59.8)
- moved R5 277.7 mm to (-51.7, 54.8)
- moved J5 276.4 mm to (-92.2, 77.9), turned to 0 degrees
- moved R42 271.7 mm to (-51.7, 57.3)
- moved R9 271.7 mm to (-93.4, 96.7), turned to 0 degrees
- moved J3 264.6 mm to (-26.3, 81.5), turned to 0 degrees
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Connections:
- net /CAN.RXD renamed /CAN FD/CAN.RXD
- net /CAN.TXD renamed /CAN FD/CAN.TXD
- net /Communication/LED1 renamed /Ethernet/LED1
- net /Communication/LED2 renamed /Ethernet/LED2
- net /Eth.CRS_DV renamed /Ethernet/Eth.CRS_DV
- net /Eth.MDC renamed /Ethernet/Eth.MDC
- net /Eth.MDIO renamed /Ethernet/Eth.MDIO
- net /Eth.REFCLKO renamed /Ethernet/Eth.REFCLKO
- net /Eth.RST renamed /Ethernet/Eth.RST
- net /Eth.RXD0 renamed /Ethernet/Eth.RXD0
- net /Eth.RXD1 renamed /Ethernet/Eth.RXD1
- net /Eth.RXER renamed /Ethernet/Eth.RXER
- net /Eth.TXD0 renamed /Ethernet/Eth.TXD0
- net /Eth.TXD1 renamed /Ethernet/Eth.TXD1
- net /Eth.TXEN renamed /Ethernet/Eth.TXEN
- net /NJTRST renamed /MCU/NJTRST
- net Net-(U1-BOOT0) renamed /MCU/Boot
- C1 pad 1: 3V3A -> 3V3
- C11 pad 1: Net-(C11-Pad1) -> 3V3
- C19 pad 1: 3V3A -> 3V3
- C20 pad 1: 3V3A -> 3V3
- C26 pad 2: Net-(C26-Pad2) -> Net-(U1-PH0)
- C27 pad 2: Net-(C27-Pad2) -> Net-(U1-PH1)
- C34 pad 1: Net-(C34-Pad1) -> Net-(U1-PC15)
- C39 pad 1: Net-(U3-TXD) -> 3V3
- C39 pad 2: GND -> CHASSIS
- C40 pad 1: Net-(U3-CANL) -> 3V3
- C41 pad 1: Net-(U3-CANH) -> 3V3
- C42 pad 1: Net-(U3-S) -> /MCU/VDD5_USB
- C43 pad 1: /CAN.FAULT -> /MCU/VDD5_USB
- C51 pad 1: Net-(J6-CRD) -> 3V3
- J5 pad 1: Net-(J5-DAT2) -> Net-(J5-Pad1)
- J5 pad 2: Net-(J5-DAT3/CD) -> GND
- J6 pad 1: /Communication/TX_P -> /Ethernet/TX_P
- J6 pad 2: /Communication/TX_N -> /Ethernet/TX_N
- J6 pad 3: Net-(J6-RD+) -> /Ethernet/RX_P
- J6 pad 4: Net-(J6-CTD) -> 3V3
- J6 pad 5: Net-(J6-CRD) -> 3V3
- J6 pad 6: Net-(J6-RD-) -> /Ethernet/RX_N
- J6 pad 8: GND -> CHASSIS
- J6 pad SH: Net-(C11-Pad1) -> CHASSIS
- J8 pad 2: Net-(U3-CANL) -> /CAN FD/CAN_N
- J8 pad 5: Net-(C87-Pad2) -> unconnected-(J8-Pad5)
- J8 pad 6: GND -> unconnected-(J8-Pad6)
- J8 pad 7: Net-(U3-CANH) -> /CAN FD/CAN_P
- R1 pad 2: /Servo.Signal2 -> /Control/Servo.Signal2
- R10 pad 2: Net-(J5-DAT3/CD) -> /Ethernet/RX_P
- R11 pad 2: /SD.CMD -> /Ethernet/RX_N
- R20 pad 1: /Servo.Signal1 -> /Control/Servo.Signal1
- R20 pad 2: Net-(J7-Pin_1) -> Net-(J5-Pad1)
- R44 pad 1: Net-(U3-CANH) -> /CAN FD/CAN_P
- R44 pad 2: Net-(U3-CANL) -> /CAN FD/CAN_N
- R46 pad 2: /CAN.FAULT -> /CAN FD/CAN.FAULT
- R5 pad 1: /CAN.STBY -> Net-(U3-S)
- R5 pad 2: Net-(U3-S) -> GND
- R6 pad 1: Net-(C44-Pad1) -> 3V3
- R6 pad 2: Net-(U3-CANL) -> /Ethernet/TX_P
- R7 pad 1: Net-(U3-CANH) -> 3V3
- R7 pad 2: Net-(C44-Pad1) -> /Ethernet/TX_N
- R9 pad 1: 3V3 -> Net-(J9-Pad1)
- R9 pad 2: Net-(J5-DAT2) -> /Control/Servo.Signal3
- U1 pad 116: /SD.DET -> /MCU/SD.DET
- U1 pad 120: /VDD5_USB -> /MCU/VDD5_USB
- U1 pad 121: /VDD33_USB -> 3V3
- U1 pad 124: /SD.DAT0 -> /MCU/SD.DAT0
- U1 pad 125: /SD.DAT1 -> /MCU/SD.DAT1
- U1 pad 130: USBC.DM -> /MCU/USBC.DM
- U1 pad 131: USBC.DP -> /MCU/USBC.DP
- U1 pad 135: 3V3 -> Net-(C44-Pad1)
- U1 pad 138: /JTCK -> /MCU/JTCK
- U1 pad 139: /JTDI -> /MCU/JTDI
- U1 pad 140: /SD.DAT2 -> /MCU/SD.DAT2
- U1 pad 141: /SD.DAT3 -> /MCU/SD.DAT3
- U1 pad 142: /SD.CLK -> /MCU/SD.CLK
- U1 pad 145: /SD.CMD -> /MCU/SD.CMD
- U1 pad 146: /CAN.STBY -> /CAN FD/CAN.FAULT
- U1 pad 162: /JTDO -> /MCU/JTDO
- U1 pad 175: 3V3 -> Net-(C44-Pad1)
- U1 pad 72: /GPIO1 -> /MCU/GPIO1
- U1 pad 73: /GPIO2 -> /MCU/GPIO2
- U1 pad 74: /GPIO3 -> /MCU/GPIO3
- U1 pad 75: /GPIO4 -> /MCU/GPIO4
- U1 pad 76: /GPIO5 -> /MCU/GPIO5
- U1 pad 77: /GPIO6 -> /MCU/GPIO6
- U1 pad 82: 3V3 -> Net-(C44-Pad1)
- U2 pad 4: USBC.DP -> /MCU/USBC.DM
- U2 pad 6: USBC.DM -> /MCU/USBC.DP
- U3 pad 5: /CAN.FAULT -> /CAN FD/CAN.FAULT
- U3 pad 6: Net-(U3-CANL) -> /CAN FD/CAN_N
- U3 pad 7: Net-(U3-CANH) -> /CAN FD/CAN_P
- U5 pad 20: /Communication/TX_N -> /Ethernet/TX_N
- U5 pad 21: /Communication/TX_P -> /Ethernet/TX_P
- U5 pad 22: Net-(J6-RD-) -> /Ethernet/RX_N
- U5 pad 23: Net-(J6-RD+) -> /Ethernet/RX_P
- U5 pad 5: /Eth.CLKIN -> unconnected-(U5-XTAL1/CLKIN-Pad5)
- Y1 pad 1: Net-(C27-Pad2) -> Net-(U1-PH1)
- Y1 pad 2: Net-(C26-Pad2) -> Net-(U1-PH0)
- Y2 pad 1: Net-(C34-Pad1) -> Net-(U1-PC15)
Routing:
- net /Ethernet/TX_P: track 0.00 -> 11.0 mm
- net /Ethernet/RX_P: track 0.00 -> 10.9 mm, vias 0 -> 2
- net /Ethernet/TX_N: track 0.00 -> 7.59 mm
- net /Ethernet/RX_N: track 0.00 -> 7.26 mm
Other:
- copper layers 2 -> 4

Commit message: début layout
Parts:
- moved J5 293.9 mm to (201.3, 93.5)
- moved D12 293.7 mm to (195.4, 119.6)
- moved R9 293.7 mm to (199.9, 112.3)
- moved D10 293.7 mm to (195.4, 110.7)
- moved D11 293.7 mm to (195.4, 115.2)
- moved J7 293.7 mm to (214.3, 93.5)
- moved J9 293.7 mm to (227.5, 93.5)
- moved R1 293.7 mm to (199.9, 109.8)
- moved R20 293.7 mm to (199.9, 114.8)
- moved J3 244.0 mm to (217.4, 68.2), turned to 90 degrees
- moved C37 226.0 mm to (177.5, 38.2)
- moved C38 226.0 mm to (177.5, 40.8)
- moved R42 226.0 mm to (173.3, 36.2)
- moved R43 226.0 mm to (173.3, 38.7)
- moved R44 226.0 mm to (173.3, 41.2)
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
Commit message: Ajout power
Parts:
- added C26: 10u, Capacitor_SMD:C_0402_1005Metric, F.Cu at (-53.8, 42.4)
- added C27: *, Capacitor_SMD:C_0402_1005Metric, F.Cu at (-53.8, 44.4)
- added C33: 100n, Capacitor_SMD:C_0402_1005Metric, F.Cu at (-53.8, 46.3)
- added C34: 10u, Capacitor_SMD:C_0402_1005Metric, F.Cu at (-53.8, 48.3)
- added C45: 0.1u, Capacitor_SMD:C_0603_1608Metric, F.Cu at (-44.0, 45.8)
- added C46: 10u, Capacitor_SMD:C_0603_1608Metric, F.Cu at (-44.0, 48.3)
- added C49: 1u, Capacitor_SMD:C_0603_1608Metric, F.Cu at (-50.3, 46.3)
- added C50: 1u, Capacitor_SMD:C_0603_1608Metric, F.Cu at (-50.3, 48.8)
- added C52: 100uF_25V, Capacitor_THT:CP_Radial_D6.3mm_P2.50mm, F.Cu at (-41.0, 9.89)
- added C53: 10uF_25V, Capacitor_THT:CP_Radial_D5.0mm_P2.00mm, F.Cu at (-41.5, 17.1)
- added C6: 100n, Capacitor_SMD:C_0402_1005Metric, F.Cu at (-53.8, 38.5)
- added C60: CdV/dT, Capacitor_SMD:C_0603_1608Metric, F.Cu at (-62.3, 7.22)
- added C7: 100n, Capacitor_SMD:C_0402_1005Metric, F.Cu at (-53.8, 40.4)
- added C79: C, Capacitor_SMD:C_0603_1608Metric, F.Cu at (-62.3, 9.73)
- added C80: C, Capacitor_SMD:C_0603_1608Metric, F.Cu at (-62.3, 12.2)
- added C81: C, Capacitor_SMD:C_0603_1608Metric, F.Cu at (-62.3, 14.8)
- added C82: C, Capacitor_SMD:C_0603_1608Metric, F.Cu at (-62.3, 17.3)
- added C83: C, Capacitor_SMD:C_0603_1608Metric, F.Cu at (-62.3, 19.8)
- added C84: C, Capacitor_SMD:C_0603_1608Metric, F.Cu at (-58.3, 7.22)
- added C85: C, Capacitor_SMD:C_0603_1608Metric, F.Cu at (-58.3, 9.73)
- added D1: LED, LED_SMD:LED_0603_1608Metric, F.Cu at (-45.8, 7.26)
- added D13: SMAJ15A, Diode_SMD:D_SMA, F.Cu at (-60.2, 33.2)
- added D6: LED, LED_SMD:LED_0603_1608Metric, F.Cu at (-45.8, 9.85)
- added D7: LED, LED_SMD:LED_0603_1608Metric, F.Cu at (-45.8, 12.4)
- added D8: LED, LED_SMD:LED_0603_1608Metric, F.Cu at (-45.8, 15.0)
- added D9: LED, LED_SMD:LED_0603_1608Metric, F.Cu at (-45.8, 17.6)
- added J10: Screw_Terminal_2_P5.00mm, TerminalBlock_Phoenix:TerminalBlock_Phoenix_PT-1,5-2-5.0-H_1x02_P5.00mm_Horizontal, F.Cu at (-48.7, 26.1)
- added R12: 22, Capacitor_SMD:C_0603_1608Metric, F.Cu at (-38.0, 45.8)
- added R13: 22, Capacitor_SMD:C_0603_1608Metric, F.Cu at (-38.0, 48.3)
- added R15: *, Resistor_SMD:R_0805_2012Metric, F.Cu at (-38.0, 22.5)
- added R16: *, Resistor_SMD:R_0805_2012Metric, F.Cu at (-38.0, 25.4)
- added R29: *, Resistor_SMD:R_0805_2012Metric, F.Cu at (-38.0, 28.4)
- added R34: *, Resistor_SMD:R_0603_1608Metric_Pad0.98x0.95mm_HandSolder, F.Cu at (-50.1, 7.22)
- added R35: *, Resistor_SMD:R_0603_1608Metric_Pad0.98x0.95mm_HandSolder, F.Cu at (-50.1, 9.73)
- added R36: 33, Resistor_SMD:R_0603_1608Metric_Pad0.98x0.95mm_HandSolder, F.Cu at (-43.8, 38.7)
- added R37: 270, Resistor_SMD:R_0603_1608Metric_Pad0.98x0.95mm_HandSolder, F.Cu at (-43.8, 41.2)
- added R38: 10k, Resistor_SMD:R_0603_1608Metric_Pad0.98x0.95mm_HandSolder, F.Cu at (-50.2, 38.7)
- added R40: *, Resistor_SMD:R_0603_1608Metric_Pad0.98x0.95mm_HandSolder, F.Cu at (-50.1, 12.2)
- added R41: *, Resistor_SMD:R_0603_1608Metric_Pad0.98x0.95mm_HandSolder, F.Cu at (-50.1, 14.8)
- added R45: *, Resistor_SMD:R_0603_1608Metric_Pad0.98x0.95mm_HandSolder, F.Cu at (-50.1, 17.3)
- added R47: 0, Resistor_SMD:R_0603_1608Metric_Pad0.98x0.95mm_HandSolder, F.Cu at (-50.2, 41.2)
- added R48: 10k, Resistor_SMD:R_0603_1608Metric_Pad0.98x0.95mm_HandSolder, F.Cu at (-50.2, 43.8)
- added R49: R_US, Resistor_SMD:R_0603_1608Metric, F.Cu at (-58.3, 12.2)
- added R50: R_US, Resistor_SMD:R_0603_1608Metric, F.Cu at (-58.3, 14.8)
- added R51: R_US, Resistor_SMD:R_0603_1608Metric, F.Cu at (-58.3, 17.3)
- added R52: R_US, Resistor_SMD:R_0603_1608Metric, F.Cu at (-58.3, 19.8)
- added R67: R_US, Resistor_SMD:R_0603_1608Metric, F.Cu at (-54.2, 7.22)
- added R68: R_US, Resistor_SMD:R_0603_1608Metric, F.Cu at (-54.2, 9.73)
- added R69: 0, Resistor_SMD:R_0603_1608Metric_Pad0.98x0.95mm_HandSolder, F.Cu at (-50.1, 19.8)
- added R89: R_US, Resistor_SMD:R_0603_1608Metric, F.Cu at (-54.2, 12.2)
- added R90: R_US, Resistor_SMD:R_0603_1608Metric, F.Cu at (-54.2, 14.8)
- added U4: TPS2116DRL, Package_TO_SOT_SMD:SOT-583-8, F.Cu at (-38.3, 31.9)
- added U7: OKI-78SR-5_1.5-W36-C, Converter_DCDC:Converter_DCDC_Murata_OKI-78SR_Vertical, F.Cu at (-60.8, 27.0)
- added Y1: ASV-32.768kHz, Oscillator:Oscillator_SMD_Abracon_ASV-4Pin_7.0x5.1mm, F.Cu at (-59.7, 41.2)
- added Y3: ASV-25.000MHz, Oscillator:Oscillator_SMD_Abracon_ASV-4Pin_7.0x5.1mm, F.Cu at (-59.7, 48.8)
- C1, C14, C15, C16, C17, C18, C19, C2, C20, C3, C4, C5, C54, C55, C56, C57, C8: footprint Capacitor_SMD:C_0603_1608Metric -> Capacitor_SMD:C_0402_1005Metric
- C12: value ~ -> 1u
- C13: value ~ -> 100n
- C21, C22, C48: footprint Capacitor_SMD:C_0603_1608Metric -> Capacitor_SMD:C_0603_1608Metric_Pad1.08x0.95mm_HandSolder
- C28: footprint Capacitor_SMD:C_0402_1005Metric -> Capacitor_SMD:C_0603_1608Metric
- R10, R11: footprint Resistor_SMD:R_0603_1608Metric_Pad0.98x0.95mm_HandSolder -> Capacitor_SMD:C_0603_1608Metric
- R26: value 2.5k -> 1k
- R28: value 33 -> 10k
- R53: value 4.42k -> *
- R54: value 620 -> *
- R55: value 280 -> *
Connections:
- net /MCU/GPIO1 renamed /Control/GPIO1
- net /MCU/GPIO2 renamed /Control/GPIO2
- net /MCU/GPIO3 renamed /Control/GPIO3
- net /MCU/GPIO4 renamed /Control/GPIO4
- net /MCU/GPIO5 renamed /Control/GPIO5
- net /MCU/GPIO6 renamed /Control/GPIO6
- net /MCU/JTCK renamed /MCU/SWCLK
- net /MCU/JTDO renamed /MCU/SWO
- C1 pad 2: GND -> Net-(C1-Pad2)
- C19 pad 2: GND -> Net-(C1-Pad2)
- C20 pad 2: GND -> Net-(C1-Pad2)
- C21 pad 2: GND -> Net-(C1-Pad2)
- C22 pad 2: GND -> Net-(C1-Pad2)
- C36 pad 2: GND -> Net-(C1-Pad2)
- C42 pad 1: /MCU/VDD5_USB -> 5V
- C43 pad 1: /MCU/VDD5_USB -> 5V
- C55 pad 2: GND -> Net-(C1-Pad2)
- C56 pad 2: GND -> Net-(C1-Pad2)
- C57 pad 2: GND -> Net-(C1-Pad2)
- D10 pad 2: +3V3 -> 3V3
- D11 pad 2: +3V3 -> 3V3
- D12 pad 2: +3V3 -> 3V3
- J4 pad 10: /MCU/JTMS -> /MCU/SWDIO
- J4 pad 6: /MCU/NJRST -> /MCU/NRST
- J4 pad 7: /MCU/JTDI -> unconnected-(J4-Pin_7-Pad7)
- R27 pad 2: Net-(U1-NRST) -> /MCU/NRST
- R28 pad 1: /Ethernet/Eth.RXER -> GND
- R53 pad 2: 24V -> 12.8V_BAT
- R54 pad 2: +5V -> 5V
- SW1 pad 2: Net-(U1-NRST) -> /MCU/NRST
- SW1 pad SH: unconnected-(SW1-B-PadSH) -> GND
- U1 pad 10: Net-(U1-PC14) -> /MCU/Clock_32.768khz
- U1 pad 11: Net-(U1-PC15) -> unconnected-(U1-PC15-Pad11)
- U1 pad 110: /Ethernet/Eth.RXER -> unconnected-(U1-PG2-Pad110)
- U1 pad 120: /MCU/VDD5_USB -> 5V
- U1 pad 132: unconnected-(U1-PA13-Pad132) -> /MCU/SWDIO
- U1 pad 139: /MCU/JTDI -> unconnected-(U1-PA15-Pad139)
- U1 pad 146: /CAN FD/CAN.FAULT -> unconnected-(U1-PD3-Pad146)
- U1 pad 157: /Ethernet/Eth.TXD0 -> unconnected-(U1-PG13-Pad157)
- U1 pad 163: /MCU/NJTRST -> unconnected-(U1-PB4-Pad163)
- U1 pad 168: /CAN FD/CAN.TXD -> /CAN FD/CAN.RXD
- U1 pad 169: /CAN FD/CAN.RXD -> /CAN FD/CAN.TXD
- U1 pad 170: unconnected-(U1-PE0-Pad170) -> /CAN FD/CAN.FAULT
- U1 pad 3: unconnected-(U1-PE4-Pad3) -> /Alimentation/LED1
- U1 pad 31: Net-(U1-PH0) -> /MCU/Clock_25Mhz
- U1 pad 32: Net-(U1-PH1) -> unconnected-(U1-PH1-Pad32)
- U1 pad 33: Net-(U1-NRST) -> /MCU/NRST
- U1 pad 4: unconnected-(U1-PE5-Pad4) -> /Alimentation/LED2
- U1 pad 5: unconnected-(U1-PE6-Pad5) -> /Alimentation/LED3
- U1 pad 67: unconnected-(U1-PE7-Pad67) -> /Control/Servo.Signal1
- U1 pad 68: unconnected-(U1-PE8-Pad68) -> /Control/Servo.Signal2
- U1 pad 69: unconnected-(U1-PE9-Pad69) -> /Control/Servo.Signal3
- U1 pad 85: unconnected-(U1-PB12-Pad85) -> /Ethernet/Eth.TXD0
- U2 pad 4: /MCU/USBC.DM -> Net-(R12-Pad1)
- U2 pad 6: /MCU/USBC.DP -> Net-(R13-Pad2)
- U5 pad 14: /Ethernet/Eth.REFCLKO -> Net-(U5-~{INT}/REFCLKO)
