File: Fill_Station_ControlBoard/Fill_Station_ControlBoard.kicad_pcb (KiCad board)
At the start: 4 copper layers, 196 parts, among them IC1 TPS259573DSGR, J1 RJ45_Wuerth_7499010211A, J10 Screw_Terminal_6_P5.00mm, J11 Micro_SD_Card_Det1, J12 Conn_02x05_Counter_Clockwise, J13 Screw_Terminal_2_P5.00mm, J14 DE9_Socket_MountingHoles, J15 USB_C_Receptacle_USB2.0_14P, J2 Ematch1, J3 436500200, J4 436500200, J5 436500200, J6 Ematch2, J7 Screw_Terminal_3_P5.00mm, J8 Screw_Terminal_3_P5.00mm, J9 Screw_Terminal_3_P5.00mm, Q1 AO3400A, Q2 AO3400A, SW1 CK_KMS2xxG, U1 LAN8742A, U2 STM32H747IITx, U3 OKI-78SR-5_1.5-W36-C, U4 TPS62130, U5 TCAN337G, U6 TPS2116DRL, U7 USBLC6-2SC6, Y1 ASV-25.000MHz, Y2 ASV-32.768kHz

Commit message: PCB fait
Parts:
- removed the C30 at (308.7, 23.6)
- removed the C39 at (204.7, 79.5)
- removed the C6 at (276.7, 117.8)
- removed the C7 at (276.7, 120.3)
- removed CR1: ESDCAN02-2BWY, ESDCAN:SOT323-3L_STM
- removed D6: SMAJ15A, Diode_SMD:D_SMA
- removed J11: Micro_SD_Card_Det1, Connector_Card:microSD_HC_Molex_47219-2001
- removed J3, J4, J5: 436500200, MOLEX:MOLEX_436500200
- removed the R50 at (162.6, 86.4)
- removed U5: TCAN337G, Package_TO_SOT_SMD:TSOT-23-8_HandSoldering
- added C14: 100n, Capacitor_SMD:C_0603_1608Metric, F.Cu at (256.2, 104.3)
- added C63: 100n, Capacitor_SMD:C_0603_1608Metric, B.Cu at (250.5, 129.4)
- added C65: 10u, Capacitor_SMD:C_0603_1608Metric, B.Cu at (249.0, 129.4)
- added C67: 10nF, Capacitor_SMD:C_0603_1608Metric, F.Cu at (168.3, 148.9)
- added C68: 1u, Capacitor_SMD:C_0603_1608Metric, F.Cu at (168.3, 147.4)
- added C69: 10u, Capacitor_SMD:C_0603_1608Metric, F.Cu at (168.3, 145.9)
- added C70: 100nF, Capacitor_SMD:C_0603_1608Metric, F.Cu at (181.7, 150.5)
- added C71: 1000p - 2000V, Capacitor_SMD:C_1210_3225Metric, F.Cu at (195.1, 156.5)
- added C72: 1u, Capacitor_SMD:C_0603_1608Metric, F.Cu at (182.9, 161.2)
- added C73: 100nF, Capacitor_SMD:C_0603_1608Metric, F.Cu at (181.2, 161.2)
- added C74: 100n, Capacitor_SMD:C_0603_1608Metric, F.Cu at (248.3, 147.1)
- added C75: 22u, Capacitor_SMD:C_0603_1608Metric, F.Cu at (248.9, 155.3)
- added C76: 1u, Capacitor_SMD:C_0603_1608Metric, F.Cu at (255.9, 151.0)
- added C77: 1u, Capacitor_SMD:C_0603_1608Metric, B.Cu at (250.4, 151.1)
- added C78: 22u, Capacitor_SMD:C_0805_2012Metric, F.Cu at (230.2, 147.7)
- added C79: 1u, Capacitor_SMD:C_0603_1608Metric, F.Cu at (234.8, 155.2)
- added C80: 1u, Capacitor_SMD:C_0603_1608Metric, F.Cu at (250.0, 167.2)
- added C81: 1u, Capacitor_SMD:C_0603_1608Metric, F.Cu at (261.8, 167.2)
- added C82: 10u, Capacitor_SMD:C_0603_1608Metric, F.Cu at (253.0, 153.2)
- added C83: 100n, Capacitor_SMD:C_0402_1005Metric, F.Cu at (189.4, 134.0)
- added C84: 10u, Capacitor_SMD:C_0402_1005Metric, F.Cu at (218.5, 151.1)
- added C85: *, Capacitor_SMD:C_0402_1005Metric, B.Cu at (208.1, 153.9)
- added C86: 100n, Capacitor_SMD:C_0603_1608Metric, F.Cu at (253.1, 123.5)
- added C87: 10u, Capacitor_SMD:C_0603_1608Metric, F.Cu at (188.1, 110.4)
- added C88: 100u, Capacitor_SMD:C_0603_1608Metric, F.Cu at (219.1, 141.1)
- added CR2: ESDCAN02-2BWY, ESDCAN:SOT323-3L_STM, B.Cu at (177.7, 165.0)
- added D16: SMAJ20A, Diode_SMD:D_SMA, F.Cu at (225.2, 164.5)
- added H1: M3_Hole_With_Spacer_H10mm, PCM_SL_Mechanical:MountingHole_3.2mm_With_Spacer_H10mm, F.Cu at (267.0, 93.0)
- added H2: M3_Hole_With_Spacer_H10mm, PCM_SL_Mechanical:MountingHole_3.2mm_With_Spacer_H10mm, F.Cu at (153.0, 93.0)
- added H3: M3_Hole_With_Spacer_H10mm, PCM_SL_Mechanical:MountingHole_3.2mm_With_Spacer_H10mm, F.Cu at (152.0, 174.0)
- added H4: M3_Hole_With_Spacer_H10mm, PCM_SL_Mechanical:MountingHole_3.2mm_With_Spacer_H10mm, F.Cu at (243.7, 173.6)
- added J16: DE9_Socket_MountingHoles, Connector_Dsub:DSUB-9_Socket_Vertical_P2.77x2.84mm_MountingHoles, F.Cu at (179.0, 169.7)
- added J18: Screw_Terminal_3_P3.50mm, TerminalBlock_Phoenix:TerminalBlock_Phoenix_PT-1,5-3-3.5-H_1x03_P3.50mm_Horizontal, F.Cu at (153.0, 121.7)
- added L1: L_Ferrite, Capacitor_SMD:C_0402_1005Metric, B.Cu at (205.7, 155.7)
- added L2: L_Ferrite, Resistor_SMD:R_0402_1005Metric, F.Cu at (189.4, 132.7)
- added L3: 2.2u, Inductor_SMD:L_Coilcraft_XAL4020-XXX, F.Cu at (235.2, 144.7)
- added R83: 1M, Resistor_SMD:R_0603_1608Metric_Pad0.98x0.95mm_HandSolder, B.Cu at (195.1, 156.8)
- added R84: 10k, Resistor_SMD:R_0603_1608Metric_Pad0.98x0.95mm_HandSolder, B.Cu at (170.2, 147.3)
- added R85: 120, Resistor_SMD:R_0603_1608Metric_Pad0.98x0.95mm_HandSolder, F.Cu at (177.6, 163.1)
- added R86: 0, Resistor_SMD:R_0603_1608Metric_Pad0.98x0.95mm_HandSolder, B.Cu at (174.9, 162.5)
- added R87: 10k, Resistor_SMD:R_0603_1608Metric_Pad0.98x0.95mm_HandSolder, F.Cu at (175.4, 147.5)
- added R88: 22, Resistor_SMD:R_0402_1005Metric, F.Cu at (174.1, 148.2)
- added R89: 22, Resistor_SMD:R_0402_1005Metric, F.Cu at (198.0, 109.0)
- added R90: 22, Resistor_SMD:R_0402_1005Metric, F.Cu at (219.0, 138.3)
- added R91: 22, Resistor_SMD:R_0402_1005Metric, B.Cu at (201.0, 113.6)
- added R92: 22, Resistor_SMD:R_0402_1005Metric, B.Cu at (208.0, 113.7)
- added R93: 22, Resistor_SMD:R_0402_1005Metric, F.Cu at (219.0, 137.3)
- added R94: 10k, Resistor_SMD:R_0402_1005Metric, F.Cu at (250.6, 126.7)
- added R95: 10k, Resistor_SMD:R_0402_1005Metric, F.Cu at (250.6, 127.8)
- added R96: 10k, Resistor_SMD:R_0402_1005Metric, F.Cu at (252.3, 129.2)
- added R97: 10k, Resistor_SMD:R_0402_1005Metric, F.Cu at (249.3, 132.5)
- added R98: 10k, Resistor_SMD:R_0402_1005Metric, F.Cu at (250.1, 135.6)
- added SW2: BOOT, Button_Switch_SMD:SW_DPDT_CK_JS202011JCQN, F.Cu at (202.3, 91.3)
- added TP1: TestPoint, TestPoint:TestPoint_Pad_D2.0mm, F.Cu at (234.7, 164.3)
- added TP2: TestPoint, TestPoint:TestPoint_Pad_D2.0mm, F.Cu at (236.8, 92.3)
- added TP3: TestPoint, TestPoint:TestPoint_Pad_D2.0mm, F.Cu at (241.9, 92.4)
- added TP4: TestPoint, TestPoint:TestPoint_Pad_D2.0mm, F.Cu at (247.3, 92.4)
- added TP5: TestPoint, TestPoint:TestPoint_Pad_D2.0mm, F.Cu at (258.2, 96.4)
- added TP6: TestPoint, TestPoint:TestPoint_Pad_D2.0mm, F.Cu at (253.9, 96.7)
- added U8: ISOW1044, Package_SO:SOIC-20W_7.5x12.8mm_P1.27mm, F.Cu at (173.4, 155.7)
- added Y3: ASV-25.000MHz, Oscillator:Oscillator_SMD_Abracon_ASV-4Pin_7.0x5.1mm, F.Cu at (212.9, 149.8)
- C1, C17, C18, C21, C24, C26, C29, C31, C39, C4, C5, C54, C6, R11, R15, R18, R20, R21, R22, R38, R40, R41, R5, R9: moved to B.Cu
- C12: value 0.1u -> 100n
- C16, C40: footprint Capacitor_SMD:C_0603_1608Metric_Pad1.08x0.95mm_HandSolder -> Capacitor_SMD:C_0402_1005Metric
- C23, C42, C9: footprint Capacitor_SMD:C_0603_1608Metric -> Capacitor_SMD:C_0402_1005Metric
- C32: value 100n -> 10u; footprint Capacitor_SMD:C_0402_1005Metric -> Capacitor_SMD:C_0603_1608Metric
- C38: footprint Capacitor_SMD:C_0603_1608Metric_Pad1.08x0.95mm_HandSolder -> Capacitor_SMD:C_0603_1608Metric
- C60: value 100nF -> 100n; moved to F.Cu
- C61: footprint Capacitor_SMD:C_0603_1608Metric -> Capacitor_SMD:C_0805_2012Metric
- C62: value 1uF -> 22u; moved to F.Cu
- C64: value CdV/dT -> 3.3n
- C7, C8: footprint Capacitor_SMD:C_0603_1608Metric -> Resistor_SMD:R_0402_1005Metric
- F1: value Fuse -> 4A
- J10: value Screw_Terminal_6_P5.00mm -> Micro_SD_Card_Det_Hirose_DM3AT; footprint TerminalBlock_Phoenix:TerminalBlock_Phoenix_PT-1,5-6-5.0-H_1x06_P5.00mm_Horizontal -> Connector_Card:microSD_HC_Hirose_DM3AT-SF-PEJM5
- J14: value DE9_Socket_MountingHoles -> Micro_SD_Card_Det_Hirose_DM3AT; footprint Connector_Dsub:DSUB-9_Socket_Vertical_P2.77x2.84mm_MountingHoles -> Connector_Card:microSD_HC_Hirose_DM3AT-SF-PEJM5
- J15: footprint Connector_USB:USB_C_Receptacle_Amphenol_12401548E4-2A_CircularHoles -> Connector_USB:USB_C_Receptacle_GCT_USB4105-xx-A_16P_TopMnt_Horizontal
- J7, J8: value Screw_Terminal_3_P5.00mm -> Screw_Terminal_3_P3.50mm; footprint TerminalBlock_Phoenix:TerminalBlock_Phoenix_PT-1,5-3-5.0-H_1x03_P5.00mm_Horizontal -> TerminalBlock_Phoenix:TerminalBlock_Phoenix_PT-1,5-3-3.5-H_1x03_P3.50mm_Horizontal
- J9: value Screw_Terminal_3_P5.00mm -> Screw_Terminal_6_P3.50mm; footprint TerminalBlock_Phoenix:TerminalBlock_Phoenix_PT-1,5-3-5.0-H_1x03_P5.00mm_Horizontal -> TerminalBlock_Phoenix:TerminalBlock_Phoenix_PT-1,5-6-3.5-H_1x06_P3.50mm_Horizontal
- R1, R19, R2, R3, R4, R7, R8: footprint Resistor_SMD:R_0603_1608Metric_Pad0.98x0.95mm_HandSolder -> Resistor_SMD:R_0402_1005Metric
- R31, R33, R71, R72, R74, R76: value * -> 680
- R49: value 100k -> 10k
- R55, R56: value 33 -> 0
- R57: footprint Resistor_SMD:R_0603_1608Metric_Pad0.98x0.95mm_HandSolder -> Capacitor_SMD:C_0402_1005Metric
- R58: value 10k -> 0; footprint Resistor_SMD:R_0603_1608Metric_Pad0.98x0.95mm_HandSolder -> Capacitor_SMD:C_0402_1005Metric
- R59: footprint Resistor_SMD:R_0805_2012Metric -> Resistor_SMD:R_0603_1608Metric
- R6: footprint Resistor_SMD:R_0603_1608Metric_Pad0.98x0.95mm_HandSolder -> Resistor_SMD:R_0402_1005Metric; moved to B.Cu
- R60: value * -> 100k; footprint Resistor_SMD:R_0805_2012Metric -> Resistor_SMD:R_0603_1608Metric
- R61: value * -> 316k; footprint Resistor_SMD:R_0805_2012Metric -> Resistor_SMD:R_0603_1608Metric
- R62: value 120 -> 22; footprint Resistor_SMD:R_0603_1608Metric_Pad0.98x0.95mm_HandSolder -> Resistor_SMD:R_0402_1005Metric; moved to B.Cu
- R63: value * -> 4.7k; footprint Resistor_SMD:R_0805_2012Metric -> Capacitor_SMD:C_0603_1608Metric
- R64, R69, R70: value * -> 1.5k
- R65: value * -> 365k
- R66: value * -> 100k
- R75: value * -> 10k
- R77: value R_US -> 1k
- SW1: value CK_KMS2xxG -> RESET; footprint Button_Switch_SMD:SW_SPST_CK_KMS2xxGP -> Button_Switch_SMD:SW_DPDT_CK_JS202011JCQN
- moved D10 150.7 mm to (260.8, 149.4)
- moved R70 149.0 mm to (260.7, 151.3), turned to 180 degrees
- moved J10 142.4 mm to (263.1, 129.4), turned to 90 degrees
- moved D9 136.8 mm to (246.8, 142.1), turned to -90 degrees
- moved R69 135.0 mm to (245.9, 144.4), turned to 180 degrees
- moved C38 129.7 mm to (234.8, 158.3), turned to 90 degrees
- moved C32 126.8 mm to (236.5, 152.5)
- moved D11 106.3 mm to (241.8, 99.3), turned to 90 degrees
- moved D8 104.9 mm to (236.8, 98.9), turned to 90 degrees
- moved R71 101.6 mm to (241.8, 96.1), turned to 90 degrees
- moved R64 100.2 mm to (236.8, 95.7), turned to 90 degrees
- moved C54 95.3 mm to (204.6, 129.4), turned to 90 degrees
- moved C22 91.5 mm to (222.8, 119.4), turned to 90 degrees
- moved C31 91.2 mm to (193.9, 134.7)
- moved J14 90.8 mm to (263.1, 113.6), turned to 90 degrees
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Connections:
- net /MCU/SD.CLK renamed /MCU/SD1.CLK
- net /MCU/SD.DAT0 renamed /MCU/SD1.DAT0
- net /MCU/SD.DAT1 renamed /MCU/SD1.DAT1
- net /MCU/SD.DAT2 renamed /MCU/SD1.DAT2
- net /MCU/SD.DAT3 renamed /MCU/SD1.DAT3
- net Net-(L3-Pad1) renamed /Alimentation/3V3_SW
- net Net-(U1-TXD0) renamed /Ethernet/TXD_P
- net Net-(U1-TXD1) renamed /Ethernet/TXD_N
- C15 pad 1: /MCU/NRST -> 3V3
- C32 pad 1: 3V3 -> 12.8V
- C38 pad 1: 3V3 -> 12.8V_BAT
- C55 pad 2: Net-(C55-Pad2) -> GND
- C56 pad 2: Net-(C55-Pad2) -> GND
- C58 pad 2: Net-(C55-Pad2) -> GND
- C6 pad 1: 3V3A -> 3V3A_Eth
- C60 pad 1: 3V3 -> 12.8V
- C62 pad 1: 3V3 -> 5V_BAT
- C7 pad 1: 3V3A -> 3V3A_Eth
- C8 pad 1: 3V3A -> 3V3A_Eth
- C9 pad 1: 3V3A -> 3V3A_Eth
- J1 pad 4: 3V3A -> 3V3A_Eth
- J1 pad 5: 3V3A -> 3V3A_Eth
- J1 pad 8: unconnected-(J1-Pad8) -> CHASSIS_ETH
- J1 pad SH: CHASSIS -> CHASSIS_ETH
- J10 pad 1: /Control/GPIO1 -> Net-(J10-DAT2)
- J10 pad 2: /Control/GPIO2 -> Net-(J10-DAT3/CD)
- J10 pad 3: /Control/GPIO3 -> /MCU/SD2.CMD
- J10 pad 4: /Control/GPIO4 -> 3V3
- J10 pad 5: /Control/GPIO5 -> Net-(J10-CLK)
- J10 pad 6: /Control/GPIO6 -> GND
- J14 pad 1: unconnected-(J14-Pad1) -> Net-(J14-DAT2)
- J14 pad 2: /CAN FD/CAN_N -> Net-(J14-DAT3/CD)
- J14 pad 3: GND -> /MCU/SD1.CMD
- J14 pad 4: unconnected-(J14-Pad4) -> 3V3
- J14 pad 5: unconnected-(J14-Pad5) -> Net-(J14-CLK)
- J14 pad 6: unconnected-(J14-Pad6) -> GND
- J14 pad 7: /CAN FD/CAN_P -> Net-(J14-DAT0)
- J14 pad 8: unconnected-(J14-Pad8) -> Net-(J14-DAT1)
- J14 pad 9: unconnected-(J14-Pad9) -> GND
- J2 pad 2: Net-(Q1-D) -> Net-(J2-Pad2)
- J6 pad 2: Net-(Q2-D) -> Net-(J6-Pad2)
- J7 pad 1: /Control/Servo1 -> /Control/Servo2
- J7 pad 3: /Control/Heater1 -> /Control/Heater2
- J8 pad 1: /Control/Servo2 -> /Control/Servo3
- J8 pad 3: /Control/Heater2 -> /Control/Heater3
- J9 pad 1: /Control/Servo3 -> /Control/GPIO1
- J9 pad 2: GND -> /Control/GPIO2
- J9 pad 3: /Control/Heater3 -> /Control/GPIO3
- R18 pad 1: 3V3A -> 3V3A_Eth
- R20 pad 1: 3V3A -> 3V3A_Eth
- R21 pad 1: 3V3A -> 3V3A_Eth
- R22 pad 1: 3V3A -> 3V3A_Eth
- R38 pad 2: Net-(J11-DAT2) -> Net-(J14-DAT2)
- R39 pad 2: Net-(J11-DAT0) -> Net-(J14-DAT0)
- R40 pad 2: Net-(J11-DAT3/CD) -> Net-(J14-DAT3/CD)
- R41 pad 2: Net-(J11-CLK) -> Net-(J14-CLK)
- R42 pad 2: Net-(J11-DAT1) -> Net-(J14-DAT1)
- R43 pad 2: Net-(J11-DAT2) -> Net-(J14-DAT2)
- R44 pad 2: Net-(J11-DAT3/CD) -> Net-(J14-DAT3/CD)
- R45 pad 2: /MCU/SD.CMD -> /MCU/SD1.CMD
- R46 pad 2: Net-(J11-DAT0) -> Net-(J14-DAT0)
- R47 pad 2: Net-(J11-DAT1) -> Net-(J14-DAT1)
- R49 pad 1: 3V3 -> Net-(SW1-B)
- R55 pad 1: /CAN FD/CAN.TXD -> Net-(J2-Pad2)
- R55 pad 2: Net-(U5-TXD) -> Net-(Q1-D)
- R56 pad 1: /CAN FD/CAN.RXD -> Net-(J6-Pad2)
- R56 pad 2: Net-(U5-RXD) -> Net-(Q2-D)
- R57 pad 2: /CAN FD/CAN.FAULT -> Net-(Y3-EN)
- R58 pad 2: GND -> /Ethernet/Eth_Clock_25Mhz
- R62 pad 1: /CAN FD/CAN_P -> /MCU/SD2.DAT2
- R62 pad 2: /CAN FD/CAN_N -> Net-(J10-DAT2)
- R65 pad 2: 5V_BAT -> 5V_USB
- R78 pad 2: VDD_3V3 -> 3V3
- SW1 pad 2: /MCU/NRST -> Net-(SW1-B)
- U1 pad 1: 3V3A -> 3V3A_Eth
- U1 pad 19: 3V3A -> 3V3A_Eth
- U1 pad 5: /MCU/Clock_25Mhz -> /Ethernet/Eth_Clock_25Mhz
- U2 pad 145: /MCU/SD.CMD -> /MCU/SD1.CMD
- U2 pad 146: unconnected-(U2-PD3-Pad146) -> /Alimentation/LED1
- U2 pad 147: unconnected-(U2-PD4-Pad147) -> /Alimentation/LED2
- U2 pad 148: unconnected-(U2-PD5-Pad148) -> /Alimentation/LED3
- U2 pad 149: unconnected-(U2-PD6-Pad149) -> /MCU/SD2.CLK
- U2 pad 162: /MCU/SWO -> /MCU/SD2.DAT2
- U2 pad 163: unconnected-(U2-PB4-Pad163) -> /MCU/SD2.DAT3
- U2 pad 169: /CAN FD/CAN.TXD -> Net-(U2-PB9)
- U2 pad 170: /CAN FD/CAN.FAULT -> /MCU/CAN.FAULT
- U2 pad 2: unconnected-(U2-PE3-Pad2) -> /Control/Heater1
- U2 pad 3: /Alimentation/LED1 -> /Control/Heater2
- U2 pad 4: /Alimentation/LED2 -> /Control/Heater3
- U2 pad 41: unconnected-(U2-PA0-Pad41) -> /MCU/SD2.CMD
- U2 pad 5: /Alimentation/LED3 -> unconnected-(U2-PE6-Pad5)
- U2 pad 87: unconnected-(U2-PB14-Pad87) -> /MCU/SD2.DAT0
- U2 pad 88: unconnected-(U2-PB15-Pad88) -> /MCU/SD2.DAT1
- U2 pad 89: unconnected-(U2-PD8-Pad89) -> /Control/E-match1_Cont
- U2 pad 90: unconnected-(U2-PD9-Pad90) -> /Control/E-match2_Cont
- U2 pad 95: unconnected-(U2-PD12-Pad95) -> /Control/E-match2_Det
- U2 pad 96: unconnected-(U2-PD13-Pad96) -> /Control/E-match2
- U2 pad 97: unconnected-(U2-PD14-Pad97) -> /Control/E-match1_Det
- U2 pad 98: unconnected-(U2-PD15-Pad98) -> /Control/E-match1
- U6 pad 3: 5V_BAT -> 5V_USB
- U6 pad 5: 5V_BAT -> 5V_USB
- U6 pad 6: 5V_USB -> 5V_BAT
Routing:
- net /CAN FD/CAN.RXD: track 0.00 -> 70.1 mm
- net Net-(J10-DAT3/CD): track 0.00 -> 69.9 mm, vias 0 -> 3
- net Net-(J10-DAT2): track 0.00 -> 68.5 mm, vias 0 -> 3
- net /Control/Heater3: track 0.00 -> 68.0 mm, vias 0 -> 1
- net /MCU/SD2.CMD: track 0.00 -> 67.1 mm, vias 0 -> 4
- net /CAN FD/CAN.TXD: track 0.00 -> 66.5 mm
- net Net-(J10-CLK): track 0.00 -> 64.5 mm, vias 0 -> 1
- net /Control/E-match2_Det: track 0.00 -> 64.2 mm, vias 0 -> 2
- net /Control/Servo.Signal3: track 5.80 -> 69.9 mm, vias 0 -> 2
- net /Control/E-match1: track 0.00 -> 63.0 mm, vias 0 -> 2
- net /Control/Heater2: track 0.00 -> 59.8 mm, vias 0 -> 1
- net /Control/E-match2: track 0.00 -> 59.5 mm
- net Net-(J14-SHIELD): track 0.00 -> 54.9 mm
- net /Control/E-match1_Det: track 0.00 -> 54.9 mm, vias 0 -> 2
- net /Control/Servo.Signal2: track 5.99 -> 60.6 mm, vias 0 -> 2
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- added copper zone on F.Cu, net /Alimentation/3V3_SW
- added copper zone on F.Cu, net 3V3
- added copper zone on In3.Cu, net 5V
- added copper zone on F.Cu, net CHASSIS_CAN
- added copper zone on In1.Cu, net CHASSIS_CAN
- added copper zone on In2.Cu, net CHASSIS_CAN
- added copper zone on In3.Cu, net CHASSIS_CAN
- added copper zone on In4.Cu, net CHASSIS_CAN
- added copper zone on F.Cu, net CHASSIS_ETH
- added copper zone on In1.Cu, net CHASSIS_ETH
- added copper zone on In2.Cu, net CHASSIS_ETH
- added copper zone on In3.Cu, net CHASSIS_ETH
- added copper zone on In4.Cu, net CHASSIS_ETH
- added copper zone on F.Cu, net GND
- added copper zone on In4.Cu, net GND
Other:
- board outline added: 124 x 90 mm
- copper layers 4 -> 6
- board text added: "3V3"
- board text added: "5V"
- board text added: "GND1"
- board text added: "GND2"

Commit message: Travail Layout
Parts:
- removed C15, C9: 100n, Capacitor_SMD:C_0402_1005Metric
- removed C60, C74: 100n, Capacitor_SMD:C_0603_1608Metric
- removed C62, C75: 22u, Capacitor_SMD:C_0603_1608Metric
- removed C71: 1000p - 2000V, Capacitor_SMD:C_1210_3225Metric
- removed C8: 100n, Resistor_SMD:R_0402_1005Metric
- removed C84: 10u, Capacitor_SMD:C_0402_1005Metric
- removed C85: *, Capacitor_SMD:C_0402_1005Metric
- removed R10, R11, R13, R14, R15, R16, R17, R5, R9: 10k, Resistor_SMD:R_0603_1608Metric_Pad0.98x0.95mm_HandSolder
- removed R12: 1k, Resistor_SMD:R_0603_1608Metric_Pad0.98x0.95mm_HandSolder
- removed R18, R20, R21, R22: 49.9, Resistor_SMD:R_0603_1608Metric_Pad0.98x0.95mm_HandSolder
- removed R19: 12.1k, Resistor_SMD:R_0402_1005Metric
- removed R23, R24: 270, Resistor_SMD:R_0603_1608Metric_Pad0.98x0.95mm_HandSolder
- removed R57: 10k, Capacitor_SMD:C_0402_1005Metric
- removed R58: 0, Capacitor_SMD:C_0402_1005Metric
- removed R6, R7, R8: 22, Resistor_SMD:R_0402_1005Metric
- removed R83: 1M, Resistor_SMD:R_0603_1608Metric_Pad0.98x0.95mm_HandSolder
- removed Y3: ASV-25.000MHz, Oscillator:Oscillator_SMD_Abracon_ASV-4Pin_7.0x5.1mm
- added C100: 10u, Capacitor_SMD:C_0603_1608Metric, F.Cu at (164.1, 139.2)
- added C101: 10u, Capacitor_SMD:C_0603_1608Metric, F.Cu at (199.8, 137.2)
- added C102: 1u, Capacitor_SMD:C_0603_1608Metric, F.Cu at (199.8, 138.7)
- added C103: 100n, Capacitor_SMD:C_0402_1005Metric, F.Cu at (199.4, 140.6)
- added C104: 10n, Capacitor_SMD:C_0402_1005Metric, F.Cu at (199.4, 141.6)
- added C105: 1000p - 2000V, Capacitor_SMD:C_1210_3225Metric, F.Cu at (192.8, 132.3)
- added C89: 1000p - 2000V, Capacitor_SMD:C_1210_3225Metric, F.Cu at (190.9, 118.4)
- added C90: 100n, Capacitor_SMD:C_0402_1005Metric, F.Cu at (208.3, 97.9)
- added C91: 100n, Capacitor_SMD:C_0402_1005Metric, F.Cu at (249.3, 113.6)
- added C92: 100n, Capacitor_SMD:C_0402_1005Metric, F.Cu at (157.8, 136.4)
- added C93: 1000p - 2000V, Capacitor_SMD:C_1210_3225Metric, F.Cu at (193.1, 153.7)
- added C94: 100n, Capacitor_SMD:C_0402_1005Metric, F.Cu at (198.5, 155.8)
- added C95: 10u, Capacitor_SMD:C_0402_1005Metric, F.Cu at (197.5, 155.7)
- added C96: *, Capacitor_SMD:C_0402_1005Metric, B.Cu at (200.4, 147.1)
- added C97: 1u, Capacitor_SMD:C_0603_1608Metric, F.Cu at (164.1, 136.7)
- added C98: 100n, Capacitor_SMD:C_0402_1005Metric, F.Cu at (157.8, 144.3)
- added C99: 10n, Capacitor_SMD:C_0402_1005Metric, F.Cu at (157.8, 146.3)
- added D10: LED, LED_SMD:LED_0603_1608Metric, F.Cu at (263.7, 234.2)
- added L4: L_Ferrite, Capacitor_SMD:C_0402_1005Metric, F.Cu at (201.2, 135.8)
- added R100: 22, Resistor_SMD:R_0402_1005Metric, F.Cu at (228.4, 108.2)
- added R101: 22, Resistor_SMD:R_0402_1005Metric, F.Cu at (202.6, 140.7)
- added R102: 6.49k, Resistor_SMD:R_0402_1005Metric, B.Cu at (201.5, 148.0)
- added R103: 22, Resistor_SMD:R_0402_1005Metric, F.Cu at (232.3, 137.8)
- added R104: 22, Resistor_SMD:R_0402_1005Metric, F.Cu at (204.9, 144.4)
- added R106: 1M, Resistor_SMD:R_0603_1608Metric_Pad0.98x0.95mm_HandSolder, F.Cu at (164.6, 142.2)
- added R107: 270, Resistor_SMD:R_0603_1608Metric_Pad0.98x0.95mm_HandSolder, F.Cu at (197.8, 133.5)
- added R111: 10k, Capacitor_SMD:C_0402_1005Metric, B.Cu at (202.4, 155.6)
- added R112: 0, Capacitor_SMD:C_0402_1005Metric, F.Cu at (200.4, 147.1)
- added R113: 22, Resistor_SMD:R_0402_1005Metric, F.Cu at (235.4, 138.0)
- added R114: 22, Resistor_SMD:R_0402_1005Metric, F.Cu at (236.4, 138.0)
- added R115: 22, Resistor_SMD:R_0402_1005Metric, F.Cu at (204.6, 145.9)
- added R116: 22, Resistor_SMD:R_0402_1005Metric, F.Cu at (204.6, 146.9)
- added R117: 10k, Resistor_SMD:R_0603_1608Metric_Pad0.98x0.95mm_HandSolder, B.Cu at (202.0, 137.3)
- added R118: 10k, Resistor_SMD:R_0603_1608Metric_Pad0.98x0.95mm_HandSolder, F.Cu at (162.6, 151.0)
- added R119: 10k, Resistor_SMD:R_0603_1608Metric_Pad0.98x0.95mm_HandSolder, B.Cu at (168.9, 134.8)
- added R120: 10k, Resistor_SMD:R_0603_1608Metric_Pad0.98x0.95mm_HandSolder, F.Cu at (163.3, 145.3)
- added R70: 1.5k, Resistor_SMD:R_0603_1608Metric_Pad0.98x0.95mm_HandSolder, F.Cu at (267.9, 231.4)
- added R99: 22, Resistor_SMD:R_0402_1005Metric, F.Cu at (231.1, 108.2)
- added U5: DP83825I, Package_DFN_QFN:Texas_RMQ0024A_WQFN-24-1EP_3x3mm_P0.4mm_EP1.9x1.9mm, F.Cu at (201.9, 143.8)
- added Y4: ASV-25.000MHz, Oscillator:Oscillator_SMD_Abracon_ASV-4Pin_7.0x5.1mm, F.Cu at (202.4, 153.8)
- C1: value 1u -> 10u; moved to F.Cu
- C2: value 1uF -> 0.1u
- C3: value 470pF -> 3.3n
- C33, C53, R73, R78, R85, R87, R90, R93: moved to B.Cu
- C4: value 100n -> 22u; footprint Capacitor_SMD:C_0603_1608Metric -> Capacitor_SMD:C_0805_2012Metric; moved to F.Cu
- C5: value 10u -> 22u; footprint Capacitor_SMD:C_0603_1608Metric -> Capacitor_SMD:C_0805_2012Metric; moved to F.Cu
- C6, C63, C65, C77, R38, R40, R41, R62, R84, R91, R92: moved to F.Cu
- C7: value 100n -> 1000p - 2000V; footprint Resistor_SMD:R_0402_1005Metric -> Capacitor_SMD:C_1210_3225Metric
- J1: value RJ45_Wuerth_7499010211A -> RJ45_Wuerth_74980111211; footprint Connector_RJ:RJ45_Wuerth_7499010211A_Horizontal -> Connector_RJ:RJ45_Wuerth_74980111211_Horizontal
- L1: value L_Ferrite -> 2.2u; footprint Capacitor_SMD:C_0402_1005Metric -> Inductor_SMD:L_Coilcraft_XAL4020-XXX; moved to F.Cu
- R1: value 22 -> 10k; footprint Resistor_SMD:R_0402_1005Metric -> Resistor_SMD:R_0603_1608Metric_Pad0.98x0.95mm_HandSolder; moved to B.Cu
- R2: value 22 -> 100k; footprint Resistor_SMD:R_0402_1005Metric -> Resistor_SMD:R_0603_1608Metric
- R3: value 22 -> 100k; footprint Resistor_SMD:R_0402_1005Metric -> Resistor_SMD:R_0603_1608Metric; moved to B.Cu
- R4: value 22 -> 316k; footprint Resistor_SMD:R_0402_1005Metric -> Resistor_SMD:R_0603_1608Metric; moved to B.Cu
- R53: footprint Resistor_SMD:R_0603_1608Metric_Pad0.98x0.95mm_HandSolder -> Capacitor_SMD:C_0402_1005Metric
- U1: value LAN8742A -> TPS62130; footprint Package_DFN_QFN:VQFN-24-1EP_4x4mm_P0.5mm_EP2.5x2.5mm_ThermalVias -> Package_DFN_QFN:VQFN-16-1EP_3x3mm_P0.5mm_EP1.68x1.68mm_ThermalVias
- U3: value OKI-78SR-5_1.5-W36-C -> INA3221; footprint Converter_DCDC:Converter_DCDC_Murata_OKI-78SR_Vertical -> Package_DFN_QFN:Texas_RGV0016A_VQFN-16-1EP_4x4mm_P0.65mm_EP2.1x2.1mm
- moved D14 151.6 mm to (263.7, 244.6), turned to 0 degrees
- moved D13 148.6 mm to (263.7, 242.0), turned to 0 degrees
- moved R76 147.3 mm to (267.9, 241.5), turned to 0 degrees
- moved D12 145.6 mm to (263.7, 239.4), turned to 0 degrees
- moved R74 144.4 mm to (267.9, 238.9), turned to 0 degrees
- moved TP2 143.3 mm to (272.1, 231.2)
- moved TP4 141.8 mm to (276.1, 231.2)
- moved R72 141.5 mm to (267.9, 236.4), turned to 0 degrees
- moved R71 140.3 mm to (267.9, 233.9), turned to 0 degrees
- moved D11 139.2 mm to (263.7, 236.8), turned to 0 degrees
- moved TP3 139.0 mm to (276.1, 227.2)
- moved TP6 137.1 mm to (280.2, 231.2)
- moved R64 134.3 mm to (267.9, 226.4), turned to 0 degrees
- moved D8 132.9 mm to (263.7, 229.0), turned to 0 degrees
- moved TP5 132.6 mm to (280.2, 227.2)
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Connections:
- C1 pad 1: 3V3 -> 12.8V
- C2 pad 1: Net-(U1-VDDCR) -> 12.8V
- C3 pad 1: Net-(U1-VDDCR) -> Net-(U1-SS/TR)
- C4 pad 1: 3V3 -> 3V3_Bat
- C5 pad 1: 3V3 -> 3V3_Bat
- C55 pad 1: 5V -> 5V_USB
- C56 pad 1: 5V -> 5V_USB
- C6 pad 1: 3V3A_Eth -> 3V3
- C61 pad 1: 3V3 -> 3V3_USB
- C7 pad 1: 3V3A_Eth -> GND
- C7 pad 2: GND -> CHASSIS_CAN
- C76 pad 1: 5V_USB -> 3V3_USB
- C77 pad 1: 5V_BAT -> 3V3_Bat
- C78 pad 1: 3V3 -> 3V3_USB
- C82 pad 1: 5V -> 3V3
- J1 pad 1: /Ethernet/TX_P -> unconnected-(J1-Pad1)
- J1 pad 10: GND -> CHASSIS_ETH
- J1 pad 11: GND -> /Ethernet/LED0
- J1 pad 2: /Ethernet/TX_N -> unconnected-(J1-Pad2)
- J1 pad 3: /Ethernet/RX_P -> /Ethernet/TX_P
- J1 pad 4: 3V3A_Eth -> Net-(J1-RCT)
- J1 pad 5: 3V3A_Eth -> /Ethernet/TX_N
- J1 pad 6: /Ethernet/RX_N -> /Ethernet/RX_P
- J1 pad 7: unconnected-(J1-NC-Pad7) -> Net-(J1-RCT)
- J1 pad 8: CHASSIS_ETH -> /Ethernet/RX_N
- J1 pad 9: Net-(J1-Pad9) -> unconnected-(J1-NC-Pad9)
- J10 pad 10: unconnected-(J10-DET_A-Pad10) -> /MCU/SD2.DET
- J10 pad 3: /MCU/SD2.CMD -> Net-(J10-CMD)
- J12 pad 8: /MCU/SWO -> unconnected-(J12-Pin_8-Pad8)
- J14 pad 3: /MCU/SD1.CMD -> Net-(J14-CMD)
- J16 pad 1: unconnected-(J16-Pad1) -> /CAN FD/CAN_N
- J16 pad 6: unconnected-(J16-Pad6) -> /CAN FD/CAN_P
- J16 pad 8: unconnected-(J16-Pad8) -> CHASSIS_CAN
- L1 pad 1: 3V3 -> /Alimentation/3V3_SW
- L1 pad 2: 3V3A_Eth -> 3V3_Bat
- L3 pad 1: /Alimentation/3V3_SW -> /Alimentation/3V3_SW_USB
- L3 pad 2: 3V3 -> 3V3_USB
- R1 pad 1: /Ethernet/Eth.RXD1 -> 3V3
- R1 pad 2: Net-(U1-RXD1/MODE1) -> /Ethernet/Eth.RST
- R2 pad 1: /Ethernet/Eth.TXD0 -> Net-(U1-PG)
- R2 pad 2: /Ethernet/TXD_P -> 3V3_Bat
- R3 pad 1: /Ethernet/Eth.REFCLKO -> Net-(U1-FB)
- R3 pad 2: Net-(U1-~{INT}/REFCLKO) -> 3V3_Bat
- R4 pad 1: /Ethernet/Eth.TXD1 -> GND
- R4 pad 2: /Ethernet/TXD_N -> Net-(U1-FB)
- R45 pad 2: /MCU/SD1.CMD -> Net-(J14-CMD)
- R59 pad 2: 3V3 -> 3V3_USB
- R60 pad 2: 3V3 -> 3V3_USB
- R65 pad 2: 5V_USB -> 3V3_USB
- R72 pad 2: /Alimentation/LED1 -> /Monitor/LED1
- R74 pad 2: /Alimentation/LED2 -> /Monitor/LED2
- R75 pad 2: 5V_BAT -> 3V3
- R76 pad 2: /Alimentation/LED3 -> /Monitor/LED3
- R78 pad 2: 3V3 -> 12.8V
- R96 pad 2: /MCU/SD2.CMD -> Net-(J10-CMD)
- U1 pad 1: 3V3A_Eth -> /Alimentation/3V3_SW
- U1 pad 10: Net-(U1-RXER/PHYAD0) -> 12.8V
- U1 pad 11: Net-(U1-CRS_DV/MODE2) -> 12.8V
- U1 pad 12: /Ethernet/Eth.MDIO -> 12.8V
- U1 pad 13: /Ethernet/Eth.MDC -> 12.8V
- U1 pad 14: Net-(U1-~{INT}/REFCLKO) -> 3V3_Bat
- U1 pad 15: /Ethernet/Eth.RST -> GND
- U1 pad 16: Net-(U1-TXEN) -> GND
- U1 pad 17: /Ethernet/TXD_P -> GND
- U1 pad 2: /Ethernet/LED2 -> /Alimentation/3V3_SW
- U1 pad 3: /Ethernet/LED1 -> /Alimentation/3V3_SW
- U1 pad 4: unconnected-(U1-XTAL2-Pad4) -> Net-(U1-PG)
- U1 pad 5: /Ethernet/Eth_Clock_25Mhz -> Net-(U1-FB)
- U1 pad 6: Net-(U1-VDDCR) -> GND
- U1 pad 7: Net-(U1-RXD1/MODE1) -> GND
- U1 pad 8: Net-(U1-RXD0/MODE0) -> GND
- U1 pad 9: 3V3 -> Net-(U1-SS/TR)
- U2 pad 1: /Ethernet/Eth.RST -> unconnected-(U2-PE2-Pad1)
- U2 pad 146: /Alimentation/LED1 -> /MCU/LED1
- U2 pad 147: /Alimentation/LED2 -> /MCU/LED2
- U2 pad 148: /Alimentation/LED3 -> /MCU/LED3
- U2 pad 150: unconnected-(U2-PD7-Pad150) -> /MCU/SD2.CMD
- U2 pad 155: /Ethernet/Eth.TXEN -> unconnected-(U2-PG11-Pad155)
- U2 pad 170: /MCU/CAN.FAULT -> unconnected-(U2-PE0-Pad170)
- U2 pad 41: /MCU/SD2.CMD -> unconnected-(U2-PA0-Pad41)
- U2 pad 51: unconnected-(U2-PA6-Pad51) -> /Ethernet/Eth.RST
- U2 pad 53: /Ethernet/Eth.RXD0 -> /Ethernet/Eth.RXD_P
- U2 pad 54: /Ethernet/Eth.RXD1 -> /Ethernet/Eth.RXD_N
- U2 pad 79: unconnected-(U2-PB11-Pad79) -> Net-(U2-PB11)
- U2 pad 85: /Ethernet/Eth.TXD0 -> Net-(U2-PB12)
- U2 pad 86: /Ethernet/Eth.TXD1 -> Net-(U2-PB13)
- U3 pad 1: 12.8V -> unconnected-(U3-IN-3-Pad1)
- U3 pad 2: GND -> unconnected-(U3-IN+3-Pad2)
- U3 pad 3: 5V_BAT -> unconnected-(U3-GND-Pad3)
- U4 pad 1: /Alimentation/3V3_SW -> /Alimentation/3V3_SW_USB
- U4 pad 10: 5V -> 5V_USB
- U4 pad 11: 5V -> 5V_USB
- U4 pad 12: 5V -> 5V_USB
- U4 pad 13: 5V -> 5V_USB
- U4 pad 14: 3V3 -> 3V3_USB
- U4 pad 2: /Alimentation/3V3_SW -> /Alimentation/3V3_SW_USB
- U4 pad 3: /Alimentation/3V3_SW -> /Alimentation/3V3_SW_USB
- U6 pad 2: 5V -> 3V3
- U6 pad 3: 5V_USB -> 3V3_USB
- U6 pad 5: 5V_USB -> 3V3_USB
- U6 pad 6: 5V_BAT -> 3V3_Bat
- U6 pad 7: 5V -> 3V3
Routing:
- net GND: track 162.2 -> 50.3 mm, vias 124 -> 54
- net 3V3: track 114.8 -> 21.5 mm, vias 71 -> 16
- net /CAN FD/CAN.RXD: track 70.1 -> 1.84 mm
- net /Control/Heater3: track 68.0 -> 0.00 mm, vias 1 -> 0
- net /MCU/SD2.CMD: track 67.1 -> 1.71 mm, vias 4 -> 0
- net /Control/Servo.Signal3: track 69.9 -> 4.73 mm, vias 2 -> 0
- net /Control/E-match1: track 63.0 -> 0.49 mm, vias 2 -> 0
- net /Control/E-match2_Det: track 64.2 -> 2.77 mm, vias 2 -> 1
- net /Control/Heater2: track 59.8 -> 0.00 mm, vias 1 -> 0
- net /Control/E-match2: track 59.5 -> 0.00 mm
- net /Control/Servo.Signal2: track 60.6 -> 4.25 mm, vias 2 -> 0
- net Net-(J10-DAT3/CD): track 69.9 -> 14.1 mm, vias 3 -> 0
- net Net-(J14-SHIELD): track 54.9 -> 0.00 mm
- net /MCU/USBC.DP: track 53.8 -> 0.00 mm
- net Net-(J10-DAT2): track 68.5 -> 14.9 mm, vias 3 -> 2
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- added copper zone on F.Cu, net /Alimentation/3V3_SW_USB
- added copper zone on F.Cu, net 3V3_Bat
- added copper zone on F.Cu, net 3V3_USB
- added copper zone on B.Cu, net CHASSIS_CAN
- added copper zone on B.Cu, net CHASSIS_ETH
- removed copper zone on F.Cu, net 5V
- removed copper zone on F.Cu, net 5V_BAT
Other:
- board size 124 x 90 mm -> 100 x 100 mm
- board text added: "+"
- board text added: "-"
- board text added: "5-18V"
- board text added: "Pas de fil icite"
- board text added: "Stitch osc"
- board text removed: "3V3"
- board text removed: "5V"
- board text removed: "GND1"
- board text removed: "GND2"
