File: Fill_Station_ControlBoard/Fill_Station_ControlBoard.kicad_pcb (KiCad board)
At the start: 6 copper layers, 100 x 100 mm, 271 parts, among them IC1 TPS259573DSGR, J1 RJ45_Wuerth_74980111211, J10 Micro_SD_Card_Det_Hirose_DM3AT, J12 Conn_02x05_Counter_Clockwise, J13 Screw_Terminal_2_P5.00mm, J14 Micro_SD_Card_Det_Hirose_DM3AT, J15 USB_C_Receptacle_USB2.0_14P, J16 DE9_Socket_MountingHoles, J18 Screw_Terminal_3_P3.50mm, J2 Ematch1, J6 Ematch2, J7 Screw_Terminal_3_P3.50mm, J8 Screw_Terminal_3_P3.50mm, J9 Screw_Terminal_6_P3.50mm, Q1 AO3400A, Q2 AO3400A, SW1 RESET, SW2 BOOT, U1 INA3221, U10 TPSM33620-Q1, U11 TPSM33620-Q1, U12 TPSM33620-Q1, U2 STM32H747IITx, U5 DP83825I, U6 TPS2116DRL, U7 USBLC6-2SC6, U8 ISOW1044, U9 TPS2116DRL, Y1 ASV-25.000MHz, Y2 ASV-32.768kHz, Y4 ASV-25.000MHz

Commit message: PCB fini avant review avec greg
Parts:
- added J11: Screw_Terminal_2_P5.00mm, TerminalBlock_Phoenix:TerminalBlock_Phoenix_PT-1,5-2-5.0-H_1x02_P5.00mm_Horizontal, F.Cu at (226.1, 165.7)
- added J17: PINHD_1x6_Male, Connector_PinHeader_2.54mm:PinHeader_1x06_P2.54mm_Vertical, B.Cu at (219.3, 174.4)
- C1, C2: moved to B.Cu
- J18: value Screw_Terminal_3_P3.50mm -> PINHD_1x6_Male; footprint TerminalBlock_Phoenix:TerminalBlock_Phoenix_PT-1,5-3-3.5-H_1x03_P3.50mm_Horizontal -> Connector_PinHeader_2.54mm:PinHeader_1x06_P2.54mm_Vertical; moved to B.Cu
- J7, J8: value Screw_Terminal_3_P3.50mm -> Screw_Terminal_2_P5.00mm; footprint TerminalBlock_Phoenix:TerminalBlock_Phoenix_PT-1,5-3-3.5-H_1x03_P3.50mm_Horizontal -> TerminalBlock_Phoenix:TerminalBlock_Phoenix_PT-1,5-2-5.0-H_1x02_P5.00mm_Horizontal
- moved R10 39.6 mm to (244.1, 138.5)
- moved BZ1 24.2 mm to (238.7, 144.7), turned to 90 degrees
- moved R11 16.6 mm to (233.1, 144.8), turned to 90 degrees
- moved D1 14.8 mm to (213.2, 152.7), turned to -90 degrees
- moved R30 14.6 mm to (209.8, 153.7), turned to 0 degrees
- moved J18 10.8 mm to (214.5, 174.4), turned to 90 degrees
- moved R32 8.78 mm to (228.7, 157.8)
- moved R29 8.74 mm to (216.4, 157.5)
- moved R8 8.20 mm to (223.5, 147.3), turned to 0 degrees
- moved D2 8.10 mm to (219.2, 157.4)
- moved D3 7.63 mm to (231.6, 157.4)
- moved J8 5.71 mm to (203.9, 165.7)
- moved J7 5.54 mm to (215.0, 165.7)
- moved R4 2.09 mm to (231.6, 152.0)
- moved H2 0.83 mm to (176.0, 82.0)
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Connections:
- J18 pad 1: /Control/Servo1 -> GND
- J18 pad 2: GND -> 3V3
- J18 pad 3: /Control/Heater1 -> /MCU/SPI5.CS
- J9 pad 6: /Control/GPIO6 -> unconnected-(J9-Pad6)
- U2 pad 155: unconnected-(U2-PG11-Pad155) -> /MCU/SPI5.CS
- U2 pad 156: unconnected-(U2-PG12-Pad156) -> /MCU/SPI5.MISO
- U2 pad 157: unconnected-(U2-PG13-Pad157) -> /MCU/SPI5.SCK
- U2 pad 158: unconnected-(U2-PG14-Pad158) -> /MCU/SPI5.MOSI
- U2 pad 74: /Control/Heater3 -> /MCU/SPI4.SCK
- U2 pad 75: /Control/Heater2 -> /MCU/SPI4.MISO
- U2 pad 76: /Control/Heater1 -> /MCU/SPI4.MOSI
- U2 pad 77: unconnected-(U2-PE15-Pad77) -> /MCU/SPI4.CS
Routing:
- net 5V: track 161.4 -> 266.4 mm, vias 4 -> 3
- net /MCU/SPI5.MOSI: track 0.00 -> 74.2 mm, vias 0 -> 3
- net /MCU/SPI5.SCK: track 0.00 -> 72.7 mm, vias 0 -> 3
- net /MCU/SPI5.MISO: track 0.00 -> 72.5 mm, vias 0 -> 3
- net /MCU/SPI5.CS: track 0.00 -> 72.0 mm, vias 0 -> 3
- net 3V3: track 201.1 -> 149.5 mm, vias 74 -> 75
- net /Control/Heater3: track 46.2 -> 0.00 mm, vias 1 -> 0
- net /MCU/SPI4.CS: track 0.00 -> 41.3 mm, vias 0 -> 1
- net /MCU/SPI4.SCK: track 0.00 -> 41.1 mm, vias 0 -> 1
- net /MCU/SPI4.MISO: track 0.00 -> 40.3 mm, vias 0 -> 1
- net /MCU/SPI4.MOSI: track 0.00 -> 39.6 mm, vias 0 -> 1
- net /Control/Heater2: track 39.5 -> 0.00 mm, vias 1 -> 0
- net /Control/Heater1: track 37.9 -> 0.00 mm, vias 1 -> 0
- net /Control/Servo.Signal3: track 52.1 -> 32.3 mm
- net /Control/Servo.Signal2: track 42.1 -> 30.2 mm
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- added copper zone on B.Cu, net GND
Other:
- board size 100 x 100 mm -> 101 x 102 mm
- board text added: "3V3"
- board text added: "CAN FD w/ term"
- board text added: "CS4"
- board text added: "CS5"
- board text added: "MI4"
- board text added: "MI5"
- board text added: "MO4"
- board text added: "MO5"
- board text added: "SCK4"
- board text added: "SCK5"
- board text added: "SD2"
- board text added: "Sig1"
- board text added: "Sig2"
- board text added: "Sig3"
- board text added: "switch?"
- board text removed: "CAN FD w/ termination"
- board text removed: "H"
- board text removed: "Sig"

Commit message: Final_V1
Parts:
- removed C106, C108, C111, C113: 10u, Capacitor_SMD:C_0603_1608Metric
- removed C109, C110, C114: 22u, Capacitor_SMD:C_0603_1608Metric
- removed C11: 47uF, Capacitor_SMD:CP_Elec_4x5.4
- added C3: 22u, Capacitor_SMD:C_1210_3225Metric, F.Cu at (258.3, 160.3)
- added C4: 22u, Capacitor_SMD:C_1210_3225Metric, F.Cu at (256.3, 136.0)
- added C5: 10u, Capacitor_SMD:C_0805_2012Metric, F.Cu at (260.9, 160.6)
- added C55: 10u, Capacitor_SMD:C_0805_2012Metric, F.Cu at (253.5, 132.7)
- added C56: 10u, Capacitor_SMD:C_0603_1608Metric, F.Cu at (268.8, 157.2)
- added C58: 10u, Capacitor_SMD:C_0603_1608Metric, F.Cu at (247.6, 132.3)
- added C61: 22u, Capacitor_SMD:C_0603_1608Metric, F.Cu at (267.2, 157.2)
- added C78: 22u, Capacitor_SMD:C_0603_1608Metric, F.Cu at (247.6, 133.7)
- added FID1: Fiducial, Fiducial:Fiducial_0.5mm_Mask1mm, F.Cu at (173.8, 87.0)
- added FID2: Fiducial, Fiducial:Fiducial_0.5mm_Mask1mm, F.Cu at (262.4, 80.1)
- added FID3: Fiducial, Fiducial:Fiducial_0.5mm_Mask1mm, F.Cu at (181.7, 175.9)
- added J19: ~, Connector_AMASS:AMASS_XT60-M_1x02_P7.20mm_Vertical, F.Cu at (240.1, 173.0)
- added Q3: AO3400A, Package_TO_SOT_SMD:SOT-23, B.Cu at (242.1, 141.8)
- added R12: 10k, Resistor_SMD:R_0402_1005Metric, F.Cu at (229.6, 97.7)
- C10: value 47uF -> 100uF_50V; footprint Capacitor_SMD:CP_Elec_4x5.4 -> Capacitor_SMD:CP_Elec_6.3x7.7
- C49, C52, C95: footprint Capacitor_SMD:C_0402_1005Metric -> Capacitor_SMD:C_0603_1608Metric
- C57: value 100uF_25V -> 100uF_50V; footprint Capacitor_THT:CP_Radial_D6.3mm_P2.50mm -> Capacitor_SMD:CP_Elec_6.3x7.7
- C59: value 10uF_25V -> 10uF_50V; footprint Capacitor_THT:CP_Radial_D5.0mm_P2.00mm -> Capacitor_SMD:CP_Elec_5x5.3
- C67: value 10nF -> 10n
- C70, C73: value 100nF -> 100n
- C71, C88: footprint Capacitor_SMD:C_0603_1608Metric -> Capacitor_SMD:C_0805_2012Metric
- C82: value 10u -> 100uF_50V; footprint Capacitor_SMD:C_0603_1608Metric -> Capacitor_SMD:CP_Elec_6.3x7.7
- C84, R5, R65, R75: footprint Capacitor_SMD:C_0603_1608Metric -> Resistor_SMD:R_0603_1608Metric
- C85: value 22u -> 10u
- C86, R45, R46, R47: moved to B.Cu
- D15: footprint Diode_SMD:D_0603_1608Metric -> Diode_SMD:D_SOD-123
- F2: footprint Fuse:Fuse_0603_1608Metric -> Fuse:Fuse_1206_3216Metric
- J13: value Screw_Terminal_2_P5.00mm -> PINHD_1x4_Male; footprint TerminalBlock_Phoenix:TerminalBlock_Phoenix_PT-1,5-2-5.0-H_1x02_P5.00mm_Horizontal -> Connector_PinHeader_2.54mm:PinHeader_1x04_P2.54mm_Vertical
- J14: value Micro_SD_Card_Det_Hirose_DM3AT -> Micro_SD_Card_Det_Hirose_DM3CS; footprint Connector_Card:microSD_HC_Hirose_DM3AT-SF-PEJM5 -> DM3CS-SF:HRS_DM3CS-SF
- L4, R111, R112, R53, R54: footprint Capacitor_SMD:C_0402_1005Metric -> Resistor_SMD:R_0402_1005Metric
- R1, R117, R118, R119, R120, R26, R28, R35, R37, R49, R50, R84, R87: footprint Resistor_SMD:R_0603_1608Metric_Pad0.98x0.95mm_HandSolder -> Resistor_SMD:R_0603_1608Metric
- R107: value 270 -> 680
- R25, R34, R51, R55, R56, R73, R79, R80, R86: footprint Resistor_SMD:R_0603_1608Metric_Pad0.98x0.95mm_HandSolder -> Resistor_SMD:R_0402_1005Metric
- R29, R30, R32: value 33 -> 22; footprint Capacitor_SMD:C_0603_1608Metric -> Resistor_SMD:R_0402_1005Metric
- R67: value R_US -> 365k
- R68: value R_US -> 32k
- R78: value R_US -> 10k
- R81, R82: footprint Capacitor_SMD:C_0603_1608Metric -> Resistor_SMD:R_0402_1005Metric
- moved J13 92.4 mm to (209.5, 81.3)
- moved D12 46.4 mm to (176.9, 125.2), turned to 0 degrees
- moved D14 46.3 mm to (176.9, 128.4), turned to 0 degrees
- moved D13 46.3 mm to (176.9, 126.8), turned to 0 degrees
- moved R72 41.8 mm to (180.1, 125.2), turned to 0 degrees
- moved R76 41.7 mm to (180.1, 128.4), turned to 0 degrees
- moved R74 41.7 mm to (180.1, 126.8), turned to 0 degrees
- moved C82 27.0 mm to (256.1, 116.5), turned to -90 degrees
- moved C85 15.5 mm to (269.3, 148.7)
- moved C60 14.3 mm to (256.0, 143.4), turned to 90 degrees
- moved C10 13.8 mm to (257.0, 102.3), turned to 0 degrees
- moved C6 11.4 mm to (267.6, 148.6), turned to -90 degrees
- moved C15 11.1 mm to (257.5, 144.3), turned to 90 degrees
- moved C59 8.77 mm to (248.7, 164.7)
- moved R47 7.58 mm to (241.1, 105.0), turned to 45 degrees
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Connections:
- C15 pad 1: 5V -> 3V3
- C6 pad 1: 3V3 -> 5V
- C60 pad 1: 5V -> 3V3
- C82 pad 1: 3V3 -> 12.8V
- C85 pad 1: 12.8V -> 5V
- J12 pad 4: unconnected-(J12-Pin_4-Pad4) -> /MCU/IO
- J13 pad 1: GND -> 3V3
- J13 pad 2: VIN -> /MCU/I2C1.SCL
- J14 pad 9: GND -> /MCU/SD.DET
- R10 pad 1: /Control/BUZZ -> Net-(Q3-G)
- R10 pad 2: Net-(Q3-B) -> /Control/BUZZ
- U2 pad 144: unconnected-(U2-PD1-Pad144) -> /MCU/IO
- U2 pad 164: /Alimentation/LED1 -> unconnected-(U2-PB5-Pad164)
- U2 pad 165: /Alimentation/LED2 -> /MCU/I2C1.SCL
- U2 pad 166: /Alimentation/LED3 -> /MCU/I2C1.SDA
- U2 pad 19: unconnected-(U2-PF1-Pad19) -> /Alimentation/LED1
- U2 pad 20: unconnected-(U2-PF2-Pad20) -> /Alimentation/LED2
- U2 pad 21: unconnected-(U2-PF3-Pad21) -> /Alimentation/LED3
- U2 pad 91: unconnected-(U2-PD10-Pad91) -> /Control/BUZZ
Routing:
- net Net-(J14-SHIELD): track 44.9 -> 0.00 mm
- net /MCU/IO: track 0.00 -> 44.0 mm, vias 0 -> 1
- net /MCU/I2C1.SCL: track 0.00 -> 33.7 mm, vias 0 -> 1
- net /MCU/I2C1.SDA: track 0.00 -> 31.1 mm, vias 0 -> 1
- net GND: track 249.1 -> 276.9 mm, vias 170 -> 190
- net /Alimentation/LED1: track 18.4 -> 35.7 mm
- net /Alimentation/LED2: track 18.6 -> 35.5 mm
- net /Alimentation/LED3: track 19.2 -> 35.2 mm
- net 3V3: track 149.5 -> 160.9 mm, vias 75 -> 81
- net /Control/BUZZ: track 0.00 -> 11.0 mm
- net VIN: track 0.00 -> 8.60 mm
- net 12.8V: track 66.5 -> 73.4 mm, vias 21 -> 20
- net Net-(J14-DAT1): track 21.6 -> 27.0 mm
- net Net-(J14-DAT0): track 23.9 -> 28.0 mm
- net Net-(Q3-D): track 7.08 -> 10.8 mm, vias 0 -> 1
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- removed copper zone on In3.Cu, net GND
Other:
- board size 101 x 102 mm -> 101 x 100 mm
- board text added: "Ethernet"
- board text added: "MATIS POULIN FILL CONTROL UNIT REV 1 MARS 2026"
- board text removed: "Stitch osc"
- board text removed: "switch?"
