File: Fill_Station_ControlBoard/MCU.kicad_sch (KiCad schematic)
At the start: 64 parts, among them J12 Conn_02x05_Counter_Clockwise, SW1 RESET, SW2 BOOT, U2 STM32H747IITx, Y1 ASV-25.000MHz, Y2 ASV-32.768kHz

Commit message: finalisé le pcb
Connections:
- net 3V3: now also C24.1, U2.135 (VDDLDO), U2.175 (VDDLDO), U2.82 (VDDLDO)
Changed lines of the file:
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@@
 	)
 	(junction
+		(at 246.38 40.64)
+		(diameter 0)
+		(color 0 0 0 0)
+	)
+	(junction
 		(at 398.78 39.37)
 		(diameter 0)
@@
 	(wire
 		(pts
+			(xy 246.38 40.64) (xy 252.73 40.64)
+		)
+		(stroke
+			(width 0)
+			(type default)
+		)
+	)
+	(wire
+		(pts
 			(xy 276.86 48.26) (xy 284.48 48.26)
 		)
@@
 	(wire
 		(pts
-			(xy 220.98 40.64) (xy 252.73 40.64)
+			(xy 220.98 40.64) (xy 246.38 40.64)
 		)
 		(stroke
@@
 		)
 	)
+	(wire
+		(pts
+			(xy 246.38 38.1) (xy 246.38 40.64)
+		)
+		(stroke
+			(width 0)
+			(type default)
+		)
+	)
 	(label "SWDIO"
 		(at 238.76 87.63 0)
@@
 					(unit 1)
 				)
+			)
+		)
+	)
+	(symbol
+		(lib_id "power:+3.3V")
+		(at 246.38 38.1 0)
+		(unit 1)
+		(exclude_from_sim no)
+		(in_bom yes)
+		(on_board yes)
+		(dnp no)
+		(property "Reference" "#PWR08"
+			(at 246.38 41.91 0)
+			(effects
+				(font
+					(size 1.27 1.27)
+				)
+				(hide yes)
+			)
+		)
+		(property "Value" "3V3"
+			(at 244.602 34.544 0)
+			(effects
+				(font
+					(size 1.27 1.27)
+				)
+				(justify left)
+			)
+		)
+		(property "Footprint" ""
+			(at 246.38 38.1 0)
+			(effects
+				(font
+					(size 1.27 1.27)
+				)
+				(hide yes)
+			)
+		)
+		(property "Datasheet" ""
+			(at 246.38 38.1 0)
+			(effects
+				(font
+					(size 1.27 1.27)
+				)
+				(hide yes)
+			)
+		)
+		(property "Description" "Power symbol creates a global label with name \"+3.3V\""
+			(at 246.38 38.1 0)
+			(effects
+				(font
+					(size 1.27 1.27)
+				)
+				(hide yes)
+			)
+		)
+		(pin "1"
+		)
+		(instances
+			(project "Fill_Station_ControlBoard"
+				(path "/eaacffe0-ee57-428e-a37e-5655e0922ccc/e0f29092-a5b7-4c06-8bb6-3f29401186b8"
+					(reference "#PWR08")
+					(unit 1)
+				)
