File: Fill_Station_ControlBoard/MCU.kicad_sch (KiCad schematic)
At the start: 64 parts, among them J12 Conn_02x05_Counter_Clockwise, SW1 RESET, SW2 BOOT, U2 STM32H747IITx, Y1 ASV-25.000MHz, Y2 ASV-32.768kHz

Commit message: PCB fini avant review avec greg
Connections:
- net SPI5.CS: now reaches U2.155 (PG11)
- net SPI5.MISO: now reaches U2.156 (PG12)
- net SPI5.SCK: now reaches U2.157 (PG13)
- net SPI5.MOSI: now reaches U2.158 (PG14)
- net SPI4.CS: now reaches U2.77 (PE15)
- net Heater1 renamed SPI4.MOSI
- net Heater2 renamed SPI4.MISO
- net Heater3 renamed SPI4.SCK
- no-connect marks 65 -> 57
Changed lines of the file:
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@@
-	)
-	(no_connect
-		(at 142.24 135.89)
 	)
 	(no_connect
@@
 	)
 	(no_connect
-		(at 142.24 224.79)
-	)
-	(no_connect
 		(at 142.24 123.19)
 	)
@@
 	)
 	(no_connect
-		(at 142.24 130.81)
-	)
-	(no_connect
 		(at 205.74 44.45)
 	)
@@
 	)
 	(no_connect
-		(at 142.24 133.35)
-	)
-	(no_connect
 		(at 142.24 153.67)
 	)
@@
 	)
 	(no_connect
-		(at 142.24 161.29)
-	)
-	(no_connect
-		(at 142.24 163.83)
-	)
-	(no_connect
 		(at 142.24 118.11)
 	)
@@
 	)
 	(no_connect
-		(at 142.24 128.27)
-	)
-	(no_connect
 		(at 142.24 189.23)
 	)
@@
 	(no_connect
 		(at 142.24 168.91)
-	)
-	(no_connect
-		(at 142.24 166.37)
 	)
 	(wire
@@
 		)
 	)
+	(hierarchical_label "SPI5.SCK"
+		(shape output)
+		(at 142.24 133.35 180)
+		(effects
+			(font
+				(size 1.27 1.27)
+			)
+			(justify right)
+		)
+	)
 	(hierarchical_label "SD1.DAT1"
 		(shape output)
@@
 			)
 			(justify left)
+		)
+	)
+	(hierarchical_label "SPI4.MISO"
+		(shape input)
+		(at 142.24 219.71 180)
+		(effects
+			(font
+				(size 1.27 1.27)
+			)
+			(justify right)
 		)
 	)
@@
 		)
 	)
+	(hierarchical_label "SPI5.MOSI"
+		(shape output)
+		(at 142.24 135.89 180)
+		(effects
+			(font
+				(size 1.27 1.27)
+			)
+			(justify right)
+		)
+	)
+	(hierarchical_label "SPI4.CS"
+		(shape output)
+		(at 142.24 224.79 180)
+		(effects
+			(font
+				(size 1.27 1.27)
+			)
+			(justify right)
+		)
+	)
 	(hierarchical_label "LED3"
 		(shape output)
@@
 		)
 	)
+	(hierarchical_label "SPI4.SCK"
+		(shape output)
+		(at 142.24 217.17 180)
+		(effects
+			(font
+				(size 1.27 1.27)
+			)
+			(justify right)
+		)
+	)
 	(hierarchical_label "SD1.DAT3"
 		(shape output)
@@
 		)
 	)
-	(hierarchical_label "Heater1"
-		(shape output)
-		(at 142.24 222.25 180)
-		(effects
-			(font
-				(size 1.27 1.27)
-			)
-			(justify right)
-		)
-	)
 	(hierarchical_label "Eth.RXD_P"
 		(shape input)
@@
 		)
 	)
-	(hierarchical_label "Heater3"
-		(shape output)
-		(at 142.24 217.17 180)
-		(effects
-			(font
-				(size 1.27 1.27)
-			)
-			(justify right)
-		)
-	)
 	(hierarchical_label "GPIO3"
 		(shape input)
@@
 		)
 	)
+	(hierarchical_label "SPI5.MISO"
+		(shape input)
+		(at 142.24 130.81 180)
+		(effects
+			(font
+				(size 1.27 1.27)
+			)
+			(justify right)
+		)
+	)
 	(hierarchical_label "Eth.MDC"
 		(shape output)
@@
 		)
 	)
+	(hierarchical_label "SPI5.CS"
+		(shape output)
+		(at 142.24 128.27 180)
+		(effects
+			(font
+				(size 1.27 1.27)
+			)
+			(justify right)
+		)
+	)
 	(hierarchical_label "LED1"
 		(shape output)
@@
 		)
 	)
-	(hierarchical_label "Heater2"
-		(shape output)
-		(at 142.24 219.71 180)
-		(effects
-			(font
+	(hierarchical_label "SPI4.MOSI"
+		(shape output)
+		(at 142.24 222.25 180)
+		(effects
+			(font

Commit message: Final_V1
Parts:
- added FID1, FID2, FID3: Fiducial, Fiducial:Fiducial_0.5mm_Mask1mm, symbol Mechanical:Fiducial
- BT1: LCSC (none) -> C910763
- C16, C23, C25, C26, C27, C28, C29, C30, C31, C33, C34, C35, C36, C37, C39, C40, C41, C42, C43, C44, C46, C48, C83, C90, C91: LCSC (none) -> C60474
- C20: LCSC (none) -> C14663
- C22, C45, C47, C50, C53: LCSC (none) -> C59302
- C24, C54: LCSC (none) -> C108342
- C49, C52: footprint Capacitor_SMD:C_0402_1005Metric -> Capacitor_SMD:C_0603_1608Metric; LCSC (none) -> C22399626
- C51: now left out of the parts list
- C87: LCSC (none) -> C22399626
- C88: footprint Capacitor_SMD:C_0603_1608Metric -> Capacitor_SMD:C_0805_2012Metric; LCSC (none) -> C141660
- L2: LCSC (none) -> C160977
- R103, R113, R114, R89: LCSC (none) -> C25092
- R49, R50: footprint Resistor_SMD:R_0603_1608Metric_Pad0.98x0.95mm_HandSolder -> Resistor_SMD:R_0603_1608Metric
- R51: footprint Resistor_SMD:R_0603_1608Metric_Pad0.98x0.95mm_HandSolder -> Resistor_SMD:R_0402_1005Metric; LCSC (none) -> C173683
- R52: LCSC (none) -> C173683
- R53: footprint Capacitor_SMD:C_0402_1005Metric -> Resistor_SMD:R_0402_1005Metric; LCSC (none) -> C173683
- R54: footprint Capacitor_SMD:C_0402_1005Metric -> Resistor_SMD:R_0402_1005Metric; LCSC (none) -> C17168
- SW1, SW2: LCSC (none) -> C221666
- U2: LCSC (none) -> C730199
- Y1: LCSC (none) -> C1987509
- Y2: LCSC (none) -> C17591433
Connections:
- net LED1: now also U2.19 (PF1); no longer U2.164 (PB5)
- net LED2: now also U2.20 (PF2); no longer U2.165 (PB6)
- net LED3: now also U2.21 (PF3); no longer U2.166 (PB7)
- net IO: now reaches J12.4 (Pin_4)
- net IO: now also U2.144 (PD1)
- net Buzz: now reaches U2.91 (PD10)
- new net I2C1.SCL: U2.165 (PB6)
- new net I2C1.SDA: U2.166 (PB7)
- no-connect marks 57 -> 55
