File: Fill_Station_ControlBoard/untitled.kicad_sch (KiCad schematic)
At the start: 3 parts, among them J7 Conn_01x04

Commit message: Assignation footprint pis valeurs resistances del
Parts:
- R1, R20: footprint (none) -> Capacitor_SMD:C_0603_1608Metric
Changed lines of the file:
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@@
 			)
 		)
-		(property "Footprint" ""
+		(property "Footprint" "Capacitor_SMD:C_0603_1608Metric"
 			(at 60.706 59.436 90)
 			(effects
@@
 			)
 		)
-		(property "Footprint" ""
+		(property "Footprint" "Capacitor_SMD:C_0603_1608Metric"
 			(at 61.214 52.324 90)
 			(effects

Commit message: arthur
Parts:
- added C21, C22, C48, C49, C52, C53: CAP_0.47uF_50V_0603, Capacitor_SMD:C_0603_1608Metric_Pad1.08x0.95mm_HandSolder, symbol 0CSL_D1_V1:CAP_0.47uF_50V_0603
- added D7, D8, D9: BAV99, Package_TO_SOT_SMD:SOT-23, symbol Diode:BAV99
- added F1, F2, F4: Fuse, Fuse:Fuse_1206_3216Metric_Pad1.42x1.75mm_HandSolder, symbol Device:Fuse
- added J19: SERVO1, Connector_PinSocket_2.54mm:PinSocket_1x03_P2.54mm_Horizontal, symbol 0CSL_D1_V1:CON-SIP-3P
- added J20: SERVO2, Connector_PinSocket_2.54mm:PinSocket_1x03_P2.54mm_Horizontal, symbol 0CSL_D1_V1:CON-SIP-3P
- added J21: SERVO3, Connector_PinSocket_2.54mm:PinSocket_1x03_P2.54mm_Horizontal, symbol 0CSL_D1_V1:CON-SIP-3P
- added J5, J9: Conn_01x04, symbol Connector_Generic:Conn_01x04
- added R10, R11, R12, R9: 33, Capacitor_SMD:C_0603_1608Metric, symbol Device:R_US
- added R35, R36, R37: 10k, Resistor_SMD:R_0603_1608Metric_Pad0.98x0.95mm_HandSolder, symbol 0CSL_D1_V1:RES0603
Connections:
- net GND: now also C21.2, C22.2, C48.2, C49.2, C52.2, C53.2, D7.1 (K), D8.1 (K), D9.1 (K), J19.1 (Pin_1), J20.1 (Pin_1), J21.1 (Pin_1), J5.2 (Pin_2), J5.4 (Pin_4), J9.2 (Pin_2), J9.4 (Pin_4), R35.2, R36.2, R37.2
- net Servo.Signal1 renamed Servo.Signal1_2
- net Servo.Signal2 renamed Servo.Signal2_2
- new net: J5.1 (Pin_1), R9.2
- new net: J5.3 (Pin_3), R10.1
- new net: C21.1, C49.1, F2.2, J19.2 (Pin_2)
- new net: C22.1, C52.1, F4.2, J21.2 (Pin_2)
- new net: J9.3 (Pin_3), R12.1
- new net: J9.1 (Pin_1), R11.2
- new net: C48.1, C53.1, F1.2, J20.2 (Pin_2)
- new net +3V3: D7.2 (A), D8.2 (A), D9.2 (A)
- new net DATA_S1: D7.3 (K), J19.3 (Pin_3), R35.1
- new net DATA_S2: D9.3 (K), J20.3 (Pin_3), R36.1
- new net DATA_S3: D8.3 (K), J21.3 (Pin_3), R37.1
- new net Servo.Signal1_1: R9.1
- new net Servo.Signal1_ex: R11.1
- new net Servo.Signal2_1: R10.2
- new net Servo.Signal2_ex: R12.2
- new net Vdrive: F1.1, F2.1, F4.1

Commit message: Modifs de l'organisation des pages
Parts:
- removed C21, C22, C48, C49, C52, C53: CAP_0.47uF_50V_0603, Capacitor_SMD:C_0603_1608Metric_Pad1.08x0.95mm_HandSolder, symbol 0CSL_D1_V1:CAP_0.47uF_50V_0603
- removed D7, D8, D9: BAV99, Package_TO_SOT_SMD:SOT-23, symbol Diode:BAV99
- removed F1, F2, F4: Fuse, Fuse:Fuse_1206_3216Metric_Pad1.42x1.75mm_HandSolder, symbol Device:Fuse
- removed J19: SERVO1, Connector_PinSocket_2.54mm:PinSocket_1x03_P2.54mm_Horizontal, symbol 0CSL_D1_V1:CON-SIP-3P
- removed J20: SERVO2, Connector_PinSocket_2.54mm:PinSocket_1x03_P2.54mm_Horizontal, symbol 0CSL_D1_V1:CON-SIP-3P
- removed J21: SERVO3, Connector_PinSocket_2.54mm:PinSocket_1x03_P2.54mm_Horizontal, symbol 0CSL_D1_V1:CON-SIP-3P
- removed J5, J7, J9: Conn_01x04, symbol Connector_Generic:Conn_01x04
- removed R10, R11, R12: 33, Capacitor_SMD:C_0603_1608Metric, symbol Device:R_US
- removed R35, R36, R37: 10k, Resistor_SMD:R_0603_1608Metric_Pad0.98x0.95mm_HandSolder, symbol 0CSL_D1_V1:RES0603
- added D10, D11, D12: BAV99, Package_TO_SOT_SMD:SOT-23, symbol Diode:BAV99
- added J1: Conn_01x06, symbol Connector_Generic:Conn_01x06
- added J5, J7, J9: 436500200, symbol MOLEX:436500200
Connections:
- net +3V3: now also D10.2 (A), D11.2 (A), D12.2 (A)
- net GND: now also D10.1 (K), D11.1 (K), D12.1 (K), J5.2, J7.2, J9.2
- net Servo.Signal3: now reaches R9.2
- net Servo.Signal3: now also D12.3 (K)
- net at R1.1: now also J7.1
- net at R20.2: now also J5.1
- net Servo.Signal1_1: no longer names the net of R9.1
- net Servo.Signal1_1: now also J9.1
- net Servo.Signal1_2 renamed Servo.Signal1
- net Servo.Signal1: now also D10.3 (K)
- net Servo.Signal2_2 renamed Servo.Signal2
- net Servo.Signal2: now also D11.3 (K)
- new net GPIO1: J1.1 (Pin_1)
- new net GPIO2: J1.2 (Pin_2)
- new net GPIO3: J1.3 (Pin_3)
- new net GPIO4: J1.4 (Pin_4)
- new net GPIO5: J1.5 (Pin_5)
- new net GPIO6: J1.6 (Pin_6)
Other:
- note added: "Heater"
- note removed: "Resistor TBD pour reduire le ringing"
- moved on the sheet: R1, R20

Commit message: Ajout power
Parts:
- J5, J7, J9: footprint (none) -> MOLEX:MOLEX_436500200
Connections:
- net +3V3 renamed 3V3
Changed lines of the file:
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@@
 			)
 		)
-		(property "Footprint" ""
+		(property "Footprint" "MOLEX:MOLEX_436500200"
 			(at 130.81 78.74 0)
 			(effects
@@
 			)
 		)
-		(property "Footprint" ""
+		(property "Footprint" "MOLEX:MOLEX_436500200"
 			(at 132.08 46.99 0)
 			(effects
@@
 			)
 		)
-		(property "Value" "+3V3"
+		(property "Value" "3V3"
 			(at 64.77 67.31 0)
 			(effects
@@
 			)
 		)
-		(property "Footprint" ""
+		(property "Footprint" "MOLEX:MOLEX_436500200"
 			(at 130.81 62.23 0)
 			(effects
@@
 			)
 		)
-		(property "Value" "+3V3"
+		(property "Value" "3V3"
 			(at 100.33 35.56 0)
 			(effects
@@
 			)
 		)
-		(property "Value" "+3V3"
+		(property "Value" "3V3"
 			(at 77.47 50.8 0)
 			(effects

Commit message: début layout
Parts:
- removed J1: Conn_01x06, symbol Connector_Generic:Conn_01x06
- added C10, C11: 47uF, Capacitor_SMD:CP_Elec_4x5.4, symbol Device:C_Polarized
- added D4, D5: LED, LED_SMD:LED_0603_1608Metric, symbol Device:LED
- added J10: Screw_Terminal_6_P5.00mm, TerminalBlock_Phoenix:TerminalBlock_Phoenix_PT-1,5-6-5.0-H_1x06_P5.00mm_Horizontal, symbol PCM_SL_Screw_Terminal:Screw_Terminal_6_P5.00mm
- added J2: Ematch1, TerminalBlock_Phoenix:TerminalBlock_Phoenix_PT-1,5-2-5.0-H_1x02_P5.00mm_Horizontal, symbol PCM_SL_Screw_Terminal:Screw_Terminal_2_P5.00mm
- added J6: Ematch2, TerminalBlock_Phoenix:TerminalBlock_Phoenix_PT-1,5-2-5.0-H_1x02_P5.00mm_Horizontal, symbol PCM_SL_Screw_Terminal:Screw_Terminal_2_P5.00mm
- added J7, J8, J9: Screw_Terminal_3_P5.00mm, TerminalBlock_Phoenix:TerminalBlock_Phoenix_PT-1,5-3-5.0-H_1x03_P5.00mm_Horizontal, symbol PCM_SL_Screw_Terminal:Screw_Terminal_3_P5.00mm
- added Q1, Q2: AO3400A, Package_TO_SOT_SMD:SOT-23, symbol Transistor_FET:AO3400A
- added R25, R34: 22, Resistor_SMD:R_0603_1608Metric_Pad0.98x0.95mm_HandSolder, symbol Device:R_US
- added R26, R28, R35, R37: 10k, Resistor_SMD:R_0603_1608Metric_Pad0.98x0.95mm_HandSolder, symbol Device:R_US
- added R27, R36: 50k, Resistor_SMD:R_0603_1608Metric_Pad0.98x0.95mm_HandSolder, symbol Device:R_US
- added R31, R33: *, Resistor_SMD:R_0603_1608Metric_Pad0.98x0.95mm_HandSolder, symbol Device:R_US
- renumbered D12 to D1, D11 to D2, D10 to D3, J7 to J3, J9 to J4, R1 to R29, R9 to R30, R20 to R32
Connections:
- net GND: now also C10.2, C11.2, D4.1 (K), D5.1 (K), J7.2, J8.2, J9.2, Q1.2 (S), Q2.2 (S), R26.2, R28.2, R35.2, R37.2
- net GPIO1: now also J10.1
- net GPIO2: now also J10.2
- net GPIO3: now also J10.3
- net GPIO4: now also J10.4
- net GPIO5: now also J10.5
- net GPIO6: now also J10.6
- net Servo3: now reaches J4.1, R30.1
- net Servo3: now also J9.1
- net Servo1: now reaches J5.1, R32.2
- net Servo1: now also J7.1
- net Servo2: now reaches J3.1, R29.1
- net Servo2: now also J8.1
- new net: D5.2 (A), R33.1
- new net: Q1.1 (G), R25.2, R26.1
- new net: J2.2, Q1.3 (D), R27.1
- new net: Q2.1 (G), R34.2, R35.1
- new net: J6.2, Q2.3 (D), R36.1
- new net: D4.2 (A), R31.1
- new net 12.8V: C10.1, C11.1, J2.1, J6.1
- new net E-match1: R25.1
- new net E-match1_Cont: R31.2
- new net E-match1_Det: R27.2, R28.1
- new net E-match2: R34.1
- new net E-match2_Cont: R33.2
- new net E-match2_Det: R36.2, R37.1
- new net Heater1: J7.3
- new net Heater2: J8.3
- new net Heater3: J9.3
Other:
- note added: "E-match"
- note added: "GPIO"
- note added: "Heater - Relay"
- note added: "Servo + Heater"
- note removed: "Heater"
- note removed: "Servo"
- moved on the sheet: D1, D2, D3, J3, J4, J5, R29, R30, R32

Commit message: PCB fait
Parts:
- removed J10: Screw_Terminal_6_P5.00mm, TerminalBlock_Phoenix:TerminalBlock_Phoenix_PT-1,5-6-5.0-H_1x06_P5.00mm_Horizontal, symbol PCM_SL_Screw_Terminal:Screw_Terminal_6_P5.00mm
- removed J7, J8, J9: Screw_Terminal_3_P5.00mm, TerminalBlock_Phoenix:TerminalBlock_Phoenix_PT-1,5-3-5.0-H_1x03_P5.00mm_Horizontal, symbol PCM_SL_Screw_Terminal:Screw_Terminal_3_P5.00mm
- added C80, C81: 1u, Capacitor_SMD:C_0603_1608Metric, symbol Device:C
- added J18, J7, J8: Screw_Terminal_3_P3.50mm, TerminalBlock_Phoenix:TerminalBlock_Phoenix_PT-1,5-3-3.5-H_1x03_P3.50mm_Horizontal, symbol PCM_SL_Screw_Terminal:Screw_Terminal_3_P3.50mm
- added J9: Screw_Terminal_6_P3.50mm, TerminalBlock_Phoenix:TerminalBlock_Phoenix_PT-1,5-6-3.5-H_1x06_P3.50mm_Horizontal, symbol PCM_SL_Screw_Terminal:Screw_Terminal_6_P3.50mm
- added R55, R56: 0, Resistor_SMD:R_0603_1608Metric_Pad0.98x0.95mm_HandSolder, symbol Device:R_US
- J3, J4, J5: now not fitted; now left out of the parts list
- R31, R33: value * -> 680
Connections:
- net 12.8V: now also C80.1, C81.1
- net GND: now also C80.2, C81.2, J18.2, J7.2, J8.2
- net GPIO1: now also J9.1
- net GPIO2: now also J9.2
- net GPIO3: now also J9.3
- net GPIO4: now also J9.4
- net GPIO5: now also J9.5
- net GPIO6: now also J9.6
- net Heater1: now also J18.3
- net Heater2: now also J7.3
- net Heater3: now also J8.3
- net Servo1: now also J18.1
- net Servo2: now also J7.1
- net Servo3: now also J8.1
- net at Q1.3 (D), R27.1: now also R55.2; no longer J2.2
- net at Q2.3 (D), R36.1: now also R56.2; no longer J6.2
- new net: J6.2, R56.1
- new net: J2.2, R55.1
Other:
- moved on the sheet: C10, C11, J2, J6

Commit message: Travail Layout
Other:
- note added: "Buzzer"
- note added: "I2C"
- note added: "maybe increase"
Changed lines of the file:
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@@
+		)
+	)
+	(text "Buzzer\n"
+		(exclude_from_sim no)
+		(at 207.264 145.288 0)
+		(effects
+			(font
+				(size 1.27 1.27)
+			)
 		)
 	)
@@
 			)
 			(justify left)
+		)
+	)
+	(text "I2C\n"
+		(exclude_from_sim no)
+		(at 191.516 139.192 0)
+		(effects
+			(font
+				(size 1.27 1.27)
+			)
 		)
 	)
@@
 		)
 	)
+	(text "maybe increase\n"
+		(exclude_from_sim no)
+		(at 52.07 130.81 0)
+		(effects
+			(font
+				(size 1.27 1.27)
+			)
+		)
+	)

Commit message: finalisé le pcb
Parts:
- added BZ1: Buzzer_TDK_PS1240, Buzzer_Beeper:Buzzer_Murata_PKMCS0909E, symbol 0CSL_D1_V1:Buzzer_TDK_PS1240
- added Q3: NPN, symbol Simulation_SPICE:NPN
- added R10, R11: 1k, Resistor_SMD:R_0603_1608Metric, symbol Device:R_US
Connections:
- net GND: now also Q3.3 (E)
- net GPIO6: no longer names the net of J9.6
- new net: BZ1.2, Q3.1 (C), R11.2
- new net: Q3.2 (B), R10.2
- new net BUZZ: R10.1
- new net VDD_3V3: BZ1.1, R11.1
- no-connect marks 0 -> 1
Other:
- note removed: "I2C"
