File: Fill_Station_ControlBoard/untitled.kicad_sch (KiCad schematic)
At the start: 39 parts, among them J18 Screw_Terminal_3_P3.50mm, J2 Ematch1, J3 436500200, J4 436500200, J5 436500200, J6 Ematch2, J7 Screw_Terminal_3_P3.50mm, J8 Screw_Terminal_3_P3.50mm, J9 Screw_Terminal_6_P3.50mm, Q1 AO3400A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

Commit message: PCB fini avant review avec greg
Parts:
- removed J18, J7, J8: Screw_Terminal_3_P3.50mm, TerminalBlock_Phoenix:TerminalBlock_Phoenix_PT-1,5-3-3.5-H_1x03_P3.50mm_Horizontal, symbol PCM_SL_Screw_Terminal:Screw_Terminal_3_P3.50mm
- added J11, J7, J8: Screw_Terminal_2_P5.00mm, TerminalBlock_Phoenix:TerminalBlock_Phoenix_PT-1,5-2-5.0-H_1x02_P5.00mm_Horizontal, symbol PCM_SL_Screw_Terminal:Screw_Terminal_2_P5.00mm
Connections:
- net GND: now also J11.2, J7.2, J8.2
- net Servo1: now also J11.1
- net Servo2: now also J7.1
- net Servo3: now also J8.1
Other:
- note removed: "Heater - Relay"
Changed lines of the file:
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@@
 	)
 	(rectangle
-		(start 188.468 72.39)
-		(end 260.35 92.71)
-		(stroke
-			(width 0)
-			(type default)
-		)
-		(fill
-			(type none)
-		)
-	)
-	(rectangle
 		(start 189.23 21.59)
 		(end 278.13 67.31)
@@
 		)
 	)
-	(text "Heater - Relay\n"
-		(exclude_from_sim no)
-		(at 191.77 78.74 0)
-		(effects
-			(font
-				(size 5 5)
-			)
-			(justify left)
-		)
-	)
 	(text "E-match"
 		(exclude_from_sim no)
@@
 	(wire
 		(pts
-			(xy 144.78 46.99) (xy 146.05 46.99)
-		)
-		(stroke
-			(width 0)
-			(type default)
-		)
-	)
-	(wire
-		(pts
 			(xy 81.28 43.18) (xy 87.63 43.18)
 		)
@@
 		)
 	)
-	(hierarchical_label "Heater3"
-		(shape input)
-		(at 146.05 77.47 180)
-		(effects
-			(font
-				(size 1.27 1.27)
-			)
-			(justify right)
-		)
-	)
 	(hierarchical_label "E-match1"
 		(shape input)
@@
 		)
 	)
-	(hierarchical_label "Heater2"
-		(shape input)
-		(at 146.05 62.23 180)
-		(effects
-			(font
-				(size 1.27 1.27)
-			)
-			(justify right)
-		)
-	)
 	(hierarchical_label "GPIO2"
 		(shape input)
@@
 		)
 	)
-	(hierarchical_label "Heater1"
-		(shape input)
-		(at 144.78 46.99 180)
-		(effects
-			(font
-				(size 1.27 1.27)
-			)
-			(justify right)
-		)
-	)
 	(hierarchical_label "E-match1_Det"
 		(shape output)
@@
 	)
 	(symbol
-		(lib_id "PCM_SL_Screw_Terminal:Screw_Terminal_3_P3.50mm")
-		(at 149.86 44.45 0)
-		(unit 1)
-		(exclude_from_sim no)
-		(in_bom yes)
-		(on_board yes)
-		(dnp no)
-		(fields_autoplaced yes)
-		(property "Reference" "J18"
-			(at 153.67 43.1799 0)
-			(effects
-				(font
-					(size 1.27 1.27)
-				)
-				(justify left)
-			)
-		)
-		(property "Value" "Screw_Terminal_3_P3.50mm"
-			(at 153.67 45.7199 0)
-			(effects
-				(font
-					(size 1.27 1.27)
-				)
-				(justify left)
-			)
-		)
-		(property "Footprint" "TerminalBlock_Phoenix:TerminalBlock_Phoenix_PT-1,5-3-3.5-H_1x03_P3.50mm_Horizontal"
-			(at 151.13 52.07 0)
-			(effects
-				(font
-					(size 1.27 1.27)
-				)
-				(hide yes)
-			)
-		)
-		(property "Datasheet" ""
-			(at 149.86 43.18 0)
-			(effects
-				(font
-					(size 1.27 1.27)
-				)
-				(hide yes)
-			)
-		)
-		(property "Description" ""
-			(at 149.86 44.45 0)
-			(effects
-				(font
-					(size 1.27 1.27)
-				)
-				(hide yes)
-			)
-		)
-		(pin "1"
-		)
-		(pin "2"
-		)
-		(pin "3"
-		)
-		(instances
-			(project ""
-				(path "/eaacffe0-ee57-428e-a37e-5655e0922ccc/2aa4b752-d5dd-41d5-96a2-06ece1279133"
-					(reference "J18")
-					(unit 1)
-				)
-			)
-		)
-	)
-	(symbol
 		(lib_id "MOLEX:436500200")
 		(at 106.68 74.93 0)
@@
 	)
 	(symbol
+		(lib_id "PCM_SL_Screw_Terminal:Screw_Terminal_2_P5.00mm")
+		(at 149.86 58.42 0)
+		(unit 1)
+		(exclude_from_sim no)
+		(in_bom yes)
+		(on_board yes)
+		(dnp no)
+		(fields_autoplaced yes)
+		(property "Reference" "J7"
+			(at 153.67 57.1499 0)
+			(effects
+				(font
+					(size 1.27 1.27)
+				)
+				(justify left)
+			)
+		)
+		(property "Value" "Screw_Terminal_2_P5.00mm"
+			(at 153.67 59.6899 0)
+			(effects
+				(font
+					(size 1.27 1.27)
+				)
+				(justify left)
+			)
+		)
+		(property "Footprint" "TerminalBlock_Phoenix:TerminalBlock_Phoenix_PT-1,5-2-5.0-H_1x02_P5.00mm_Horizontal"
+			(at 151.13 64.77 0)
+			(effects
+				(font
+					(size 1.27 1.27)
+				)
+				(hide yes)
+			)
+		)
+		(property "Datasheet" ""
+			(at 149.86 58.42 0)
+			(effects
+				(font
+					(size 1.27 1.27)
+				)
+				(hide yes)
+			)
+		)
+		(property "Description" ""
+			(at 149.86 58.42 0)
+			(effects
+				(font
+					(size 1.27 1.27)
+				)
+				(hide yes)
+			)
+		)
+		(pin "2"
+		)
+		(pin "1"
+		)
+		(instances
+			(project "Fill_Station_ControlBoard"
+				(path "/eaacffe0-ee57-428e-a37e-5655e0922ccc/2aa4b752-d5dd-41d5-96a2-06ece1279133"
+					(reference "J7")
+					(unit 1)
+				)
+			)
+		)
+	)
+	(symbol
 		(lib_id "Device:R_US")
 		(at 69.85 161.29 90)
@@
 	)
 	(symbol
+		(lib_id "PCM_SL_Screw_Terminal:Screw_Terminal_2_P5.00mm")
+		(at 149.86 73.66 0)
+		(unit 1)
+		(exclude_from_sim no)
+		(in_bom yes)
+		(on_board yes)
+		(dnp no)
+		(fields_autoplaced yes)
+		(property "Reference" "J8"
+			(at 153.67 72.3899 0)
+			(effects
+				(font
+					(size 1.27 1.27)
+				)
+				(justify left)
+			)
+		)
+		(property "Value" "Screw_Terminal_2_P5.00mm"
+			(at 153.67 74.9299 0)
+			(effects
+				(font
+					(size 1.27 1.27)
+				)
+				(justify left)
+			)
+		)
+		(property "Footprint" "TerminalBlock_Phoenix:TerminalBlock_Phoenix_PT-1,5-2-5.0-H_1x02_P5.00mm_Horizontal"
+			(at 151.13 80.01 0)
+			(effects
+				(font
+					(size 1.27 1.27)
+				)
+				(hide yes)
+			)
+		)
+		(property "Datasheet" ""
+			(at 149.86 73.66 0)
+			(effects
+				(font
+					(size 1.27 1.27)
+				)
+				(hide yes)
+			)
+		)
+		(property "Description" ""
+			(at 149.86 73.66 0)
+			(effects
+				(font
+					(size 1.27 1.27)
+				)
+				(hide yes)
+			)
+		)
+		(pin "2"
+		)
+		(pin "1"
+		)
+		(instances
+			(project "Fill_Station_ControlBoard"
+				(path "/eaacffe0-ee57-428e-a37e-5655e0922ccc/2aa4b752-d5dd-41d5-96a2-06ece1279133"
+					(reference "J8")
+					(unit 1)
+				)
+			)
+		)
+	)
+	(symbol
 		(lib_id "Device:LED")
 		(at 87.63 127 90)
@@
 	)
 	(symbol
-		(lib_id "PCM_SL_Screw_Terminal:Screw_Terminal_3_P3.50mm")
-		(at 149.86 74.93 0)
+		(lib_id "PCM_SL_Screw_Terminal:Screw_Terminal_2_P5.00mm")
+		(at 149.86 43.18 0)
 		(unit 1)
 		(exclude_from_sim no)
@@
 		(dnp no)
 		(fields_autoplaced yes)
-		(property "Reference" "J8"
-			(at 153.67 73.6599 0)
+		(property "Reference" "J11"
+			(at 153.67 41.9099 0)
 			(effects
 				(font
@@
 			)
 		)
-		(property "Value" "Screw_Terminal_3_P3.50mm"
-			(at 153.67 76.1999 0)
+		(property "Value" "Screw_Terminal_2_P5.00mm"
+			(at 153.67 44.4499 0)
 			(effects
 				(font
@@
 			)
 		)
-		(property "Footprint" "TerminalBlock_Phoenix:TerminalBlock_Phoenix_PT-1,5-3-3.5-H_1x03_P3.50mm_Horizontal"
-			(at 151.13 82.55 0)
+		(property "Footprint" "TerminalBlock_Phoenix:TerminalBlock_Phoenix_PT-1,5-2-5.0-H_1x02_P5.00mm_Horizontal"
+			(at 151.13 49.53 0)
 			(effects
 				(font
@@
 		)
 		(property "Datasheet" ""
-			(at 149.86 73.66 0)
+			(at 149.86 43.18 0)
 			(effects
 				(font
@@
 		)
 		(property "Description" ""
-			(at 149.86 74.93 0)
+			(at 149.86 43.18 0)
 			(effects
 				(font
@@
 			)
 		)
-		(pin "1"
-		)
 		(pin "2"
 		)
-		(pin "3"
+		(pin "1"
 		)
 		(instances
-			(project "Fill_Station_ControlBoard"
+			(project ""
 				(path "/eaacffe0-ee57-428e-a37e-5655e0922ccc/2aa4b752-d5dd-41d5-96a2-06ece1279133"
-					(reference "J8")
+					(reference "J11")
 					(unit 1)
 				)
@@
 					(unit 1)
 				)
-			)
-		)
-	)
-	(symbol
-		(lib_id "PCM_SL_Screw_Terminal:Screw_Terminal_3_P3.50mm")
-		(at 149.86 59.69 0)
-		(unit 1)
-		(exclude_from_sim no)
-		(in_bom yes)
-		(on_board yes)
-		(dnp no)
-		(fields_autoplaced yes)
-		(property "Reference" "J7"
-			(at 153.67 58.4199 0)
-			(effects
-				(font
-					(size 1.27 1.27)
-				)
-				(justify left)
-			)
-		)
-		(property "Value" "Screw_Terminal_3_P3.50mm"
-			(at 153.67 60.9599 0)
-			(effects
-				(font
-					(size 1.27 1.27)
-				)
-				(justify left)
-			)
-		)
-		(property "Footprint" "TerminalBlock_Phoenix:TerminalBlock_Phoenix_PT-1,5-3-3.5-H_1x03_P3.50mm_Horizontal"
-			(at 151.13 67.31 0)
-			(effects
-				(font
-					(size 1.27 1.27)
-				)
-				(hide yes)
-			)
-		)
-		(property "Datasheet" ""
-			(at 149.86 58.42 0)
-			(effects
-				(font
-					(size 1.27 1.27)
-				)
-				(hide yes)
-			)
-		)
-		(property "Description" ""
-			(at 149.86 59.69 0)
-			(effects
-				(font
-					(size 1.27 1.27)
-				)
-				(hide yes)
-			)
-		)
-		(pin "1"
-		)
-		(pin "2"
-		)
-		(pin "3"
-		)
-		(instances
-			(project "Fill_Station_ControlBoard"
-				(path "/eaacffe0-ee57-428e-a37e-5655e0922ccc/2aa4b752-d5dd-41d5-96a2-06ece1279133"
-					(reference "J7")
-					(unit 1)
-				)

Commit message: Final_V1
Parts:
- removed C10, C11: 47uF, Capacitor_SMD:CP_Elec_4x5.4, symbol Device:C_Polarized
- removed Q3: NPN, symbol Simulation_SPICE:NPN
- added C10, C82: 100uF_50V, Capacitor_SMD:CP_Elec_6.3x7.7, symbol PCM_SL_Capacitors:100uF_25V
- added Q3: AO3400A, Package_TO_SOT_SMD:SOT-23, symbol Transistor_FET:AO3400A
- BZ1: LCSC (none) -> C910763
- C80, C81: LCSC (none) -> C59302
- D1, D2, D3: LCSC (none) -> C68983
- D4, D5: LCSC (none) -> C2286
- Q1, Q2: LCSC (none) -> C20917
- R10, R11: LCSC (none) -> C22356624
- R25, R34: footprint Resistor_SMD:R_0603_1608Metric_Pad0.98x0.95mm_HandSolder -> Resistor_SMD:R_0402_1005Metric; LCSC (none) -> C25092
- R26, R28, R35, R37: footprint Resistor_SMD:R_0603_1608Metric_Pad0.98x0.95mm_HandSolder -> Resistor_SMD:R_0603_1608Metric; LCSC (none) -> C22369937
- R27, R36: LCSC (none) -> C861451
- R29, R30, R32: value 33 -> 22; footprint Capacitor_SMD:C_0603_1608Metric -> Resistor_SMD:R_0402_1005Metric; LCSC (none) -> C25092
- R31, R33: LCSC (none) -> C22356475
- R55, R56: footprint Resistor_SMD:R_0603_1608Metric_Pad0.98x0.95mm_HandSolder -> Resistor_SMD:R_0402_1005Metric; LCSC (none) -> C17168
Connections:
- net 12.8V: now also C10.1, C82.1
- net BUZZ: now also R10.2; no longer R10.1
- net GND: now also C10.2, C82.2, Q3.2 (S)
- net at BZ1.2, R11.2: now also Q3.3 (D)
- new net: Q3.1 (G), R10.1
Other:
- note added: "Servo"
- note removed: "Servo + Heater"
- note removed: "maybe increase"
- moved on the sheet: R10
