File: Fill_Station_ControlBoard/Alimentation.kicad_sch (KiCad schematic)
At the start: 6 parts

Commit message: Ajout power
Parts:
- added C52: 100uF_25V, Capacitor_THT:CP_Radial_D6.3mm_P2.50mm, symbol PCM_SL_Capacitors:100uF_25V
- added C53: 10uF_25V, Capacitor_THT:CP_Radial_D5.0mm_P2.00mm, symbol PCM_SL_Capacitors:10uF_25V
- added C58: 0.1u, symbol Device:C_Polarized_US
- added C59: COUT, symbol Device:C_Polarized_US
- added C60: CdV/dT, Capacitor_SMD:C_0603_1608Metric, symbol Device:C
- added C79, C80, C81, C82, C83, C84, C85: C, Capacitor_SMD:C_0603_1608Metric, symbol Device:C
- added D1, D6, D7, D8, D9: LED, LED_SMD:LED_0603_1608Metric, symbol Device:LED
- added D13: SMAJ15A, Diode_SMD:D_SMA, symbol Diode:SMAJ15A
- added F1: Fuse, symbol Device:Fuse
- added IC2: TPS259573DSGR, SON50P200X200X80-9N, symbol TPS259573DSGR:TPS259573DSGR
- added J10: Screw_Terminal_2_P5.00mm, TerminalBlock_Phoenix:TerminalBlock_Phoenix_PT-1,5-2-5.0-H_1x02_P5.00mm_Horizontal, symbol PCM_SL_Screw_Terminal:Screw_Terminal_2_P5.00mm
- added L3: 4.7u, symbol Device:L
- added R15, R16, R29: *, Resistor_SMD:R_0805_2012Metric, symbol Device:R_US
- added R34, R35, R40, R41, R45: *, Resistor_SMD:R_0603_1608Metric_Pad0.98x0.95mm_HandSolder, symbol Device:R_US
- added R49, R50, R51, R52, R67, R68, R89, R90: R_US, Resistor_SMD:R_0603_1608Metric, symbol Device:R_US
- added R69: 0, Resistor_SMD:R_0603_1608Metric_Pad0.98x0.95mm_HandSolder, symbol Device:R_US
- added U4: TPS2116DRL, Package_TO_SOT_SMD:SOT-583-8, symbol Power_Management:TPS2116DRL
- added U7: OKI-78SR-5_1.5-W36-C, Converter_DCDC:Converter_DCDC_Murata_OKI-78SR_Vertical, symbol Converter_DCDC:OKI-78SR-5_1.5-W36-C
- added U8: TPS55285, symbol SiriusLib:TPS55285
- R53: value 4.42k -> *
- R54: value 620 -> *
- R55: value 280 -> *
Connections:
- net 3V3: now also C83.1, U8.9 (VOUT)
- net GND: now also C52.2, C53.2, C58.2, C59.2, C60.2, C81.2, C82.2, C83.2, C84.2, C85.2, D1.1 (K), D13.2 (A2), D6.1 (K), D7.1 (K), D8.1 (K), D9.1 (K), IC2.8 (GND_1), IC2.9 (GND_2), J10.1, R16.1, R49.2, R52.2, R67.2, R89.2, U4.1 (GND), U7.2 (GND), U8.12 (AGND), U8.7 (PGND)
- net +5V renamed 5V
- net 5V: now also C81.1, R90.1, U4.2 (VOUT), U4.7 (VOUT), U8.5 (VIN)
- net 24V renamed 12.8V_BAT
- net 12.8V_BAT: now also C52.1, C53.1, C58.1, D13.1 (A1), F1.2, IC2.3 (IN_1), IC2.4 (IN_2), R51.1, R69.1
- new net: C84.1, R50.1, U8.11 (COMP)
- new net: F1.1, J10.2
- new net: C82.1, U8.13 (VCC)
- new net: D8.2 (A), R41.1
- new net: C85.1, R50.2
- new net: R15.1, R16.2, U4.4 (PR1)
- new net: D1.2 (A), R34.1
- new net: R49.1, U8.1 (MODE)
- new net: C80.2, U8.14 (BOOT2)
- new net: C79.2, U8.15 (BOOT1)
- new net: R89.1, R90.2, U8.4 (EN/UVLO)
- new net: C79.1, L3.1, U8.6 (SW1)
- new net: C80.1, L3.2, U8.8 (SW2)
- new net: C60.1, IC2.1 (DVDT)
- new net: IC2.2 (~{EN}/OVLO), R51.2, R52.1
- new net: IC2.7 (ILM), R67.1
- new net: D7.2 (A), R40.1
- new net: R29.1, U4.8 (ST)
- new net: D6.2 (A), R35.1
- new net: D9.2 (A), R45.1
- new net 12.8V: C59.1, IC2.5 (OUT), R69.2, U7.1 (IN)
- new net 5V_BAT: R15.2, R29.2, R34.2, U4.3 (VIN1), U7.3 (OUT)
- new net 5V_USB: R35.2, U4.6 (VIN2)
- new net EFUSE_FLT: IC2.6 (~{FLT}), R68.1
- new net LED1: R40.2
- new net LED2: R41.2
- new net LED3: R45.2
- new net TPS3V5_INT: U8.10 (FB/INT)
- new net TPS3V5_SCL: U8.2 (SCL)
- new net TPS3V5_SDA: U8.3 (SDA)
- new net VDD_3V3: R68.2
Other:
- note added: "12.8V -> 5V SWR"
- note added: "5V -> 3.3V SWR"
- note added: "5V Bus"
- note added: "Batt"
- note added: "Calcul des compos"
- note added: "EFuse"
- note added: "TPS55285"
- note removed: "DEL d'alim"
- moved on the sheet: D2, D4, D5, R53, R54, R55

Commit message: début layout
Parts:
- removed C79, C80, C81, C82, C84, C85: C, Capacitor_SMD:C_0603_1608Metric, symbol Device:C
- removed R49, R50, R89, R90: R_US, Resistor_SMD:R_0603_1608Metric, symbol Device:R_US
- removed U8: TPS55285, symbol SiriusLib:TPS55285
- added C55: 10u, Capacitor_SMD:C_0603_1608Metric, symbol Device:C
- added C56: 0.1u, Capacitor_SMD:C_0603_1608Metric, symbol Device:C
- added C58: 3.3n, Capacitor_SMD:C_0603_1608Metric, symbol Device:C
- added R59: 100k, Resistor_SMD:R_0805_2012Metric, symbol Device:R_US
- added R60, R61: *, Resistor_SMD:R_0805_2012Metric, symbol Device:R_US
- added U4: TPS62130, Package_DFN_QFN:VQFN-16-1EP_3x3mm_P0.5mm_EP1.68x1.68mm_ThermalVias, symbol Regulator_Switching:TPS62130
- C61: renamed from C83; value C -> 22u
- C65: renamed from C59; value COUT -> 100u
- F1: footprint (none) -> Fuse:Fuse_0603_1608Metric
- IC1: renamed from IC2; footprint SON50P200X200X80-9N -> Package_SON:WSON-8-1EP_2x2mm_P0.5mm_EP0.9x1.6mm_ThermalVias
- L3: value 4.7u -> 2.2u
- R65: renamed from R15; footprint Resistor_SMD:R_0805_2012Metric -> Capacitor_SMD:C_0603_1608Metric
- R66: renamed from R16; footprint Resistor_SMD:R_0805_2012Metric -> Capacitor_SMD:C_0603_1608Metric
- R75: renamed from R29; footprint Resistor_SMD:R_0805_2012Metric -> Capacitor_SMD:C_0603_1608Metric
- renumbered C52 to C57, C53 to C59, C58 to C63, C60 to C64, D6 to D10, D5 to D11, D7 to D12, D8 to D13, D9 to D14, D13 to D6, D2 to D7, D4 to D8, D1 to D9, J10 to J13, R53 to R63, R54 to R64, R51 to R67, R52 to R68, R34 to R69, R35 to R70, R55 to R71, R40 to R72, R69 to R73, R41 to R74, R45 to R76, R67 to R77, R68 to R78, U7 to U3, U4 to U6
Connections:
- net 3V3: now also L3.2, R59.2, R60.2, U4.14 (VOS)
- net 5V: now also C55.1, C56.1, U4.10 (VIN), U4.11 (VIN), U4.12 (VIN), U4.13 (EN)
- net 5V_BAT: now also U6.5 (MODE)
- net GND: now also R61.1, U4.15 (GND), U4.16 (GND), U4.17 (GND), U4.6 (GND), U4.7 (FSW), U4.8 (DEF)
- net at L3.1: now also U4.1 (SW), U4.2 (SW), U4.3 (SW)
- new net: C55.2, C56.2, C58.2
- new net: R59.1, U4.4 (PG)
- new net: R60.1, R61.2, U4.5 (FB)
- new net: C58.1, U4.9 (SS/TR)
Other:
- note added: "LED"
- note removed: "TPS55285"
- moved on the sheet: C57, C59, C61, C63, C64, C65, D10, D11, D12, D13, D14, D6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

Commit message: PCB fait
Parts:
- removed C63: 0.1u, symbol Device:C_Polarized_US
- removed C65: 100u, symbol Device:C_Polarized_US
- removed D6: SMAJ15A, Diode_SMD:D_SMA, symbol Diode:SMAJ15A
- added C32, C82: 10u, Capacitor_SMD:C_0603_1608Metric, symbol Device:C
- added C38, C60, C74: 100n, Capacitor_SMD:C_0603_1608Metric, symbol Device:C
- added C62, C75: 22u, Capacitor_SMD:C_0603_1608Metric, symbol Device:C
- added C76, C77, C79: 1u, Capacitor_SMD:C_0603_1608Metric, symbol Device:C
- added C78: 22u, Capacitor_SMD:C_0805_2012Metric, symbol Device:C
- added D16: SMAJ20A, Diode_SMD:D_SMA, symbol Diode:SMAJ20A
- added TP1, TP2, TP3, TP4, TP5, TP6: TestPoint, TestPoint:TestPoint_Pad_D2.0mm, symbol Connector:TestPoint
- C61: footprint Capacitor_SMD:C_0603_1608Metric -> Capacitor_SMD:C_0805_2012Metric
- C64: value CdV/dT -> 3.3n
- F1: value Fuse -> 4A; now not fitted
- L3: footprint (none) -> Inductor_SMD:L_Coilcraft_XAL4020-XXX
- R59: footprint Resistor_SMD:R_0805_2012Metric -> Resistor_SMD:R_0603_1608Metric
- R60: value * -> 100k; footprint Resistor_SMD:R_0805_2012Metric -> Resistor_SMD:R_0603_1608Metric
- R61: value * -> 316k; footprint Resistor_SMD:R_0805_2012Metric -> Resistor_SMD:R_0603_1608Metric
- R63: value * -> 4.7k; footprint Resistor_SMD:R_0805_2012Metric -> Capacitor_SMD:C_0603_1608Metric
- R64, R69, R70: value * -> 1.5k
- R65: value * -> 365k
- R66: value * -> 100k
- R71, R72, R74, R76: value * -> 680
- R75: value * -> 10k
- R77: value R_US -> 1k
Connections:
- net VDD_3V3 is gone; now on net 3V3: R78.2
- net 12.8V: now also C32.1, C60.1, C75.1, C79.1
- net 12.8V_BAT: now also C38.1, D16.1 (A1), TP1.1
- net 3V3: now also C78.1, TP3.1
- net 5V: now also C82.1, TP2.1
- net 5V_BAT: now also U6.6 (VIN2), C62.1, C74.1, C77.1; no longer R65.2, U6.3 (VIN1), U6.5 (MODE)
- net 5V_USB: now also R65.2, U6.3 (VIN1), U6.5 (MODE), C76.1; no longer U6.6 (VIN2)
- net GND: now also C55.2, C56.2, C58.2, C32.2, C38.2, C60.2, C62.2, C74.2, C75.2, C76.2, C77.2, C78.2, C79.2, C82.2, D16.2 (A2), TP4.1
- net 3V3_SW: now reaches L3.1, U4.1 (SW), U4.2 (SW), U4.3 (SW)
Other:
- note added: "Confirmer les resistors en fonction de la couleur des leds"
- note added: "I_lim : 1A"
- moved on the sheet: C57, C58, C59, C61, J13, L3, R60, R61

Commit message: Travail Layout
Parts:
- removed C60, C74: 100n, Capacitor_SMD:C_0603_1608Metric, symbol Device:C
- removed C62, C75: 22u, Capacitor_SMD:C_0603_1608Metric, symbol Device:C
- removed D10, D11, D12, D13, D14, D7, D8, D9: LED, LED_SMD:LED_0603_1608Metric, symbol Device:LED
- removed R63: 4.7k, Capacitor_SMD:C_0603_1608Metric, symbol Device:R_US
- removed R64, R69, R70: 1.5k, Resistor_SMD:R_0603_1608Metric_Pad0.98x0.95mm_HandSolder, symbol Device:R_US
- removed R71, R72, R74, R76: 680, Resistor_SMD:R_0603_1608Metric_Pad0.98x0.95mm_HandSolder, symbol Device:R_US
- removed TP1, TP2, TP3, TP4, TP5, TP6: TestPoint, TestPoint:TestPoint_Pad_D2.0mm, symbol Connector:TestPoint
- removed U3: OKI-78SR-5_1.5-W36-C, Converter_DCDC:Converter_DCDC_Murata_OKI-78SR_Vertical, symbol Converter_DCDC:OKI-78SR-5_1.5-W36-C
- added C1, C6: 10u, Capacitor_SMD:C_0603_1608Metric, symbol Device:C
- added C2: 0.1u, Capacitor_SMD:C_0603_1608Metric, symbol Device:C
- added C3: 3.3n, Capacitor_SMD:C_0603_1608Metric, symbol Device:C
- added C4, C5: 22u, Capacitor_SMD:C_0805_2012Metric, symbol Device:C
- added L1: 2.2u, Inductor_SMD:L_Coilcraft_XAL4020-XXX, symbol Device:L
- added R2, R3: 100k, Resistor_SMD:R_0603_1608Metric, symbol Device:R_US
- added R4: 316k, Resistor_SMD:R_0603_1608Metric, symbol Device:R_US
- added U1: TPS62130, Package_DFN_QFN:VQFN-16-1EP_3x3mm_P0.5mm_EP1.68x1.68mm_ThermalVias, symbol Regulator_Switching:TPS62130
Connections:
- net 12.8V: now also R78.2, C1.1, C2.1, U1.10 (VIN), U1.11 (VIN), U1.12 (VIN), U1.13 (EN)
- net 3V3: now also C82.1, R75.2, U6.2 (VOUT), U6.7 (VOUT), C6.1; no longer C61.1, C78.1, L3.2, R59.2, R60.2, R78.2, U4.14 (VOS)
- net 3V3_SW: now also L1.1, U1.1 (SW), U1.2 (SW), U1.3 (SW); no longer L3.1, U4.1 (SW), U4.2 (SW), U4.3 (SW)
- net 5V_USB: now also C55.1, C56.1, U4.10 (VIN), U4.11 (VIN), U4.12 (VIN), U4.13 (EN); no longer C76.1, R65.2, U6.3 (VIN1), U6.5 (MODE)
- net GND: now also C1.2, C2.2, C3.2, C4.2, C5.2, C6.2, R4.1, U1.15 (GND), U1.16 (GND), U1.17 (GND), U1.6 (GND), U1.7 (FSW), U1.8 (DEF)
- removed net 5V: C55.1, C56.1, C82.1, U4.10 (VIN), U4.11 (VIN), U4.12 (VIN), U4.13 (EN), U6.2 (VOUT), U6.7 (VOUT)
- net 5V_BAT renamed 3V3_Bat
- net 3V3_Bat: now also C4.1, C5.1, L1.2, R2.2, R3.2, U1.14 (VOS); no longer R75.2
- new net: C3.1, U1.9 (SS/TR)
- new net: R3.1, R4.2, U1.5 (FB)
- new net: R2.1, U1.4 (PG)
- new net 3V3_SW_USB: L3.1, U4.1 (SW), U4.2 (SW), U4.3 (SW)
- new net 3V3_USB: C61.1, C76.1, C78.1, L3.2, R59.2, R60.2, R65.2, U4.14 (VOS), U6.3 (VIN1), U6.5 (MODE)
Other:
- note added: "12.8V -> 3.3V SWR"
- note added: "5V USB -> 3.3V SWR"
- note removed: "12.8V -> 5V SWR"
- note removed: "5V -> 3.3V SWR"
- note removed: "Confirmer les resistors en fonction de la couleur des leds"
- note removed: "LED"
- moved on the sheet: C55, C56, C58, C61, C78, C82, L3, R59, R60, R61, U4

Commit message: PCB presque terminé
Modifs de l'alim
Parts:
- removed C3, C58: 3.3n, Capacitor_SMD:C_0603_1608Metric, symbol Device:C
- removed C4, C5, C61, C78: 22u, Capacitor_SMD:C_0805_2012Metric, symbol Device:C
- removed C55: 10u, Capacitor_SMD:C_0603_1608Metric, symbol Device:C
- removed C56: 0.1u, Capacitor_SMD:C_0603_1608Metric, symbol Device:C
- removed L1, L3: 2.2u, Inductor_SMD:L_Coilcraft_XAL4020-XXX, symbol Device:L
- removed R59, R60: 100k, Resistor_SMD:R_0603_1608Metric, symbol Device:R_US
- removed R61: 316k, Resistor_SMD:R_0603_1608Metric, symbol Device:R_US
- removed U1, U4: TPS62130, Package_DFN_QFN:VQFN-16-1EP_3x3mm_P0.5mm_EP1.68x1.68mm_ThermalVias, symbol Regulator_Switching:TPS62130
- added C106, C108, C111, C113, C15, C60, C71, C74: 10u, Capacitor_SMD:C_0603_1608Metric, symbol Device:C
- added C107, C112, C62, C8, C9: 1u, Capacitor_SMD:C_0603_1608Metric, symbol Device:C
- added C109, C110, C114, C75, C84, C85: 22u, Capacitor_SMD:C_0603_1608Metric, symbol Device:C
- added C115, C116, C117: 100n, Capacitor_SMD:C_0603_1608Metric, symbol Device:C
- added D10, D11, D12, D13, D14, D7, D8, D9: LED, LED_SMD:LED_0603_1608Metric, symbol Device:LED
- added R132, R133, R134, R8, R9: 10k, Resistor_SMD:R_0402_1005Metric, symbol Device:R_US
- added R162: 50m, Resistor_SMD:R_0603_1608Metric, symbol Device:R_US
- added R5: 365k, Capacitor_SMD:C_0603_1608Metric, symbol Device:R_US
- added R6: 100k, Capacitor_SMD:C_0603_1608Metric, symbol Device:R_US
- added R63: 4.7k, Capacitor_SMD:C_0603_1608Metric, symbol Device:R_US
- added R64, R69, R70: 1.5k, Resistor_SMD:R_0603_1608Metric_Pad0.98x0.95mm_HandSolder, symbol Device:R_US
- added R7: 10k, Capacitor_SMD:C_0603_1608Metric, symbol Device:R_US
- added R71, R72, R74, R76: 680, Resistor_SMD:R_0603_1608Metric_Pad0.98x0.95mm_HandSolder, symbol Device:R_US
- added TP1, TP2, TP3, TP4, TP5, TP6: TestPoint, TestPoint:TestPoint_Pad_D2.0mm, symbol Connector:TestPoint
- added U1: INA3221, Package_DFN_QFN:Texas_RGV0016A_VQFN-16-1EP_4x4mm_P0.65mm_EP2.1x2.1mm, symbol Power_Management:INA3221
- added U10, U11, U12: TPSM33620-Q1, TPSM365:RDN0011A-MFG, symbol matispoulin:TPSM336
- added U9: TPS2116DRL, Package_TO_SOT_SMD:SOT-583-8, symbol Power_Management:TPS2116DRL
- C1: value 10u -> 100n
- C2: value 0.1u -> 10u
- R2, R3: value 100k -> 50m; # (none) -> ERJ-3BWFR050V
- R4: value 316k -> 10k; footprint Resistor_SMD:R_0603_1608Metric -> Resistor_SMD:R_0402_1005Metric
Connections:
- net 12.8V: now also R3.2, C106.1, C116.1, C117.1, C71.1, C84.1, C85.1, R63.2, U1.11 (IN-1), U10.2 (EN), U10.3 (VIN), U11.2 (EN), U11.3 (VIN); no longer C1.1, C2.1, IC1.5 (OUT), R73.2
- net 12.8V_BAT: now also TP1.1
- net 3V3: now also C1.1, C2.2, R2.2, R4.1, R133.1, R134.1, R71.2, R8.1, R9.1, TP3.1, U1.1 (IN-3), U1.4 (VS); no longer U6.2 (VOUT), U6.7 (VOUT)
- net 3V3_Bat: now also C74.1, C75.1, U10.4 (VOUT), U10.9 (FB); no longer R2.2, R3.2
- net 3V3_USB: now also C113.1, C114.1, U12.4 (VOUT), U12.9 (FB)
- net 5V_USB: now also C110.1, C111.1, C115.1, C9.1, R5.2, R70.2, U12.2 (EN), U12.3 (VIN), U9.3 (VIN1), U9.5 (MODE)
- net GND: now also C2.1, C106.2, C107.2, C108.2, C109.2, C110.2, C111.2, C112.2, C113.2, C114.2, C115.2, C116.2, C117.2, C15.2, C60.2, C62.2, C71.2, C74.2, C75.2, C8.2, C84.2, C85.2, C9.2, D10.1 (K), D11.1 (K), D12.1 (K), D13.1 (K), D14.1 (K), D7.1 (K), D8.1 (K), D9.1 (K), R6.1, TP4.1, U1.17 (EP), U1.3 (GND), U1.5 (A0), U10.10 (GND), U10.11 (MODE/SYNC), U11.10 (GND), U11.11 (MODE/SYNC), U12.10 (GND), U12.11 (MODE/SYNC), U9.1 (GND); no longer C2.2, R4.1
- net PM_TC: now reaches R4.2
- net PM_TC: now also U1.13 (TC); no longer R3.1
- net Psense3_IN+: now reaches R2.1
- net Psense3_IN+: now also U6.2 (VOUT), U6.7 (VOUT), U1.2 (IN+3)
- new net: R5.1, R6.2, U9.4 (PR1)
- new net: C112.1, U12.8 (VCC)
- new net: D13.2 (A), R74.1
- new net: D11.2 (A), R71.1
- new net: D8.2 (A), R64.1
- new net: D9.2 (A), R69.1
- new net: R132.2, U1.10 (PV)
- new net: R132.1, U1.16 (VPU)
- new net: D7.2 (A), R63.1
- new net: C62.1, U10.8 (VCC)
- new net: D12.2 (A), R72.1
- new net: R7.1, U9.8 (ST)
- new net: D10.2 (A), R70.1
- new net: C107.1, U11.8 (VCC)
- new net: D14.2 (A), R76.1
- new net 5V: C15.1, C60.1, R162.2, R64.2, R7.2, TP2.1, U1.14 (IN-2)
- new net 5V_Bat: C108.1, C109.1, C8.1, R69.2, U11.4 (VOUT), U11.9 (FB), U9.6 (VIN2)
- new net LED1: R72.2
- new net LED2: R74.2
- new net LED3: R76.2
- new net PM_CRIT: R133.2, U1.9 (CRITICAL)
- new net PM_SCL: R9.2, U1.6 (SCL)
- new net PM_SDA: R8.2, U1.7 (SDA)
- new net PM_WARN: R134.2, U1.8 (WARNING)
- new net Psense1_IN+: IC1.5 (OUT), R3.1, R73.2, U1.12 (IN+1)
- new net Psense2_IN+: R162.1, U1.15 (IN+2), U9.2 (VOUT), U9.7 (VOUT)
- no-connect marks 0 -> 2
Other:
- note added: "12.8V -> 3.3V"
- note added: "12.8V -> 5V"
- note added: "3V3 Bus"
- note added: "5V USB -> 3.3V USB"
- note added: "Capacitor -25V -X7R"
- note added: "Confirmer les resistors en fonction de la couleur des leds"
- note added: "LED"
- note added: "Monitor"
- note removed: "12.8V -> 3.3V SWR"
- note removed: "5V USB -> 3.3V SWR"
- moved on the sheet: C32, C38, C57, C59, C6, C64, C76, C77, C79, C82, D16, F1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

Commit message: finalisé le pcb
Parts:
- removed TP5, TP6: TestPoint, TestPoint:TestPoint_Pad_D2.0mm, symbol Connector:TestPoint
- R6: footprint Capacitor_SMD:C_0603_1608Metric -> Resistor_SMD:R_0603_1608Metric
Connections:
- net 12.8V: now also TP1.1
- net 12.8V_BAT: no longer C57.1, C59.1, TP1.1
- net VIN: now reaches F1.1, J13.2
- net VIN: now also C57.1, C59.1
- no-connect marks 2 -> 0
Other:
- moved on the sheet: F1
Changed lines of the file:
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@@
 	(rectangle
 		(start 379.73 68.58)
-		(end 412.75 123.19)
+		(end 412.75 113.03)
 		(stroke
 			(width 0)
@@
 	)
 	(junction
+		(at 64.77 35.56)
+		(diameter 0)
+		(color 0 0 0 0)
+	)
+	(junction
 		(at 156.21 180.34)
 		(diameter 0)
@@
 		(color 0 0 0 0)
 	)
-	(no_connect
-		(at 398.78 120.65)
-	)
-	(no_connect
-		(at 398.78 113.03)
-	)
 	(wire
 		(pts
@@
 	(wire
 		(pts
+			(xy 64.77 30.48) (xy 64.77 35.56)
+		)
+		(stroke
+			(width 0)
+			(type default)
+		)
+	)
+	(wire
+		(pts
 			(xy 203.2 62.23) (xy 203.2 59.69)
 		)
@@
 	(wire
 		(pts
-			(xy 55.88 35.56) (xy 59.69 35.56)
-		)
-		(stroke
-			(width 0)
-			(type default)
-		)
-	)
-	(wire
-		(pts
 			(xy 41.91 232.41) (xy 53.34 232.41)
 		)
@@
 	(wire
 		(pts
+			(xy 88.9 35.56) (xy 92.71 35.56)
+		)
+		(stroke
+			(width 0)
+			(type default)
+		)
+	)
+	(wire
+		(pts
 			(xy 387.35 172.72) (xy 384.81 172.72)
 		)
@@
 	(wire
 		(pts
+			(xy 77.47 35.56) (xy 64.77 35.56)
+		)
+		(stroke
+			(width 0)
+			(type default)
+		)
+	)
+	(wire
+		(pts
 			(xy 358.14 201.93) (xy 358.14 199.39)
 		)
@@
 	(wire
 		(pts
-			(xy 36.83 35.56) (xy 48.26 35.56)
+			(xy 36.83 35.56) (xy 59.69 35.56)
 		)
 		(stroke
@@
 	(wire
 		(pts
+			(xy 64.77 35.56) (xy 59.69 35.56)
+		)
+		(stroke
+			(width 0)
+			(type default)
+		)
+	)
+	(wire
+		(pts
 			(xy 156.21 62.23) (xy 167.64 62.23)
 		)
@@
 	(wire
 		(pts
-			(xy 59.69 35.56) (xy 77.47 35.56)
-		)
-		(stroke
-			(width 0)
-			(type default)
-		)
-	)
-	(wire
-		(pts
 			(xy 207.01 21.59) (xy 224.79 21.59)
 		)
@@
 	(wire
 		(pts
-			(xy 77.47 35.56) (xy 92.71 35.56)
+			(xy 77.47 35.56) (xy 81.28 35.56)
 		)
 		(stroke
@@
 			)
 		)
-		(property "Footprint" "Capacitor_SMD:C_0603_1608Metric"
+		(property "Footprint" "Resistor_SMD:R_0603_1608Metric"
 			(at 165.354 143.256 90)
 			(effects
@@
 	(symbol
 		(lib_id "Device:Fuse")
-		(at 52.07 35.56 90)
+		(at 85.09 35.56 90)
 		(unit 1)
 		(exclude_from_sim no)
@@
 		(fields_autoplaced yes)
 		(property "Reference" "F1"
-			(at 52.07 29.21 90)
+			(at 85.09 29.21 90)
 			(effects
 				(font
@@
 		)
 		(property "Value" "4A"
-			(at 52.07 31.75 90)
+			(at 85.09 31.75 90)
 			(effects
 				(font
@@
 		)
 		(property "Footprint" "Fuse:Fuse_0603_1608Metric"
-			(at 52.07 37.338 90)
+			(at 85.09 37.338 90)
 			(effects
 				(font
@@
 		)
 		(property "Datasheet" "~"
-			(at 52.07 35.56 0)
+			(at 85.09 35.56 0)
 			(effects
 				(font
@@
 		)
 		(property "Description" "Fuse"
-			(at 52.07 35.56 0)
+			(at 85.09 35.56 0)
 			(effects
 				(font
@@
 	)
 	(symbol
+		(lib_id "power:+3.3V")
+		(at 64.77 30.48 0)
+		(unit 1)
+		(exclude_from_sim no)
+		(in_bom yes)
+		(on_board yes)
+		(dnp no)
+		(property "Reference" "#PWR011"
+			(at 64.77 34.29 0)
+			(effects
+				(font
+					(size 1.27 1.27)
+				)
+				(hide yes)
+			)
+		)
+		(property "Value" "VIN"
+			(at 60.452 26.924 0)
+			(effects
+				(font
+					(size 1.27 1.27)
+				)
+				(justify left)
+			)
+		)
+		(property "Footprint" ""
+			(at 64.77 30.48 0)
+			(effects
+				(font
+					(size 1.27 1.27)
+				)
+				(hide yes)
+			)
+		)
+		(property "Datasheet" ""
+			(at 64.77 30.48 0)
+			(effects
+				(font
+					(size 1.27 1.27)
+				)
+				(hide yes)
+			)
+		)
+		(property "Description" ""
+			(at 64.77 30.48 0)
+			(effects
+				(font
+					(size 1.27 1.27)
+				)
+				(hide yes)
+			)
+		)
+		(pin "1"
+		)
+		(instances
+			(project "Fill_Station_ControlBoard"
+				(path "/eaacffe0-ee57-428e-a37e-5655e0922ccc/5d95e092-c448-4af3-bba5-d28c074fd0e0"
+					(reference "#PWR011")
+					(unit 1)
+				)
+			)
+		)
+	)
+	(symbol
 		(lib_id "Device:LED")
 		(at 396.24 48.26 90)
@@
 	)
 	(symbol
-		(lib_id "Connector:TestPoint")
-		(at 398.78 120.65 0)
-		(unit 1)
-		(exclude_from_sim no)
-		(in_bom yes)
-		(on_board yes)
-		(dnp no)
-		(fields_autoplaced yes)
-		(property "Reference" "TP6"
-			(at 401.32 116.0779 0)
-			(effects
-				(font
-					(size 1.27 1.27)
-				)
-				(justify left)
-			)
-		)
-		(property "Value" "TestPoint"
-			(at 401.32 118.6179 0)
-			(effects
-				(font
-					(size 1.27 1.27)
-				)
-				(justify left)
-			)
-		)
-		(property "Footprint" "TestPoint:TestPoint_Pad_D2.0mm"
-			(at 403.86 120.65 0)
-			(effects
-				(font
-					(size 1.27 1.27)
-				)
-				(hide yes)
-			)
-		)
-		(property "Datasheet" "~"
-			(at 403.86 120.65 0)
-			(effects
-				(font
-					(size 1.27 1.27)
-				)
-				(hide yes)
-			)
-		)
-		(property "Description" "test point"
-			(at 398.78 120.65 0)
-			(effects
-				(font
-					(size 1.27 1.27)
-				)
-				(hide yes)
-			)
-		)
-		(pin "1"
-		)
-		(instances
-			(project "Fill_Station_ControlBoard"
-				(path "/eaacffe0-ee57-428e-a37e-5655e0922ccc/5d95e092-c448-4af3-bba5-d28c074fd0e0"
-					(reference "TP6")
-					(unit 1)
-				)
-			)
-		)
-	)
-	(symbol
 		(lib_id "power:GND")
 		(at 30.48 240.03 0)
@@
 			)
 		)
-		(property "Value" "12.8V_BAT"
+		(property "Value" "12.8V"
 			(at 381.762 77.724 0)
 			(effects
@@
 					(unit 1)
 				)
-			)
-		)
-	)
-	(symbol
-		(lib_id "Connector:TestPoint")
-		(at 398.78 113.03 0)
-		(unit 1)
-		(exclude_from_sim no)
-		(in_bom yes)
-		(on_board yes)
-		(dnp no)
-		(fields_autoplaced yes)
-		(property "Reference" "TP5"
-			(at 401.32 108.4579 0)
-			(effects
-				(font
-					(size 1.27 1.27)
-				)
-				(justify left)
-			)
-		)
-		(property "Value" "TestPoint"
-			(at 401.32 110.9979 0)
-			(effects
-				(font
-					(size 1.27 1.27)
-				)
-				(justify left)
-			)
-		)
-		(property "Footprint" "TestPoint:TestPoint_Pad_D2.0mm"
-			(at 403.86 113.03 0)
-			(effects
-				(font
-					(size 1.27 1.27)
-				)
-				(hide yes)
-			)
-		)
-		(property "Datasheet" "~"
-			(at 403.86 113.03 0)
-			(effects
-				(font
-					(size 1.27 1.27)
-				)
-				(hide yes)
-			)
-		)
-		(property "Description" "test point"
-			(at 398.78 113.03 0)
-			(effects
-				(font
-					(size 1.27 1.27)
-				)
-				(hide yes)
-			)
-		)
-		(pin "1"
-		)
-		(instances
-			(project "Fill_Station_ControlBoard"
-				(path "/eaacffe0-ee57-428e-a37e-5655e0922ccc/5d95e092-c448-4af3-bba5-d28c074fd0e0"
-					(reference "TP5")
-					(unit 1)
-				)
