File: Fill_Station_ControlBoard/Alimentation.kicad_sch (KiCad schematic)
At the start: 84 parts, among them IC1 TPS259573DSGR, J13 Screw_Terminal_2_P5.00mm, U1 INA3221, U10 TPSM33620-Q1, U11 TPSM33620-Q1, U12 TPSM33620-Q1, U6 TPS2116DRL, U9 TPS2116DRL

Commit message: Final_V1
Parts:
- removed C106, C108, C111, C113, C82: 10u, Capacitor_SMD:C_0603_1608Metric, symbol Device:C
- removed C109, C110, C114: 22u, Capacitor_SMD:C_0603_1608Metric, symbol Device:C
- removed J13: Screw_Terminal_2_P5.00mm, TerminalBlock_Phoenix:TerminalBlock_Phoenix_PT-1,5-2-5.0-H_1x02_P5.00mm_Horizontal, symbol PCM_SL_Screw_Terminal:Screw_Terminal_2_P5.00mm
- added C3, C4: 22u, Capacitor_SMD:C_1210_3225Metric, symbol Device:C
- added C5, C55: 10u, Capacitor_SMD:C_0805_2012Metric, symbol Device:C
- added C56, C58: 10u, Capacitor_SMD:C_0603_1608Metric, symbol Device:C
- added C61, C78: 22u, Capacitor_SMD:C_0603_1608Metric, symbol Device:C
- added J19: ~, Connector_AMASS:AMASS_XT60-M_1x02_P7.20mm_Vertical, symbol matispoulin:AMASS_XT60PW
- C1, C115, C116, C117, C38: LCSC (none) -> C14663
- C107, C112, C62, C76, C77, C79, C8, C9: LCSC (none) -> C59302
- C15, C2, C6, C60, C74: LCSC (none) -> C22399626
- C57: value 100uF_25V -> 100uF_50V; footprint Capacitor_THT:CP_Radial_D6.3mm_P2.50mm -> Capacitor_SMD:CP_Elec_6.3x7.7; LCSC (none) -> C165974
- C59: value 10uF_25V -> 10uF_50V; footprint Capacitor_THT:CP_Radial_D5.0mm_P2.00mm -> Capacitor_SMD:CP_Elec_5x5.3
- C71: footprint Capacitor_SMD:C_0603_1608Metric -> Capacitor_SMD:C_0805_2012Metric; LCSC (none) -> C326595
- C75: LCSC (none) -> C60077
- C84: footprint Capacitor_SMD:C_0603_1608Metric -> Resistor_SMD:R_0603_1608Metric; LCSC (none) -> C5341638
- C85: value 22u -> 10u; LCSC (none) -> C22399626
- D10, D8, D9: LCSC (none) -> C2288
- D11, D12, D7: LCSC (none) -> C12065
- D13, D14: LCSC (none) -> C2286
- D16: LCSC (none) -> C10763
- F1: LCSC (none) -> C187606; now fitted
- IC1: LCSC (none) -> C471038
- R132, R133, R134, R4, R8, R9: LCSC (none) -> C173683
- R162, R2, R3: LCSC (none) -> C2074926
- R5, R65: footprint Capacitor_SMD:C_0603_1608Metric -> Resistor_SMD:R_0603_1608Metric
- R67: value R_US -> 365k
- R68: value R_US -> 32k
- R7: LCSC (none) -> C22369937
- R71, R72, R74, R76: LCSC (none) -> C22356475
- R73: footprint Resistor_SMD:R_0603_1608Metric_Pad0.98x0.95mm_HandSolder -> Resistor_SMD:R_0402_1005Metric
- R75: footprint Capacitor_SMD:C_0603_1608Metric -> Resistor_SMD:R_0603_1608Metric; LCSC (none) -> C22369937
- R77: LCSC (none) -> C22356624
- R78: value R_US -> 10k; LCSC (none) -> C22369937
- U1: LCSC (none) -> C181255
- U10, U12: LCSC (none) -> C49261907
- U11: LCSC (none) -> C51956999
- U6, U9: LCSC (none) -> C3235557
Connections:
- net 12.8V: now also C3.1, C5.1; no longer C85.1
- net 3V3: now also C15.1, C60.1; no longer C6.1
- net 3V3_USB: now also C58.1, C78.1
- net 5V: now also C6.1, C85.1; no longer C15.1, C60.1
- net 5V_Bat: now also C56.1, C61.1
- net 5V_USB: now also C4.1, C55.1
- net GND: now also C3.2, C4.2, C5.2, C55.2, C56.2, C58.2, C61.2, C78.2, J19.1
- net VIN: now also J19.2
Other:
- note added: "1.7A max"
- note removed: "Confirmer les resistors en fonction de la couleur des leds"
- note removed: "I_lim : 1A"
