File: Fill_Station_ControlBoard/CANFD.kicad_sch (KiCad schematic)
At the start: 10 parts, among them J8 DE9_Socket_MountingHoles, U3 TCAN337G

Commit message: Ajout power
Parts:
- CR1: footprint SOT323-3L_STM -> (none)
Changed lines of the file:
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@@
 			)
 		)
-		(property "Footprint" "SOT323-3L_STM"
+		(property "Footprint" ""
 			(at 163.83 91.44 0)
 			(effects

Commit message: début layout
Parts:
- CR1: footprint (none) -> ESDCAN:SOT323-3L_STM
- renumbered C37 to C60, C38 to C62, J8 to J14, R42 to R55, R43 to R56, R46 to R57, R5 to R58, R44 to R62, U3 to U5
Changed lines of the file:
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@@
 		(on_board yes)
 		(dnp no)
-		(property "Reference" "#PWR053"
+		(property "Reference" "#PWR091"
 			(at 83.82 64.77 0)
 			(effects
@@
 			(project "Fill_Station_ControlBoard"
 				(path "/eaacffe0-ee57-428e-a37e-5655e0922ccc/89a4eee6-f04c-46ec-a929-95355d7dfe4e"
-					(reference "#PWR053")
+					(reference "#PWR091")
 					(unit 1)
 				)
@@
 		(on_board yes)
 		(dnp no)
-		(property "Reference" "R44"
+		(property "Reference" "R62"
 			(at 156.21 81.28 0)
 			(effects
@@
 			(project "Fill_Station_ControlBoard"
 				(path "/eaacffe0-ee57-428e-a37e-5655e0922ccc/89a4eee6-f04c-46ec-a929-95355d7dfe4e"
-					(reference "R44")
+					(reference "R62")
 					(unit 1)
 				)
@@
 		(dnp no)
 		(fields_autoplaced yes)
-		(property "Reference" "J8"
+		(property "Reference" "J14"
 			(at 193.04 77.4699 0)
 			(effects
@@
 			(project "Fill_Station_ControlBoard"
 				(path "/eaacffe0-ee57-428e-a37e-5655e0922ccc/89a4eee6-f04c-46ec-a929-95355d7dfe4e"
-					(reference "J8")
+					(reference "J14")
 					(unit 1)
 				)
@@
 		(dnp no)
 		(fields_autoplaced yes)
-		(property "Reference" "C37"
+		(property "Reference" "C60"
 			(at 127 55.8799 0)
 			(effects
@@
 			(project "Fill_Station_ControlBoard"
 				(path "/eaacffe0-ee57-428e-a37e-5655e0922ccc/89a4eee6-f04c-46ec-a929-95355d7dfe4e"
-					(reference "C37")
+					(reference "C60")
 					(unit 1)
 				)
@@
 		(dnp no)
 		(fields_autoplaced yes)
-		(property "Reference" "U3"
+		(property "Reference" "U5"
 			(at 118.9833 66.04 0)
 			(effects
@@
 			(project "Fill_Station_ControlBoard"
 				(path "/eaacffe0-ee57-428e-a37e-5655e0922ccc/89a4eee6-f04c-46ec-a929-95355d7dfe4e"
-					(reference "U3")
+					(reference "U5")
 					(unit 1)
 				)
@@
 		(on_board yes)
 		(dnp no)
-		(property "Reference" "R43"
+		(property "Reference" "R56"
 			(at 74.676 78.486 90)
 			(effects
@@
 			(project "Fill_Station_ControlBoard"
 				(path "/eaacffe0-ee57-428e-a37e-5655e0922ccc/89a4eee6-f04c-46ec-a929-95355d7dfe4e"
-					(reference "R43")
+					(reference "R56")
 					(unit 1)
 				)
@@
 		(dnp no)
 		(fields_autoplaced yes)
-		(property "Reference" "#PWR017"
+		(property "Reference" "#PWR095"
 			(at 116.84 100.33 0)
 			(effects
@@
 			(project "Fill_Station_ControlBoard"
 				(path "/eaacffe0-ee57-428e-a37e-5655e0922ccc/89a4eee6-f04c-46ec-a929-95355d7dfe4e"
-					(reference "#PWR017")
+					(reference "#PWR095")
 					(unit 1)
 				)
@@
 		(on_board yes)
 		(dnp no)
-		(property "Reference" "R5"
+		(property "Reference" "R58"
 			(at 100.33 87.63 0)
 			(effects
@@
 			(project "Fill_Station_ControlBoard"
 				(path "/eaacffe0-ee57-428e-a37e-5655e0922ccc/89a4eee6-f04c-46ec-a929-95355d7dfe4e"
-					(reference "R5")
+					(reference "R58")
 					(unit 1)
 				)
@@
 		(on_board yes)
 		(dnp no)
-		(property "Reference" "#PWR022"
+		(property "Reference" "#PWR0110"
 			(at 187.96 102.87 0)
 			(effects
@@
 			(project "Fill_Station_ControlBoard"
 				(path "/eaacffe0-ee57-428e-a37e-5655e0922ccc/89a4eee6-f04c-46ec-a929-95355d7dfe4e"
-					(reference "#PWR022")
+					(reference "#PWR0110")
 					(unit 1)
 				)
@@
 		(dnp no)
 		(fields_autoplaced yes)
-		(property "Reference" "#PWR020"
+		(property "Reference" "#PWR094"
 			(at 116.84 52.07 0)
 			(effects
@@
 			(project "Fill_Station_ControlBoard"
 				(path "/eaacffe0-ee57-428e-a37e-5655e0922ccc/89a4eee6-f04c-46ec-a929-95355d7dfe4e"
-					(reference "#PWR020")
+					(reference "#PWR094")
 					(unit 1)
 				)
@@
 		(on_board yes)
 		(dnp no)
-		(property "Reference" "R46"
+		(property "Reference" "R57"
 			(at 85.09 66.04 0)
 			(effects
@@
 			(project "Fill_Station_ControlBoard"
 				(path "/eaacffe0-ee57-428e-a37e-5655e0922ccc/89a4eee6-f04c-46ec-a929-95355d7dfe4e"
-					(reference "R46")
+					(reference "R57")
 					(unit 1)
 				)
@@
 		(dnp no)
 		(fields_autoplaced yes)
-		(property "Reference" "#PWR039"
+		(property "Reference" "#PWR092"
 			(at 99.06 99.06 0)
 			(effects
@@
 			(project "Fill_Station_ControlBoard"
 				(path "/eaacffe0-ee57-428e-a37e-5655e0922ccc/89a4eee6-f04c-46ec-a929-95355d7dfe4e"
-					(reference "#PWR039")
+					(reference "#PWR092")
 					(unit 1)
 				)
@@
 		(on_board yes)
 		(dnp no)
-		(property "Reference" "R42"
+		(property "Reference" "R55"
 			(at 74.93 71.628 90)
 			(effects
@@
 			(project "Fill_Station_ControlBoard"
 				(path "/eaacffe0-ee57-428e-a37e-5655e0922ccc/89a4eee6-f04c-46ec-a929-95355d7dfe4e"
-					(reference "R42")
+					(reference "R55")
 					(unit 1)
 				)
@@
 		(dnp no)
 		(fields_autoplaced yes)
-		(property "Reference" "#PWR021"
+		(property "Reference" "#PWR0100"
 			(at 163.83 120.65 0)
 			(effects
@@
 			(project "Fill_Station_ControlBoard"
 				(path "/eaacffe0-ee57-428e-a37e-5655e0922ccc/89a4eee6-f04c-46ec-a929-95355d7dfe4e"
-					(reference "#PWR021")
+					(reference "#PWR0100")
 					(unit 1)
 				)
@@
 		(dnp no)
 		(fields_autoplaced yes)
-		(property "Reference" "C38"
+		(property "Reference" "C62"
 			(at 139.7 55.8799 0)
 			(effects
@@
 			(project "Fill_Station_ControlBoard"
 				(path "/eaacffe0-ee57-428e-a37e-5655e0922ccc/89a4eee6-f04c-46ec-a929-95355d7dfe4e"
-					(reference "C38")
+					(reference "C62")
 					(unit 1)
 				)
@@
 		(on_board yes)
 		(dnp no)
-		(property "Reference" "#PWR054"
+		(property "Reference" "#PWR099"
 			(at 135.89 69.85 0)
 			(effects
@@
 			(project "Fill_Station_ControlBoard"
 				(path "/eaacffe0-ee57-428e-a37e-5655e0922ccc/89a4eee6-f04c-46ec-a929-95355d7dfe4e"
-					(reference "#PWR054")
+					(reference "#PWR099")
 					(unit 1)
 				)
@@
 		(dnp no)
 		(fields_autoplaced yes)
-		(property "Reference" "#PWR018"
+		(property "Reference" "#PWR0104"
 			(at 173.99 87.63 0)
 			(effects
@@
 			(project "Fill_Station_ControlBoard"
 				(path "/eaacffe0-ee57-428e-a37e-5655e0922ccc/89a4eee6-f04c-46ec-a929-95355d7dfe4e"
-					(reference "#PWR018")
+					(reference "#PWR0104")
 					(unit 1)
 				)
@@
 			)
 		)
-		(property "Footprint" ""
+		(property "Footprint" "ESDCAN:SOT323-3L_STM"
 			(at 163.83 91.44 0)
 			(effects

Commit message: PCB fait
Parts:
- removed C60: 100nF, Capacitor_SMD:C_0603_1608Metric, symbol Device:C
- removed C62: 1uF, Capacitor_SMD:C_0603_1608Metric, symbol Device:C
- removed CR1: ESDCAN02-2BWY, ESDCAN:SOT323-3L_STM, symbol ESDCAN:ESDCAN02-2BWY
- removed J14: DE9_Socket_MountingHoles, Connector_Dsub:DSUB-9_Socket_Vertical_P2.77x2.84mm_MountingHoles, symbol Connector:DE9_Socket_MountingHoles
- removed R55, R56: 33, Resistor_SMD:R_0603_1608Metric_Pad0.98x0.95mm_HandSolder, symbol Device:R_US
- removed R57, R58: 10k, Resistor_SMD:R_0603_1608Metric_Pad0.98x0.95mm_HandSolder, symbol Device:R_US
- removed R62: 120, Resistor_SMD:R_0603_1608Metric_Pad0.98x0.95mm_HandSolder, symbol Device:R_US
- removed U5: TCAN337G, Package_TO_SOT_SMD:TSOT-23-8_HandSoldering, symbol Interface_CAN_LIN:TCAN337G
- added C67: 10nF, Capacitor_SMD:C_0603_1608Metric, symbol Device:C
- added C68, C72: 1u, Capacitor_SMD:C_0603_1608Metric, symbol Device:C
- added C69: 10u, Capacitor_SMD:C_0603_1608Metric, symbol Device:C
- added C70, C73: 100nF, Capacitor_SMD:C_0603_1608Metric, symbol Device:C
- added CR2: ESDCAN02-2BWY, ESDCAN:SOT323-3L_STM, symbol ESDCAN:ESDCAN02-2BWY
- added J16: DE9_Socket_MountingHoles, Connector_Dsub:DSUB-9_Socket_Vertical_P2.77x2.84mm_MountingHoles, symbol Connector:DE9_Socket_MountingHoles
- added R84, R87: 10k, Resistor_SMD:R_0603_1608Metric_Pad0.98x0.95mm_HandSolder, symbol Device:R_US
- added R85: 120, Resistor_SMD:R_0603_1608Metric_Pad0.98x0.95mm_HandSolder, symbol Device:R_US
- added R86: 0, Resistor_SMD:R_0603_1608Metric_Pad0.98x0.95mm_HandSolder, symbol Device:R_US
- added R88: 22, Resistor_SMD:R_0402_1005Metric, symbol Device:R_US
- added U8: ISOW1044, Package_SO:SOIC-20W_7.5x12.8mm_P1.27mm, symbol Interface_CAN_LIN:ISOW1044
Connections:
- net 3V3: now also C70.1, R84.1, U8.1 (VIO)
- net CAN.RXD: now also R88.1
- net CAN.TXD: now also U8.3 (TXD)
- net CAN_N: now also CR2.2, J16.2, R85.1, U8.18 (CANL)
- net CAN_P: now also CR2.1, J16.7, R85.2, U8.19 (CANH)
- net GND: now also C67.1, C68.1, C69.1, C70.2, R87.2, U8.10 (GND1), U8.6 (GNDIO)
- new net: R88.2, U8.5 (RXD)
- new net: R86.2, U8.12 (VISOOUT), U8.13 (VSIN)
- new net: C72.2, C73.2, R86.1, U8.20 (VISOIN)
- new net: R87.1, U8.4 (STB)
- new net: R84.2, U8.8 (EN/FLT)
- new net 5V: C67.2, C68.2, C69.2, U8.9 (VDD)
- new net CHASSIS_CAN: C72.1, C73.1, CR2.3, J16.0 (PAD), J16.3, U8.11 (GND2), U8.15 (GISOIN), U8.16 (GISOIN), U8.17 (GISOIN)
- no-connect marks 6 -> 2
Other:
- note removed: "Internal TXD pull-up"

Commit message: Travail Layout
Parts:
- added C7, C89: 1000p - 2000V, Capacitor_SMD:C_1210_3225Metric, symbol Device:C
Connections:
- net CAN_N: now also J16.1
- net CAN_P: now also J16.6
- net CHASSIS_CAN: now also J16.8, C7.2, C89.2
- net GND: now also C7.1, C89.1
Other:
- moved on the sheet: C67, C68, C69, C70, C72, C73, CR2, J16, R84, R85, R86, R87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

Commit message: PCB presque terminé
Modifs de l'alim
Connections:
- no-connect marks 2 -> 5
Changed lines of the file:
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@@
+	)
+	(no_connect
+		(at 168.91 83.82)
 	)
 	(no_connect
 		(at 64.77 78.74)
 	)
+	(no_connect
+		(at 168.91 86.36)
+	)
+	(no_connect
+		(at 168.91 81.28)
+	)
 	(wire

Commit message: Final_V1
Parts:
- C67: value 10nF -> 10n; LCSC (none) -> C100042
- C68, C72: LCSC (none) -> C59302
- C69: LCSC (none) -> C22399626
- C7, C89: LCSC (none) -> C9196
- C70, C73: value 100nF -> 100n; LCSC (none) -> C14663
- CR2: LCSC (none) -> C2969759
- J16: LCSC (none) -> C141882
- R84, R87: footprint Resistor_SMD:R_0603_1608Metric_Pad0.98x0.95mm_HandSolder -> Resistor_SMD:R_0603_1608Metric; LCSC (none) -> C22369937
- R85: LCSC (none) -> C177328
- R86: footprint Resistor_SMD:R_0603_1608Metric_Pad0.98x0.95mm_HandSolder -> Resistor_SMD:R_0402_1005Metric; LCSC (none) -> C17168
- R88: LCSC (none) -> C25092
- U8: LCSC (none) -> C3234830
Changed lines of the file:
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@@
+			)
+		)
+		(property "LCSC" "C25092"
+			(at 58.42 73.66 90)
+			(effects
+				(font
+					(size 1.27 1.27)
+				)
+				(hide yes)
 			)
 		)
@@
 		(property "Description" ""
 			(at 134.62 76.2 0)
+			(effects
+				(font
+					(size 1.27 1.27)
+				)
+				(hide yes)
+			)
+		)
+		(property "LCSC" "C2969759"
+			(at 134.62 76.2 90)
 			(effects
 				(font
@@
 			)
 		)
+		(property "LCSC" "C3234830"
+			(at 80.01 78.74 0)
+			(effects
+				(font
+					(size 1.27 1.27)
+				)
+				(hide yes)
+			)
+		)
 		(pin "10"
 		)
@@
 			)
 		)
+		(property "LCSC" "C59302"
+			(at 107.95 57.15 0)
+			(effects
+				(font
+					(size 1.27 1.27)
+				)
+				(hide yes)
+			)
+		)
 		(pin "1"
 		)
@@
 		(property "Description" "Unpolarized capacitor"
 			(at 77.47 111.76 0)
+			(effects
+				(font
+					(size 1.27 1.27)
+				)
+				(hide yes)
+			)
+		)
+		(property "LCSC" "C9196"
+			(at 77.47 111.76 90)
 			(effects
 				(font
@@
 			)
 		)
+		(property "LCSC" "C141882"
+			(at 176.53 76.2 0)
+			(effects
+				(font
+					(size 1.27 1.27)
+				)
+				(hide yes)
+			)
+		)
 		(pin "2"
 		)
@@
 			)
 		)
-		(property "Value" "10nF"
-			(at 93.472 36.83 0)
+		(property "Value" "10n"
+			(at 92.202 36.83 0)
 			(effects
 				(font
@@
 			)
 		)
+		(property "LCSC" "C100042"
+			(at 85.09 38.1 0)
+			(effects
+				(font
+					(size 1.27 1.27)
+				)
+				(hide yes)
+			)
+		)
 		(pin "1"
 		)
@@
 			)
 		)
-		(property "Footprint" "Resistor_SMD:R_0603_1608Metric_Pad0.98x0.95mm_HandSolder"
+		(property "Footprint" "Resistor_SMD:R_0402_1005Metric"
 			(at 100.076 59.944 90)
 			(effects
@@
 			)
 		)
+		(property "LCSC" "C17168"
+			(at 99.06 59.69 0)
+			(effects
+				(font
+					(size 1.27 1.27)
+				)
+				(hide yes)
+			)
+		)
 		(pin "1"
 		)
@@
 			)
 		)
-		(property "Value" "100nF"
+		(property "Value" "100n"
 			(at 125.222 55.88 0)
 			(effects
@@
 		)
 		(property "Description" "Unpolarized capacitor"
+			(at 116.84 57.15 0)
+			(effects
+				(font
+					(size 1.27 1.27)
+				)
+				(hide yes)
+			)
+		)
+		(property "LCSC" "C14663"
 			(at 116.84 57.15 0)
 			(effects
@@
 			)
 		)
+		(property "LCSC" "C9196"
+			(at 77.47 102.87 90)
+			(effects
+				(font
+					(size 1.27 1.27)
+				)
+				(hide yes)
+			)
+		)
 		(pin "1"
 		)
@@
 		(property "Description" "Resistor, US symbol"
 			(at 104.14 77.47 0)
+			(effects
+				(font
+					(size 1.27 1.27)
+				)
+				(hide yes)
+			)
+		)
+		(property "LCSC" "C177328"
+			(at 104.14 77.47 90)
 			(effects
 				(font
@@
 			)
 		)
-		(property "Value" "100nF"
+		(property "Value" "100n"
 			(at 58.42 58.4199 0)
 			(effects
@@
 			)
 		)
+		(property "LCSC" "C14663"
+			(at 54.61 57.15 0)
+			(effects
+				(font
+					(size 1.27 1.27)
+				)
+				(hide yes)
+			)
+		)
 		(pin "1"
 		)
@@
 			)
 		)
-		(property "Footprint" "Resistor_SMD:R_0603_1608Metric_Pad0.98x0.95mm_HandSolder"
+		(property "Footprint" "Resistor_SMD:R_0603_1608Metric"
 			(at 41.656 81.534 90)
 			(effects
@@
 			)
 		)
+		(property "LCSC" "C22369937"
+			(at 40.64 81.28 0)
+			(effects
+				(font
+					(size 1.27 1.27)
+				)
+				(hide yes)
+			)
+		)
 		(pin "1"
 		)
@@
 			)
 		)
+		(property "LCSC" "C59302"
+			(at 95.25 38.1 0)
+			(effects
+				(font
+					(size 1.27 1.27)
+				)
+				(hide yes)
+			)
+		)
 		(pin "1"
 		)
@@
 			)
 		)
-		(property "Footprint" "Resistor_SMD:R_0603_1608Metric_Pad0.98x0.95mm_HandSolder"
+		(property "Footprint" "Resistor_SMD:R_0603_1608Metric"
 			(at 59.436 92.964 90)
 			(effects
@@
 		)
 		(property "Description" "Resistor, US symbol"
+			(at 58.42 92.71 0)
+			(effects
+				(font
+					(size 1.27 1.27)
+				)
+				(hide yes)
+			)
+		)
+		(property "LCSC" "C22369937"
 			(at 58.42 92.71 0)
 			(effects
@@
 			(at 105.41 38.1 0)
 			(effects
+				(font
+					(size 1.27 1.27)
+				)
+				(hide yes)
+			)
+		)
+		(property "LCSC" "C22399626"
+			(at 105.41 38.1 0)
+			(effects
