File: Fill_Station_ControlBoard/Fill_Station_ControlBoard.kicad_sch (KiCad schematic)
At the start: 0 parts

Commit message: PCB fini avant review avec greg
Other:
- added sheet SPI (SPI.kicad_sch)
- sheet Control ports: added none; removed Heater1, Heater2, Heater3
- sheet MCU ports: added SPI4.CS, SPI4.MISO, SPI4.MOSI, SPI4.SCK, SPI5.CS, SPI5.MISO, SPI5.MOSI, SPI5.SCK; removed Heater1, Heater2, Heater3
Changed lines of the file:
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@@
 	(wire
 		(pts
-			(xy 252.73 73.66) (xy 303.53 73.66)
-		)
-		(stroke
-			(width 0)
-			(type default)
-		)
-	)
-	(wire
-		(pts
-			(xy 176.53 99.06) (xy 99.06 99.06)
-		)
-		(stroke
-			(width 0)
-			(type default)
-		)
-	)
-	(wire
-		(pts
-			(xy 252.73 76.2) (xy 303.53 76.2)
+			(xy 99.06 71.12) (xy 176.53 71.12)
+		)
+		(stroke
+			(width 0)
+			(type default)
+		)
+	)
+	(wire
+		(pts
+			(xy 99.06 99.06) (xy 176.53 99.06)
+		)
+		(stroke
+			(width 0)
+			(type default)
+		)
+	)
+	(wire
+		(pts
+			(xy 99.06 68.58) (xy 176.53 68.58)
 		)
 		(stroke
@@
 	(wire
 		(pts
+			(xy 176.53 66.04) (xy 99.06 66.04)
+		)
+		(stroke
+			(width 0)
+			(type default)
+		)
+	)
+	(wire
+		(pts
 			(xy 252.73 162.56) (xy 303.53 162.56)
 		)
@@
 	(wire
 		(pts
+			(xy 99.06 53.34) (xy 176.53 53.34)
+		)
+		(stroke
+			(width 0)
+			(type default)
+		)
+	)
+	(wire
+		(pts
 			(xy 252.73 102.87) (xy 303.53 102.87)
 		)
@@
 	(wire
 		(pts
+			(xy 99.06 73.66) (xy 176.53 73.66)
+		)
+		(stroke
+			(width 0)
+			(type default)
+		)
+	)
+	(wire
+		(pts
 			(xy 252.73 173.99) (xy 303.53 173.99)
 		)
@@
 	(wire
 		(pts
+			(xy 99.06 58.42) (xy 176.53 58.42)
+		)
+		(stroke
+			(width 0)
+			(type default)
+		)
+	)
+	(wire
+		(pts
 			(xy 252.73 154.94) (xy 303.53 154.94)
 		)
@@
 	(wire
 		(pts
-			(xy 252.73 71.12) (xy 303.53 71.12)
-		)
-		(stroke
-			(width 0)
-			(type default)
-		)
-	)
-	(wire
-		(pts
 			(xy 252.73 160.02) (xy 303.53 160.02)
 		)
@@
 		(pts
 			(xy 99.06 176.53) (xy 176.53 176.53)
+		)
+		(stroke
+			(width 0)
+			(type default)
+		)
+	)
+	(wire
+		(pts
+			(xy 99.06 55.88) (xy 176.53 55.88)
+		)
+		(stroke
+			(width 0)
+			(type default)
+		)
+	)
+	(wire
+		(pts
+			(xy 99.06 60.96) (xy 176.53 60.96)
 		)
 		(stroke
@@
 	)
 	(sheet
+		(at 60.96 49.53)
+		(size 38.1 29.21)
+		(exclude_from_sim no)
+		(in_bom yes)
+		(on_board yes)
+		(dnp no)
+		(fields_autoplaced yes)
+		(stroke
+			(width 0.1524)
+			(type solid)
+		)
+		(fill
+			(color 0 0 0 0.0000)
+		)
+		(property "Sheetname" "SPI"
+			(at 60.96 48.8184 0)
+			(effects
+				(font
+					(size 1.27 1.27)
+				)
+				(justify left bottom)
+			)
+		)
+		(property "Sheetfile" "SPI.kicad_sch"
+			(at 60.96 79.3246 0)
+			(effects
+				(font
+					(size 1.27 1.27)
+				)
+				(justify left top)
+			)
+		)
+		(pin "SPI4.MOSI" input
+			(at 99.06 55.88 0)
+			(effects
+				(font
+					(size 1.27 1.27)
+				)
+				(justify right)
+			)
+		)
+		(pin "SPI4.SCK" input
+			(at 99.06 58.42 0)
+			(effects
+				(font
+					(size 1.27 1.27)
+				)
+				(justify right)
+			)
+		)
+		(pin "SPI4.CS" input
+			(at 99.06 60.96 0)
+			(effects
+				(font
+					(size 1.27 1.27)
+				)
+				(justify right)
+			)
+		)
+		(pin "SPI5.MOSI" input
+			(at 99.06 68.58 0)
+			(effects
+				(font
+					(size 1.27 1.27)
+				)
+				(justify right)
+			)
+		)
+		(pin "SPI5.SCK" input
+			(at 99.06 71.12 0)
+			(effects
+				(font
+					(size 1.27 1.27)
+				)
+				(justify right)
+			)
+		)
+		(pin "SPI5.CS" input
+			(at 99.06 73.66 0)
+			(effects
+				(font
+					(size 1.27 1.27)
+				)
+				(justify right)
+			)
+		)
+		(pin "SPI4.MISO" output
+			(at 99.06 53.34 0)
+			(effects
+				(font
+					(size 1.27 1.27)
+				)
+				(justify right)
+			)
+		)
+		(pin "SPI5.MISO" output
+			(at 99.06 66.04 0)
+			(effects
+				(font
+					(size 1.27 1.27)
+				)
+				(justify right)
+			)
+		)
+		(instances
+			(project "Fill_Station_ControlBoard"
+				(path "/eaacffe0-ee57-428e-a37e-5655e0922ccc"
+					(page "9")
+				)
+			)
+		)
+	)
+	(sheet
 		(at 303.53 48.26)
 		(size 38.1 63.5)
@@
 		(pin "E-match1_Det" output
 			(at 303.53 53.34 180)
-			(effects
-				(font
-					(size 1.27 1.27)
-				)
-				(justify left)
-			)
-		)
-		(pin "Heater2" input
-			(at 303.53 73.66 180)
-			(effects
-				(font
-					(size 1.27 1.27)
-				)
-				(justify left)
-			)
-		)
-		(pin "Heater1" input
-			(at 303.53 71.12 180)
-			(effects
-				(font
-					(size 1.27 1.27)
-				)
-				(justify left)
-			)
-		)
-		(pin "Heater3" input
-			(at 303.53 76.2 180)
 			(effects
 				(font
@@
 			)
 		)
-		(pin "Heater2" output
-			(at 252.73 73.66 0)
-			(effects
-				(font
-					(size 1.27 1.27)
-				)
-				(justify right)
-			)
-		)
-		(pin "Heater3" output
-			(at 252.73 76.2 0)
-			(effects
-				(font
-					(size 1.27 1.27)
-				)
-				(justify right)
-			)
-		)
-		(pin "Heater1" output
-			(at 252.73 71.12 0)
-			(effects
-				(font
-					(size 1.27 1.27)
-				)
-				(justify right)
-			)
-		)
 		(pin "SD2.DET" input
 			(at 176.53 176.53 180)
@@
 			(effects
 				(font
+					(size 1.27 1.27)
+				)
+				(justify left)
+			)
+		)
+		(pin "SPI4.MISO" input
+			(at 176.53 53.34 180)
+			(effects
+				(font
+					(size 1.27 1.27)
+				)
+				(justify left)
+			)
+		)
+		(pin "SPI4.SCK" output
+			(at 176.53 58.42 180)
+			(effects
+				(font
+					(size 1.27 1.27)
+				)
+				(justify left)
+			)
+		)
+		(pin "SPI4.MOSI" output
+			(at 176.53 55.88 180)
+			(effects
+				(font
+					(size 1.27 1.27)
+				)
+				(justify left)
+			)
+		)
+		(pin "SPI5.MOSI" output
+			(at 176.53 68.58 180)
+			(effects
+				(font
+					(size 1.27 1.27)
+				)
+				(justify left)
+			)
+		)
+		(pin "SPI5.MISO" input
+			(at 176.53 66.04 180)
+			(effects
+				(font
+					(size 1.27 1.27)
+				)
+				(justify left)
+			)
+		)
+		(pin "SPI5.SCK" output
+			(at 176.53 71.12 180)
+			(effects
+				(font
+					(size 1.27 1.27)
+				)
+				(justify left)
+			)
+		)
+		(pin "SPI5.CS" output
+			(at 176.53 73.66 180)
+			(effects
+				(font
+					(size 1.27 1.27)
+				)
+				(justify left)
+			)
+		)
+		(pin "SPI4.CS" output
+			(at 176.53 60.96 180)
+			(effects
+				(font

Commit message: Final_V1
Other:
- sheet SPI renamed Serial
- sheet MCU ports: added Buzz, I2C1.SCL, I2C1.SDA; removed none
- sheet Serial ports: added I2C1.SCL, I2C1.SDA; removed none
Changed lines of the file:
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@@
+	(wire
+		(pts
+			(xy 252.73 109.22) (xy 303.53 109.22)
+		)
+		(stroke
+			(width 0)
+			(type default)
+		)
+	)
 	(wire
 		(pts
@@
 	(wire
 		(pts
+			(xy 99.06 78.74) (xy 176.53 78.74)
+		)
+		(stroke
+			(width 0)
+			(type default)
+		)
+	)
+	(wire
+		(pts
 			(xy 99.06 166.37) (xy 176.53 166.37)
 		)
@@
 		(pts
 			(xy 99.06 154.94) (xy 176.53 154.94)
+		)
+		(stroke
+			(width 0)
+			(type default)
+		)
+	)
+	(wire
+		(pts
+			(xy 99.06 81.28) (xy 176.53 81.28)
 		)
 		(stroke
@@
 	(sheet
 		(at 60.96 49.53)
-		(size 38.1 29.21)
+		(size 38.1 35.56)
 		(exclude_from_sim no)
 		(in_bom yes)
@@
 			(color 0 0 0 0.0000)
 		)
-		(property "Sheetname" "SPI"
+		(property "Sheetname" "Serial"
 			(at 60.96 48.8184 0)
 			(effects
@@
 		)
 		(property "Sheetfile" "SPI.kicad_sch"
-			(at 60.96 79.3246 0)
+			(at 60.96 85.6746 0)
 			(effects
 				(font
@@
 		(pin "SPI5.MISO" output
 			(at 99.06 66.04 0)
+			(effects
+				(font
+					(size 1.27 1.27)
+				)
+				(justify right)
+			)
+		)
+		(pin "I2C1.SCL" input
+			(at 99.06 78.74 0)
+			(effects
+				(font
+					(size 1.27 1.27)
+				)
+				(justify right)
+			)
+		)
+		(pin "I2C1.SDA" bidirectional
+			(at 99.06 81.28 0)
 			(effects
 				(font
@@
 			(effects
 				(font
+					(size 1.27 1.27)
+				)
+				(justify left)
+			)
+		)
+		(pin "Buzz" output
+			(at 252.73 109.22 0)
+			(effects
+				(font
+					(size 1.27 1.27)
+				)
+				(justify right)
+			)
+		)
+		(pin "I2C1.SDA" bidirectional
+			(at 176.53 81.28 180)
+			(effects
+				(font
+					(size 1.27 1.27)
+				)
+				(justify left)
+			)
+		)
+		(pin "I2C1.SCL" output
+			(at 176.53 78.74 180)
+			(effects
+				(font
