File: Fill_Station_ControlBoard/SPI.kicad_sch (KiCad schematic)
At the start: 2 parts, among them J17 PINHD_1x6_Male, J18 PINHD_1x6_Male

Commit message: Final_V1
Parts:
- added J13: PINHD_1x4_Male, Connector_PinHeader_2.54mm:PinHeader_1x04_P2.54mm_Vertical, symbol PCM_SL_Pin_Headers:PINHD_1x4_Male
- J17, J18: now not fitted; now left out of the parts list
Connections:
- net 3V3: now also J13.1
- net GND: now also J13.4
- new net I2C1.SCL: J13.2
- new net I2C1.SDA: J13.3
Other:
- note added: "I2C1"
