File: Fill_Station_ControlBoard/Storage.kicad_sch (KiCad schematic)
At the start: 15 parts, among them J2 Micro_SD_Card_Det1

Commit message: Ajout de footprint
Parts:
- J2: footprint (none) -> Connector_Card:microSD_HC_Molex_47219-2001
Changed lines of the file:
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@@
 			)
 		)
-		(property "Footprint" ""
+		(property "Footprint" "Connector_Card:microSD_HC_Molex_47219-2001"
 			(at 236.22 85.09 0)
 			(effects

Commit message: début layout
Parts:
- R38: renamed from R56; footprint (none) -> Resistor_SMD:R_0402_1005Metric
- R39: renamed from R59; footprint (none) -> Resistor_SMD:R_0402_1005Metric
- R40: renamed from R57; footprint (none) -> Resistor_SMD:R_0402_1005Metric
- R41: renamed from R58; footprint (none) -> Resistor_SMD:R_0402_1005Metric
- R42: renamed from R60; footprint (none) -> Resistor_SMD:R_0402_1005Metric
- R43: renamed from R61; footprint (none) -> Resistor_SMD:R_0402_1005Metric
- R44: renamed from R62; footprint (none) -> Resistor_SMD:R_0402_1005Metric
- R45: renamed from R63; footprint (none) -> Resistor_SMD:R_0402_1005Metric
- R46: renamed from R64; footprint (none) -> Resistor_SMD:R_0402_1005Metric
- R47: renamed from R65; footprint (none) -> Resistor_SMD:R_0402_1005Metric
- R48: renamed from R66; footprint (none) -> Resistor_SMD:R_0402_1005Metric
- renumbered C45 to C12, C46 to C13, C47 to C14, J2 to J11
Changed lines of the file:
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@@
 		(on_board yes)
 		(dnp no)
-		(property "Reference" "R58"
+		(property "Reference" "R41"
 			(at 86.106 101.854 90)
 			(effects
@@
 			)
 		)
-		(property "Footprint" ""
+		(property "Footprint" "Resistor_SMD:R_0402_1005Metric"
 			(at 90.424 101.854 90)
 			(effects
@@
 			(project "Fill_Station_ControlBoard"
 				(path "/eaacffe0-ee57-428e-a37e-5655e0922ccc/86dfffbf-ac08-41cb-ab8f-382cca5b005c"
-					(reference "R58")
+					(reference "R41")
 					(unit 1)
 				)
@@
 		(dnp no)
 		(fields_autoplaced yes)
-		(property "Reference" "#PWR042"
+		(property "Reference" "#PWR044"
 			(at 157.48 125.73 0)
 			(effects
@@
 			(project "Fill_Station_ControlBoard"
 				(path "/eaacffe0-ee57-428e-a37e-5655e0922ccc/86dfffbf-ac08-41cb-ab8f-382cca5b005c"
-					(reference "#PWR042")
+					(reference "#PWR044")
 					(unit 1)
 				)
@@
 		(dnp no)
 		(fields_autoplaced yes)
-		(property "Reference" "C47"
+		(property "Reference" "C14"
 			(at 208.28 120.6499 0)
 			(effects
@@
 			(project "Fill_Station_ControlBoard"
 				(path "/eaacffe0-ee57-428e-a37e-5655e0922ccc/86dfffbf-ac08-41cb-ab8f-382cca5b005c"
-					(reference "C47")
+					(reference "C14")
 					(unit 1)
 				)
@@
 		(dnp no)
 		(fields_autoplaced yes)
-		(property "Reference" "C46"
+		(property "Reference" "C13"
 			(at 189.23 66.0399 0)
 			(effects
@@
 			(project "Fill_Station_ControlBoard"
 				(path "/eaacffe0-ee57-428e-a37e-5655e0922ccc/86dfffbf-ac08-41cb-ab8f-382cca5b005c"
-					(reference "C46")
+					(reference "C13")
 					(unit 1)
 				)
@@
 		(dnp no)
 		(fields_autoplaced yes)
-		(property "Reference" "R66"
+		(property "Reference" "R48"
 			(at 151.13 67.3099 0)
 			(effects
@@
 			)
 		)
-		(property "Footprint" ""
+		(property "Footprint" "Resistor_SMD:R_0402_1005Metric"
 			(at 149.606 68.834 90)
 			(effects
@@
 			(project "Fill_Station_ControlBoard"
 				(path "/eaacffe0-ee57-428e-a37e-5655e0922ccc/86dfffbf-ac08-41cb-ab8f-382cca5b005c"
-					(reference "R66")
+					(reference "R48")
 					(unit 1)
 				)
@@
 		(dnp no)
 		(fields_autoplaced yes)
-		(property "Reference" "#PWR073"
+		(property "Reference" "#PWR047"
 			(at 204.47 134.62 0)
 			(effects
@@
 			(project "Fill_Station_ControlBoard"
 				(path "/eaacffe0-ee57-428e-a37e-5655e0922ccc/86dfffbf-ac08-41cb-ab8f-382cca5b005c"
-					(reference "#PWR073")
+					(reference "#PWR047")
 					(unit 1)
 				)
@@
 		(dnp no)
 		(fields_autoplaced yes)
-		(property "Reference" "#PWR072"
+		(property "Reference" "#PWR046"
 			(at 173.99 78.74 0)
 			(effects
@@
 			(project "Fill_Station_ControlBoard"
 				(path "/eaacffe0-ee57-428e-a37e-5655e0922ccc/86dfffbf-ac08-41cb-ab8f-382cca5b005c"
-					(reference "#PWR072")
+					(reference "#PWR046")
 					(unit 1)
 				)
@@
 		(on_board yes)
 		(dnp no)
-		(property "Reference" "#PWR052"
+		(property "Reference" "#PWR043"
 			(at 124.46 63.5 0)
 			(effects
@@
 			(project "Fill_Station_ControlBoard"
 				(path "/eaacffe0-ee57-428e-a37e-5655e0922ccc/86dfffbf-ac08-41cb-ab8f-382cca5b005c"
-					(reference "#PWR052")
+					(reference "#PWR043")
 					(unit 1)
 				)
@@
 		(dnp no)
 		(fields_autoplaced yes)
-		(property "Reference" "R64"
+		(property "Reference" "R46"
 			(at 134.62 67.3099 0)
 			(effects
@@
 			)
 		)
-		(property "Footprint" ""
+		(property "Footprint" "Resistor_SMD:R_0402_1005Metric"
 			(at 133.096 68.834 90)
 			(effects
@@
 			(project "Fill_Station_ControlBoard"
 				(path "/eaacffe0-ee57-428e-a37e-5655e0922ccc/86dfffbf-ac08-41cb-ab8f-382cca5b005c"
-					(reference "R64")
+					(reference "R46")
 					(unit 1)
 				)
@@
 		(on_board yes)
 		(dnp no)
-		(property "Reference" "R60"
+		(property "Reference" "R42"
 			(at 87.376 109.474 90)
 			(effects
@@
 			)
 		)
-		(property "Footprint" ""
+		(property "Footprint" "Resistor_SMD:R_0402_1005Metric"
 			(at 91.694 109.474 90)
 			(effects
@@
 			(project "Fill_Station_ControlBoard"
 				(path "/eaacffe0-ee57-428e-a37e-5655e0922ccc/86dfffbf-ac08-41cb-ab8f-382cca5b005c"
-					(reference "R60")
+					(reference "R42")
 					(unit 1)
 				)
@@
 		(on_board yes)
 		(dnp no)
-		(property "Reference" "R57"
+		(property "Reference" "R40"
 			(at 85.852 94.234 90)
 			(effects
@@
 			)
 		)
-		(property "Footprint" ""
+		(property "Footprint" "Resistor_SMD:R_0402_1005Metric"
 			(at 90.424 94.234 90)
 			(effects
@@
 			(project "Fill_Station_ControlBoard"
 				(path "/eaacffe0-ee57-428e-a37e-5655e0922ccc/86dfffbf-ac08-41cb-ab8f-382cca5b005c"
-					(reference "R57")
+					(reference "R40")
 					(unit 1)
 				)
@@
 		(dnp no)
 		(fields_autoplaced yes)
-		(property "Reference" "R63"
+		(property "Reference" "R45"
 			(at 127 67.3099 0)
 			(effects
@@
 			)
 		)
-		(property "Footprint" ""
+		(property "Footprint" "Resistor_SMD:R_0402_1005Metric"
 			(at 125.476 68.834 90)
 			(effects
@@
 			(project "Fill_Station_ControlBoard"
 				(path "/eaacffe0-ee57-428e-a37e-5655e0922ccc/86dfffbf-ac08-41cb-ab8f-382cca5b005c"
-					(reference "R63")
+					(reference "R45")
 					(unit 1)
 				)
@@
 		(dnp no)
 		(fields_autoplaced yes)
-		(property "Reference" "R62"
+		(property "Reference" "R44"
 			(at 118.11 67.3099 0)
 			(effects
@@
 			)
 		)
-		(property "Footprint" ""
+		(property "Footprint" "Resistor_SMD:R_0402_1005Metric"
 			(at 116.586 68.834 90)
 			(effects
@@
 			(project "Fill_Station_ControlBoard"
 				(path "/eaacffe0-ee57-428e-a37e-5655e0922ccc/86dfffbf-ac08-41cb-ab8f-382cca5b005c"
-					(reference "R62")
+					(reference "R44")
 					(unit 1)
 				)
@@
 		(dnp no)
 		(fields_autoplaced yes)
-		(property "Reference" "J2"
+		(property "Reference" "J11"
 			(at 184.785 81.28 0)
 			(effects
@@
 			(project "Fill_Station_ControlBoard"
 				(path "/eaacffe0-ee57-428e-a37e-5655e0922ccc/86dfffbf-ac08-41cb-ab8f-382cca5b005c"
-					(reference "J2")
+					(reference "J11")
 					(unit 1)
 				)
@@
 		(dnp no)
 		(fields_autoplaced yes)
-		(property "Reference" "C45"
+		(property "Reference" "C12"
 			(at 177.8 66.0399 0)
 			(effects
@@
 			(project "Fill_Station_ControlBoard"
 				(path "/eaacffe0-ee57-428e-a37e-5655e0922ccc/86dfffbf-ac08-41cb-ab8f-382cca5b005c"
-					(reference "C45")
+					(reference "C12")
 					(unit 1)
 				)
@@
 		(on_board yes)
 		(dnp no)
-		(property "Reference" "R59"
+		(property "Reference" "R39"
 			(at 78.232 106.934 90)
 			(effects
@@
 			)
 		)
-		(property "Footprint" ""
+		(property "Footprint" "Resistor_SMD:R_0402_1005Metric"
 			(at 82.804 106.934 90)
 			(effects
@@
 			(project "Fill_Station_ControlBoard"
 				(path "/eaacffe0-ee57-428e-a37e-5655e0922ccc/86dfffbf-ac08-41cb-ab8f-382cca5b005c"
-					(reference "R59")
+					(reference "R39")
 					(unit 1)
 				)
@@
 		(on_board yes)
 		(dnp no)
-		(property "Reference" "#PWR063"
+		(property "Reference" "#PWR045"
 			(at 158.75 63.5 0)
 			(effects
@@
 			(project "Fill_Station_ControlBoard"
 				(path "/eaacffe0-ee57-428e-a37e-5655e0922ccc/86dfffbf-ac08-41cb-ab8f-382cca5b005c"
-					(reference "#PWR063")
+					(reference "#PWR045")
 					(unit 1)
 				)
@@
 		(on_board yes)
 		(dnp no)
-		(property "Reference" "R56"
+		(property "Reference" "R38"
 			(at 77.216 91.694 90)
 			(effects
@@
 			)
 		)
-		(property "Footprint" ""
+		(property "Footprint" "Resistor_SMD:R_0402_1005Metric"
 			(at 81.534 91.694 90)
 			(effects
@@
 			(project "Fill_Station_ControlBoard"
 				(path "/eaacffe0-ee57-428e-a37e-5655e0922ccc/86dfffbf-ac08-41cb-ab8f-382cca5b005c"
-					(reference "R56")
+					(reference "R38")
 					(unit 1)
 				)
@@
 		(dnp no)
 		(fields_autoplaced yes)
-		(property "Reference" "R65"
+		(property "Reference" "R47"
 			(at 143.51 67.3099 0)
 			(effects
@@
 			)
 		)
-		(property "Footprint" ""
+		(property "Footprint" "Resistor_SMD:R_0402_1005Metric"
 			(at 141.986 68.834 90)
 			(effects
@@
 			(project "Fill_Station_ControlBoard"
 				(path "/eaacffe0-ee57-428e-a37e-5655e0922ccc/86dfffbf-ac08-41cb-ab8f-382cca5b005c"
-					(reference "R65")
+					(reference "R47")
 					(unit 1)
 				)
@@
 		(dnp no)
 		(fields_autoplaced yes)
-		(property "Reference" "R61"
+		(property "Reference" "R43"
 			(at 109.22 67.3099 0)
 			(effects
@@
 			)
 		)
-		(property "Footprint" ""
+		(property "Footprint" "Resistor_SMD:R_0402_1005Metric"
 			(at 107.696 68.834 90)
 			(effects
@@
 			(project "Fill_Station_ControlBoard"
 				(path "/eaacffe0-ee57-428e-a37e-5655e0922ccc/86dfffbf-ac08-41cb-ab8f-382cca5b005c"
-					(reference "R61")
-					(unit 1)
-				)
+					(reference "R43")
+					(unit 1)
+				)

Commit message: PCB fait
Parts:
- removed J11: Micro_SD_Card_Det1, Connector_Card:microSD_HC_Molex_47219-2001, symbol Connector:Micro_SD_Card_Det1
- added C63, C86: 100n, Capacitor_SMD:C_0603_1608Metric, symbol Device:C
- added C65: 10u, Capacitor_SMD:C_0603_1608Metric, symbol Device:C
- added J10, J14: Micro_SD_Card_Det_Hirose_DM3AT, Connector_Card:microSD_HC_Hirose_DM3AT-SF-PEJM5, symbol Connector:Micro_SD_Card_Det_Hirose_DM3AT
- added R62, R90, R91, R92, R93: 22, Resistor_SMD:R_0402_1005Metric, symbol Device:R_US
- added R94, R95, R96, R97, R98: 10k, Resistor_SMD:R_0402_1005Metric, symbol Device:R_US
- C12: value 0.1u -> 100n
- C14: footprint (none) -> Capacitor_SMD:C_0603_1608Metric
Connections:
- net 3V3: now also C63.1, C65.1, J10.4 (VDD), J14.4 (VDD), R94.1, R95.1, R96.1, R97.1, R98.1
- net GND: now also C63.2, C65.2, C86.2, J10.6 (VSS), J10.9 (DET_B), J14.6 (VSS), J14.9 (DET_B)
- net SD.DET: now also J14.10 (DET_A)
- net at R41.2: now also J14.5 (CLK)
- net at C14.1: now also J14.11 (SHIELD)
- net at R39.2, R46.2: now also J14.7 (DAT0)
- net at R42.2, R47.2: now also J14.8 (DAT1)
- net at R40.2, R44.2: now also J14.2 (DAT3/CD)
- net at R38.2, R43.2: now also J14.1 (DAT2)
- net SD.CLK renamed SD1.CLK
- net SD.CMD renamed SD1.CMD
- net SD1.CMD: now also J14.3 (CMD)
- net SD.DAT0 renamed SD1.DAT0
- net SD.DAT1 renamed SD1.DAT1
- net SD.DAT2 renamed SD1.DAT2
- net SD.DAT3 renamed SD1.DAT3
- new net: J10.2 (DAT3/CD), R91.2, R95.2
- new net: J10.1 (DAT2), R62.2, R94.2
- new net: C86.1, J10.11 (SHIELD)
- new net: J10.5 (CLK), R92.2
- new net: J10.7 (DAT0), R90.2, R97.2
- new net: J10.8 (DAT1), R93.2, R98.2
- new net SD2.CLK: R92.1
- new net SD2.CMD: J10.3 (CMD), R96.2
- new net SD2.DAT0: R90.1
- new net SD2.DAT1: R93.1
- new net SD2.DAT2: R62.1
- new net SD2.DAT3: R91.1
- no-connect marks 0 -> 1

Commit message: Travail Layout
Parts:
- added R100, R99: 22, Resistor_SMD:R_0402_1005Metric, symbol Device:R_US
Connections:
- net SD1.CMD: now also R99.1; no longer J14.3 (CMD), R45.2
- net SD2.CMD: now also R100.1; no longer J10.3 (CMD), R96.2
- net SD2.DET: now reaches J10.10 (DET_A)
- new net: J10.3 (CMD), R100.2, R96.2
- new net: J14.3 (CMD), R45.2, R99.2
- no-connect marks 1 -> 0
Changed lines of the file:
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@@
 		(color 0 0 0 0)
 	)
-	(no_connect
-		(at 162.56 223.52)
-	)
 	(wire
 		(pts
@@
 	(wire
 		(pts
+			(xy 104.14 97.79) (xy 124.46 97.79)
+		)
+		(stroke
+			(width 0)
+			(type default)
+		)
+	)
+	(wire
+		(pts
 			(xy 107.95 171.45) (xy 116.84 171.45)
 		)
@@
 	(wire
 		(pts
-			(xy 71.12 97.79) (xy 124.46 97.79)
+			(xy 71.12 97.79) (xy 96.52 97.79)
 		)
 		(stroke
@@
 	(wire
 		(pts
+			(xy 151.13 223.52) (xy 162.56 223.52)
+		)
+		(stroke
+			(width 0)
+			(type default)
+		)
+	)
+	(wire
+		(pts
 			(xy 162.56 210.82) (xy 160.02 210.82)
 		)
@@
 	(wire
 		(pts
-			(xy 72.39 208.28) (xy 125.73 208.28)
+			(xy 72.39 208.28) (xy 96.52 208.28)
 		)
 		(stroke
@@
 		(pts
 			(xy 124.46 59.69) (xy 124.46 60.96)
+		)
+		(stroke
+			(width 0)
+			(type default)
+		)
+	)
+	(wire
+		(pts
+			(xy 104.14 208.28) (xy 125.73 208.28)
 		)
 		(stroke
@@
 		(shape input)
 		(at 72.39 208.28 180)
+		(effects
+			(font
+				(size 1.27 1.27)
+			)
+			(justify right)
+		)
+	)
+	(hierarchical_label "SD2.DET"
+		(shape output)
+		(at 151.13 223.52 180)
 		(effects
 			(font
@@
 	)
 	(symbol
+		(lib_id "Device:R_US")
+		(at 100.33 208.28 90)
+		(unit 1)
+		(exclude_from_sim no)
+		(in_bom yes)
+		(on_board yes)
+		(dnp no)
+		(property "Reference" "R100"
+			(at 96.012 207.264 90)
+			(effects
+				(font
+					(size 1.27 1.27)
+				)
+			)
+		)
+		(property "Value" "22"
+			(at 96.774 209.296 90)
+			(effects
+				(font
+					(size 1.27 1.27)
+				)
+			)
+		)
+		(property "Footprint" "Resistor_SMD:R_0402_1005Metric"
+			(at 100.584 207.264 90)
+			(effects
+				(font
+					(size 1.27 1.27)
+				)
+				(hide yes)
+			)
+		)
+		(property "Datasheet" "~"
+			(at 100.33 208.28 0)
+			(effects
+				(font
+					(size 1.27 1.27)
+				)
+				(hide yes)
+			)
+		)
+		(property "Description" "Resistor, US symbol"
+			(at 100.33 208.28 0)
+			(effects
+				(font
+					(size 1.27 1.27)
+				)
+				(hide yes)
+			)
+		)
+		(pin "2"
+		)
+		(pin "1"
+		)
+		(instances
+			(project "Fill_Station_ControlBoard"
+				(path "/eaacffe0-ee57-428e-a37e-5655e0922ccc/86dfffbf-ac08-41cb-ab8f-382cca5b005c"
+					(reference "R100")
+					(unit 1)
+				)
+			)
+		)
+	)
+	(symbol
 		(lib_id "Device:C")
 		(at 185.42 67.31 0)
@@
 					(unit 1)
 				)
+			)
+		)
+	)
+	(symbol
+		(lib_id "Device:R_US")
+		(at 100.33 97.79 90)
+		(unit 1)
+		(exclude_from_sim no)
+		(in_bom yes)
+		(on_board yes)
+		(dnp no)
+		(property "Reference" "R99"
+			(at 96.012 96.774 90)
+			(effects
+				(font
+					(size 1.27 1.27)
+				)
+			)
+		)
+		(property "Value" "22"
+			(at 96.774 98.806 90)
+			(effects
+				(font
+					(size 1.27 1.27)
+				)
+			)
+		)
+		(property "Footprint" "Resistor_SMD:R_0402_1005Metric"
+			(at 100.584 96.774 90)
+			(effects
+				(font
+					(size 1.27 1.27)
+				)
+				(hide yes)
+			)
+		)
+		(property "Datasheet" "~"
+			(at 100.33 97.79 0)
+			(effects
+				(font
+					(size 1.27 1.27)
+				)
+				(hide yes)
+			)
+		)
+		(property "Description" "Resistor, US symbol"
+			(at 100.33 97.79 0)
+			(effects
+				(font
+					(size 1.27 1.27)
+				)
+				(hide yes)
+			)
+		)
+		(pin "2"
+		)
+		(pin "1"
+		)
+		(instances
+			(project "Fill_Station_ControlBoard"
+				(path "/eaacffe0-ee57-428e-a37e-5655e0922ccc/86dfffbf-ac08-41cb-ab8f-382cca5b005c"
+					(reference "R99")
+					(unit 1)
+				)

Commit message: PCB presque terminé
Modifs de l'alim
Changed lines of the file:
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@@
 	(wire
 		(pts
-			(xy 151.13 223.52) (xy 162.56 223.52)
+			(xy 72.39 223.52) (xy 162.56 223.52)
 		)
 		(stroke
@@
 	(hierarchical_label "SD2.DET"
 		(shape output)
-		(at 151.13 223.52 180)
-		(effects
-			(font
+		(at 72.39 223.52 180)
+		(effects
+			(font

Commit message: Final_V1
Parts:
- added R12: 10k, Resistor_SMD:R_0402_1005Metric, symbol Device:R_US
- C12, C14, C63, C86: LCSC (none) -> C14663
- C13, C65: LCSC (none) -> C22399626
- J10: LCSC (none) -> C114218
- J14: value Micro_SD_Card_Det_Hirose_DM3AT -> Micro_SD_Card_Det_Hirose_DM3CS; footprint Connector_Card:microSD_HC_Hirose_DM3AT-SF-PEJM5 -> DM3CS-SF:HRS_DM3CS-SF; LCSC (none) -> C202111
- R100, R38, R39, R40, R41, R42, R62, R90, R91, R92, R93, R99: LCSC (none) -> C25092
- R43, R44, R45, R46, R47, R48, R94, R95, R96, R97, R98: LCSC (none) -> C173683
Connections:
- net 3V3: now also R12.1
- net GND: now also J14.10 (DET_A); no longer J14.9 (DET_B)
- net SD.DET: now also J14.9 (DET_B); no longer J14.10 (DET_A)
- net SD2.DET: now also R12.2
