File: Fill_Station_ControlBoard/USB.kicad_sch (KiCad schematic)
At the start: 9 parts, among them J3 USB_C_Receptacle_USB2.0_14P, U2 USBLC6-2SC6

Commit message: Ajout power
Parts:
- removed C6: 0.1uF, Capacitor_SMD:C_0603_1608Metric, symbol Device:C
- removed C7: 10uF, Capacitor_SMD:C_0603_1608Metric, symbol Device:C
- added R12, R13: 22, Capacitor_SMD:C_0603_1608Metric, symbol Device:R_US
Connections:
- net USB_N: now also R12.2; no longer U2.4 (I/O2)
- net USB_P: now also R13.1; no longer U2.6 (I/O1)
- net D-: now reaches J3.A7 (D-), J3.B7 (D-), U2.1 (I/O1)
- net D+: now reaches J3.A6 (D+), J3.B6 (D+), U2.3 (I/O2)
- net +5V renamed 5V_USB
- new net: R12.1, U2.4 (I/O2)
- new net: R13.2, U2.6 (I/O1)
Other:
- moved on the sheet: D3

Commit message: Ajout de footprint
Parts:
- D3: footprint (none) -> Diode_SMD:D_0603_1608Metric
- F3: footprint (none) -> Fuse:Fuse_0603_1608Metric
Changed lines of the file:
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@@
 			)
 		)
-		(property "Footprint" ""
+		(property "Footprint" "Fuse:Fuse_0603_1608Metric"
 			(at 143.51 72.39 0)
 			(effects
@@
 			)
 		)
-		(property "Footprint" ""
+		(property "Footprint" "Diode_SMD:D_0603_1608Metric"
 			(at 158.75 81.28 0)
 			(effects

Commit message: début layout
Parts:
- renumbered C35 to C66, D3 to D15, F3 to F2, J3 to J15, R3 to R79, R4 to R80, R13 to R81, R12 to R82, U2 to U7
Changed lines of the file:
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@@
 		(on_board yes)
 		(dnp no)
-		(property "Reference" "#PWR015"
+		(property "Reference" "#PWR0127"
 			(at 137.16 106.68 0)
 			(effects
@@
 			(project "Fill_Station_ControlBoard"
 				(path "/eaacffe0-ee57-428e-a37e-5655e0922ccc/bd5f43b0-eb43-448d-8e3c-0f3b56e55349"
-					(reference "#PWR015")
+					(reference "#PWR0127")
 					(unit 1)
 				)
@@
 		(dnp no)
 		(fields_autoplaced yes)
-		(property "Reference" "#PWR012"
+		(property "Reference" "#PWR0131"
 			(at 158.75 95.25 0)
 			(effects
@@
 			(project "Fill_Station_ControlBoard"
 				(path "/eaacffe0-ee57-428e-a37e-5655e0922ccc/bd5f43b0-eb43-448d-8e3c-0f3b56e55349"
-					(reference "#PWR012")
+					(reference "#PWR0131")
 					(unit 1)
 				)
@@
 		(dnp no)
 		(fields_autoplaced yes)
-		(property "Reference" "R3"
+		(property "Reference" "R79"
 			(at 138.43 86.3599 0)
 			(effects
@@
 			(project "Fill_Station_ControlBoard"
 				(path "/eaacffe0-ee57-428e-a37e-5655e0922ccc/bd5f43b0-eb43-448d-8e3c-0f3b56e55349"
-					(reference "R3")
+					(reference "R79")
 					(unit 1)
 				)
@@
 		(dnp no)
 		(fields_autoplaced yes)
-		(property "Reference" "F3"
+		(property "Reference" "F2"
 			(at 138.43 67.31 90)
 			(effects
@@
 			(project "Fill_Station_ControlBoard"
 				(path "/eaacffe0-ee57-428e-a37e-5655e0922ccc/bd5f43b0-eb43-448d-8e3c-0f3b56e55349"
-					(reference "F3")
+					(reference "F2")
 					(unit 1)
 				)
@@
 		(dnp no)
 		(fields_autoplaced yes)
-		(property "Reference" "#PWR014"
+		(property "Reference" "#PWR0126"
 			(at 106.68 132.08 0)
 			(effects
@@
 			(project "Fill_Station_ControlBoard"
 				(path "/eaacffe0-ee57-428e-a37e-5655e0922ccc/bd5f43b0-eb43-448d-8e3c-0f3b56e55349"
-					(reference "#PWR014")
+					(reference "#PWR0126")
 					(unit 1)
 				)
@@
 		(dnp no)
 		(fields_autoplaced yes)
-		(property "Reference" "D3"
+		(property "Reference" "D15"
 			(at 161.29 80.0099 90)
 			(effects
@@
 			(project "Fill_Station_ControlBoard"
 				(path "/eaacffe0-ee57-428e-a37e-5655e0922ccc/bd5f43b0-eb43-448d-8e3c-0f3b56e55349"
-					(reference "D3")
+					(reference "D15")
 					(unit 1)
 				)
@@
 		(dnp no)
 		(fields_autoplaced yes)
-		(property "Reference" "U2"
+		(property "Reference" "U7"
 			(at 138.8111 102.87 0)
 			(effects
@@
 			(project "Fill_Station_ControlBoard"
 				(path "/eaacffe0-ee57-428e-a37e-5655e0922ccc/bd5f43b0-eb43-448d-8e3c-0f3b56e55349"
-					(reference "U2")
+					(reference "U7")
 					(unit 1)
 				)
@@
 		(on_board yes)
 		(dnp no)
-		(property "Reference" "#PWR010"
+		(property "Reference" "#PWR0130"
 			(at 158.75 72.39 0)
 			(effects
@@
 			(project "Fill_Station_ControlBoard"
 				(path "/eaacffe0-ee57-428e-a37e-5655e0922ccc/bd5f43b0-eb43-448d-8e3c-0f3b56e55349"
-					(reference "#PWR010")
+					(reference "#PWR0130")
 					(unit 1)
 				)
@@
 		(on_board yes)
 		(dnp no)
-		(property "Reference" "R4"
+		(property "Reference" "R80"
 			(at 146.05 86.3599 0)
 			(effects
@@
 			(project "Fill_Station_ControlBoard"
 				(path "/eaacffe0-ee57-428e-a37e-5655e0922ccc/bd5f43b0-eb43-448d-8e3c-0f3b56e55349"
-					(reference "R4")
+					(reference "R80")
 					(unit 1)
 				)
@@
 		(dnp no)
 		(fields_autoplaced yes)
-		(property "Reference" "#PWR016"
+		(property "Reference" "#PWR0128"
 			(at 137.16 128.27 0)
 			(effects
@@
 			(project "Fill_Station_ControlBoard"
 				(path "/eaacffe0-ee57-428e-a37e-5655e0922ccc/bd5f43b0-eb43-448d-8e3c-0f3b56e55349"
-					(reference "#PWR016")
+					(reference "#PWR0128")
 					(unit 1)
 				)
@@
 		(dnp no)
 		(fields_autoplaced yes)
-		(property "Reference" "#PWR013"
+		(property "Reference" "#PWR0129"
 			(at 143.51 101.6 0)
 			(effects
@@
 			(project "Fill_Station_ControlBoard"
 				(path "/eaacffe0-ee57-428e-a37e-5655e0922ccc/bd5f43b0-eb43-448d-8e3c-0f3b56e55349"
-					(reference "#PWR013")
+					(reference "#PWR0129")
 					(unit 1)
 				)
@@
 		(on_board yes)
 		(dnp no)
-		(property "Reference" "R13"
+		(property "Reference" "R81"
 			(at 159.512 108.204 90)
 			(effects
@@
 			(project "Fill_Station_ControlBoard"
 				(path "/eaacffe0-ee57-428e-a37e-5655e0922ccc/bd5f43b0-eb43-448d-8e3c-0f3b56e55349"
-					(reference "R13")
+					(reference "R81")
 					(unit 1)
 				)
@@
 		(on_board yes)
 		(dnp no)
-		(property "Reference" "R12"
+		(property "Reference" "R82"
 			(at 155.448 115.316 90)
 			(effects
@@
 			(project "Fill_Station_ControlBoard"
 				(path "/eaacffe0-ee57-428e-a37e-5655e0922ccc/bd5f43b0-eb43-448d-8e3c-0f3b56e55349"
-					(reference "R12")
+					(reference "R82")
 					(unit 1)
 				)
@@
 		(on_board yes)
 		(dnp no)
-		(property "Reference" "C35"
+		(property "Reference" "C66"
 			(at 99.314 117.094 0)
 			(effects
@@
 			(project "Fill_Station_ControlBoard"
 				(path "/eaacffe0-ee57-428e-a37e-5655e0922ccc/bd5f43b0-eb43-448d-8e3c-0f3b56e55349"
-					(reference "C35")
+					(reference "C66")
 					(unit 1)
 				)
@@
 		(dnp no)
 		(fields_autoplaced yes)
-		(property "Reference" "J3"
+		(property "Reference" "J15"
 			(at 106.68 66.04 0)
 			(effects
@@
 			(project "Fill_Station_ControlBoard"
 				(path "/eaacffe0-ee57-428e-a37e-5655e0922ccc/bd5f43b0-eb43-448d-8e3c-0f3b56e55349"
-					(reference "J3")
-					(unit 1)
-				)
+					(reference "J15")
+					(unit 1)
+				)

Commit message: PCB fait
Parts:
- J15: footprint Connector_USB:USB_C_Receptacle_Amphenol_12401548E4-2A_CircularHoles -> Connector_USB:USB_C_Receptacle_GCT_USB4105-xx-A_16P_TopMnt_Horizontal
Changed lines of the file:
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@@
 			)
 		)
-		(property "Footprint" "Connector_USB:USB_C_Receptacle_Amphenol_12401548E4-2A_CircularHoles"
+		(property "Footprint" "Connector_USB:USB_C_Receptacle_GCT_USB4105-xx-A_16P_TopMnt_Horizontal"
 			(at 110.49 88.9 0)
 			(effects

Commit message: finalisé le pcb
Connections:
- net USB_N: now also R81.1; no longer R82.2
- net USB_P: now also R82.2; no longer R81.1
Changed lines of the file:
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@@
 	(hierarchical_label "USB_N"
 		(shape output)
-		(at 177.8 113.03 0)
+		(at 177.8 110.49 0)
 		(effects
 			(font
@@
 	(hierarchical_label "USB_P"
 		(shape output)
-		(at 177.8 110.49 0)
+		(at 177.8 113.03 0)
 		(effects
 			(font

Commit message: Final_V1
Parts:
- C66: LCSC (none) -> C100042
- D15: footprint Diode_SMD:D_0603_1608Metric -> Diode_SMD:D_SOD-123; LCSC (none) -> C79598
- F2: footprint Fuse:Fuse_0603_1608Metric -> Fuse:Fuse_1206_3216Metric; LCSC (none) -> C70083
- J15: LCSC (none) -> C393939
- R79, R80: footprint Resistor_SMD:R_0603_1608Metric_Pad0.98x0.95mm_HandSolder -> Resistor_SMD:R_0402_1005Metric; LCSC (none) -> C25905
- R81, R82: footprint Capacitor_SMD:C_0603_1608Metric -> Resistor_SMD:R_0402_1005Metric; LCSC (none) -> C25092
- U7: LCSC (none) -> C7519
Changed lines of the file:
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@@
 			)
 		)
-		(property "Footprint" "Resistor_SMD:R_0603_1608Metric_Pad0.98x0.95mm_HandSolder"
+		(property "Footprint" "Resistor_SMD:R_0402_1005Metric"
 			(at 136.906 87.884 90)
 			(effects
@@
 		)
 		(property "Description" "Resistor, US symbol"
+			(at 135.89 87.63 0)
+			(effects
+				(font
+					(size 1.27 1.27)
+				)
+				(hide yes)
+			)
+		)
+		(property "LCSC" "C25905"
 			(at 135.89 87.63 0)
 			(effects
@@
 			)
 		)
-		(property "Footprint" "Fuse:Fuse_0603_1608Metric"
+		(property "Footprint" "Fuse:Fuse_1206_3216Metric"
 			(at 143.51 72.39 0)
 			(effects
@@
 		(property "Description" "Resettable fuse, polymeric positive temperature coefficient"
 			(at 138.43 73.66 0)
+			(effects
+				(font
+					(size 1.27 1.27)
+				)
+				(hide yes)
+			)
+		)
+		(property "LCSC" "C70083"
+			(at 138.43 73.66 90)
 			(effects
 				(font
@@
 			)
 		)
-		(property "Footprint" "Diode_SMD:D_0603_1608Metric"
+		(property "Footprint" "Diode_SMD:D_SOD-123"
 			(at 158.75 81.28 0)
 			(effects
@@
 		(property "Description" "Zener diode"
 			(at 158.75 81.28 0)
+			(effects
+				(font
+					(size 1.27 1.27)
+				)
+				(hide yes)
+			)
+		)
+		(property "LCSC" "C79598"
+			(at 158.75 81.28 90)
 			(effects
 				(font
@@
 			)
 		)
+		(property "LCSC" "C7519"
+			(at 137.16 110.49 0)
+			(effects
+				(font
+					(size 1.27 1.27)
+				)
+				(hide yes)
+			)
+		)
 		(pin "1"
 		)
@@
 			)
 		)
-		(property "Footprint" "Resistor_SMD:R_0603_1608Metric_Pad0.98x0.95mm_HandSolder"
+		(property "Footprint" "Resistor_SMD:R_0402_1005Metric"
 			(at 144.526 87.884 90)
 			(effects
@@
 		)
 		(property "Description" "Resistor, US symbol"
+			(at 143.51 87.63 0)
+			(effects
+				(font
+					(size 1.27 1.27)
+				)
+				(hide yes)
+			)
+		)
+		(property "LCSC" "C25905"
 			(at 143.51 87.63 0)
 			(effects
@@
 			)
 		)
-		(property "Footprint" "Capacitor_SMD:C_0603_1608Metric"
+		(property "Footprint" "Resistor_SMD:R_0402_1005Metric"
 			(at 157.226 111.506 90)
 			(effects
@@
 			)
 		)
+		(property "LCSC" "C25092"
+			(at 157.48 110.49 90)
+			(effects
+				(font
+					(size 1.27 1.27)
+				)
+				(hide yes)
+			)
+		)
 		(pin "2"
 		)
@@
 			)
 		)
-		(property "Footprint" "Capacitor_SMD:C_0603_1608Metric"
+		(property "Footprint" "Resistor_SMD:R_0402_1005Metric"
 			(at 157.734 112.014 90)
 			(effects
@@
 			)
 		)
+		(property "LCSC" "C25092"
+			(at 157.48 113.03 90)
+			(effects
+				(font
+					(size 1.27 1.27)
+				)
+				(hide yes)
+			)
+		)
 		(pin "2"
 		)
@@
 		)
 		(property "Description" "Unpolarized capacitor"
+			(at 99.06 119.38 0)
+			(effects
+				(font
+					(size 1.27 1.27)
+				)
+				(hide yes)
+			)
+		)
+		(property "LCSC" "C100042"
 			(at 99.06 119.38 0)
 			(effects
@@
 			(at 106.68 88.9 0)
 			(effects
+				(font
+					(size 1.27 1.27)
+				)
+				(hide yes)
+			)
+		)
+		(property "LCSC" "C393939"
+			(at 106.68 88.9 0)
+			(effects
